File: isokey/isokey.kicad_pcb (KiCad board)
At the start: 2 copper layers, 0 parts

Commit message: Place all sw
Parts:
- added D1: 1N4448W, Diode_SMD:D_SOD-123, F.Cu at (602.5, -47.0)
- added D10: 1N4448W, Diode_SMD:D_SOD-123, F.Cu at (614.1, -43.7)
- added D100: SK6812MINI, LED_SMD:LED_SK6812MINI_PLCC4_3.5x3.5mm_P1.75mm, F.Cu at (646.9, -31.0)
- added D101: SK6812MINI, LED_SMD:LED_SK6812MINI_PLCC4_3.5x3.5mm_P1.75mm, F.Cu at (646.9, -26.0)
- added D102: SK6812MINI, LED_SMD:LED_SK6812MINI_PLCC4_3.5x3.5mm_P1.75mm, F.Cu at (646.9, -20.9)
- added D103: SK6812MINI, LED_SMD:LED_SK6812MINI_PLCC4_3.5x3.5mm_P1.75mm, F.Cu at (646.9, -15.9)
- added D104: SK6812MINI, LED_SMD:LED_SK6812MINI_PLCC4_3.5x3.5mm_P1.75mm, F.Cu at (646.9, -10.8)
- added D105: SK6812MINI, LED_SMD:LED_SK6812MINI_PLCC4_3.5x3.5mm_P1.75mm, F.Cu at (646.9, -5.78)
- added D106: SK6812MINI, LED_SMD:LED_SK6812MINI_PLCC4_3.5x3.5mm_P1.75mm, F.Cu at (646.9, -0.72)
- added D107: SK6812MINI, LED_SMD:LED_SK6812MINI_PLCC4_3.5x3.5mm_P1.75mm, F.Cu at (646.9, 4.33)
- added D108: SK6812MINI, LED_SMD:LED_SK6812MINI_PLCC4_3.5x3.5mm_P1.75mm, F.Cu at (653.9, 4.33)
- added D109: SK6812MINI, LED_SMD:LED_SK6812MINI_PLCC4_3.5x3.5mm_P1.75mm, F.Cu at (661.0, -36.1)
- added D11: 1N4448W, Diode_SMD:D_SOD-123, F.Cu at (614.1, -33.6)
- added D110: SK6812MINI, LED_SMD:LED_SK6812MINI_PLCC4_3.5x3.5mm_P1.75mm, F.Cu at (661.0, -15.9)
- added D111: SK6812MINI, LED_SMD:LED_SK6812MINI_PLCC4_3.5x3.5mm_P1.75mm, F.Cu at (661.0, 4.33)
- added D112: SK6812MINI, LED_SMD:LED_SK6812MINI_PLCC4_3.5x3.5mm_P1.75mm, F.Cu at (646.9, 9.38)
- added D113: SK6812MINI, LED_SMD:LED_SK6812MINI_PLCC4_3.5x3.5mm_P1.75mm, F.Cu at (653.9, -41.1)
- added D114: SK6812MINI, LED_SMD:LED_SK6812MINI_PLCC4_3.5x3.5mm_P1.75mm, F.Cu at (653.9, -36.1)
- added D115: SK6812MINI, LED_SMD:LED_SK6812MINI_PLCC4_3.5x3.5mm_P1.75mm, F.Cu at (653.9, -31.0)
- added D116: SK6812MINI, LED_SMD:LED_SK6812MINI_PLCC4_3.5x3.5mm_P1.75mm, F.Cu at (653.9, -26.0)
- added D117: SK6812MINI, LED_SMD:LED_SK6812MINI_PLCC4_3.5x3.5mm_P1.75mm, F.Cu at (653.9, -20.9)
- added D118: SK6812MINI, LED_SMD:LED_SK6812MINI_PLCC4_3.5x3.5mm_P1.75mm, F.Cu at (653.9, -15.9)
- added D119: SK6812MINI, LED_SMD:LED_SK6812MINI_PLCC4_3.5x3.5mm_P1.75mm, F.Cu at (653.9, -10.8)
- added D12: 1N4448W, Diode_SMD:D_SOD-123, F.Cu at (614.1, -23.6)
- added D120: SK6812MINI, LED_SMD:LED_SK6812MINI_PLCC4_3.5x3.5mm_P1.75mm, F.Cu at (653.9, 9.38)
- added D121: SK6812MINI, LED_SMD:LED_SK6812MINI_PLCC4_3.5x3.5mm_P1.75mm, F.Cu at (661.0, -31.0)
- added D122: SK6812MINI, LED_SMD:LED_SK6812MINI_PLCC4_3.5x3.5mm_P1.75mm, F.Cu at (661.0, -10.8)
- added D123: SK6812MINI, LED_SMD:LED_SK6812MINI_PLCC4_3.5x3.5mm_P1.75mm, F.Cu at (661.0, 9.38)
- added D124: SK6812MINI, LED_SMD:LED_SK6812MINI_PLCC4_3.5x3.5mm_P1.75mm, F.Cu at (668.0, -46.2)
- added D125: SK6812MINI, LED_SMD:LED_SK6812MINI_PLCC4_3.5x3.5mm_P1.75mm, F.Cu at (668.0, -41.1)
- added D126: SK6812MINI, LED_SMD:LED_SK6812MINI_PLCC4_3.5x3.5mm_P1.75mm, F.Cu at (668.0, -36.1)
- added D127: SK6812MINI, LED_SMD:LED_SK6812MINI_PLCC4_3.5x3.5mm_P1.75mm, F.Cu at (668.0, -31.0)
- added D128: SK6812MINI, LED_SMD:LED_SK6812MINI_PLCC4_3.5x3.5mm_P1.75mm, F.Cu at (668.0, -26.0)
- added D129: SK6812MINI, LED_SMD:LED_SK6812MINI_PLCC4_3.5x3.5mm_P1.75mm, F.Cu at (668.0, -20.9)
- added D13: 1N4448W, Diode_SMD:D_SOD-123, F.Cu at (614.1, -13.5)
- added D130: SK6812MINI, LED_SMD:LED_SK6812MINI_PLCC4_3.5x3.5mm_P1.75mm, F.Cu at (668.0, -15.9)
- added D131: SK6812MINI, LED_SMD:LED_SK6812MINI_PLCC4_3.5x3.5mm_P1.75mm, F.Cu at (668.0, -10.8)
- added D132: SK6812MINI, LED_SMD:LED_SK6812MINI_PLCC4_3.5x3.5mm_P1.75mm, F.Cu at (668.0, -5.78)
- added D133: SK6812MINI, LED_SMD:LED_SK6812MINI_PLCC4_3.5x3.5mm_P1.75mm, F.Cu at (668.0, -0.72)
- added D134: SK6812MINI, LED_SMD:LED_SK6812MINI_PLCC4_3.5x3.5mm_P1.75mm, F.Cu at (668.0, 4.33)
- added D135: SK6812MINI, LED_SMD:LED_SK6812MINI_PLCC4_3.5x3.5mm_P1.75mm, F.Cu at (668.0, 9.38)
- added D136: SK6812MINI, LED_SMD:LED_SK6812MINI_PLCC4_3.5x3.5mm_P1.75mm, F.Cu at (675.0, -46.2)
- added D137: SK6812MINI, LED_SMD:LED_SK6812MINI_PLCC4_3.5x3.5mm_P1.75mm, F.Cu at (675.0, -41.1)
- added D138: SK6812MINI, LED_SMD:LED_SK6812MINI_PLCC4_3.5x3.5mm_P1.75mm, F.Cu at (675.0, -36.1)
- added D139: SK6812MINI, LED_SMD:LED_SK6812MINI_PLCC4_3.5x3.5mm_P1.75mm, F.Cu at (675.0, -31.0)
- added D14: 1N4448W, Diode_SMD:D_SOD-123, F.Cu at (619.9, -47.0)
- added D140: SK6812MINI, LED_SMD:LED_SK6812MINI_PLCC4_3.5x3.5mm_P1.75mm, F.Cu at (675.0, -26.0)
- added D141: SK6812MINI, LED_SMD:LED_SK6812MINI_PLCC4_3.5x3.5mm_P1.75mm, F.Cu at (675.0, -20.9)
- added D142: SK6812MINI, LED_SMD:LED_SK6812MINI_PLCC4_3.5x3.5mm_P1.75mm, F.Cu at (675.0, -15.9)
- added D143: SK6812MINI, LED_SMD:LED_SK6812MINI_PLCC4_3.5x3.5mm_P1.75mm, F.Cu at (675.0, -10.8)
- added D144: SK6812MINI, LED_SMD:LED_SK6812MINI_PLCC4_3.5x3.5mm_P1.75mm, F.Cu at (675.0, -5.78)
- added D145: SK6812MINI, LED_SMD:LED_SK6812MINI_PLCC4_3.5x3.5mm_P1.75mm, F.Cu at (675.0, -0.72)
- added D146: SK6812MINI, LED_SMD:LED_SK6812MINI_PLCC4_3.5x3.5mm_P1.75mm, F.Cu at (675.0, 4.33)
- added D147: SK6812MINI, LED_SMD:LED_SK6812MINI_PLCC4_3.5x3.5mm_P1.75mm, F.Cu at (675.0, 9.38)
- added D148: SK6812MINI, LED_SMD:LED_SK6812MINI_PLCC4_3.5x3.5mm_P1.75mm, F.Cu at (682.0, -46.2)
- added D149: SK6812MINI, LED_SMD:LED_SK6812MINI_PLCC4_3.5x3.5mm_P1.75mm, F.Cu at (682.0, -41.1)
- added D15: 1N4448W, Diode_SMD:D_SOD-123, F.Cu at (619.9, -37.0)
- added D150: SK6812MINI, LED_SMD:LED_SK6812MINI_PLCC4_3.5x3.5mm_P1.75mm, F.Cu at (682.0, -36.1)
- added D151: SK6812MINI, LED_SMD:LED_SK6812MINI_PLCC4_3.5x3.5mm_P1.75mm, F.Cu at (682.0, -31.0)
- added D152: SK6812MINI, LED_SMD:LED_SK6812MINI_PLCC4_3.5x3.5mm_P1.75mm, F.Cu at (682.0, -26.0)
- added D16: 1N4448W, Diode_SMD:D_SOD-123, F.Cu at (602.5, -30.3)
- added D17: 1N4448W, Diode_SMD:D_SOD-123, F.Cu at (602.5, -26.9)
- added D18: 1N4448W, Diode_SMD:D_SOD-123, F.Cu at (602.5, -23.6)
- added D19: 1N4448W, Diode_SMD:D_SOD-123, F.Cu at (602.5, -20.2)
- added D2: 1N4448W, Diode_SMD:D_SOD-123, F.Cu at (602.5, -43.7)
- added D20: 1N4448W, Diode_SMD:D_SOD-123, F.Cu at (602.5, -16.9)
- added D21: 1N4448W, Diode_SMD:D_SOD-123, F.Cu at (608.3, -37.0)
- added D22: 1N4448W, Diode_SMD:D_SOD-123, F.Cu at (608.3, -26.9)
- added D23: 1N4448W, Diode_SMD:D_SOD-123, F.Cu at (608.3, -16.9)
- added D24: 1N4448W, Diode_SMD:D_SOD-123, F.Cu at (608.3, -6.83)
- added D25: 1N4448W, Diode_SMD:D_SOD-123, F.Cu at (614.1, -40.3)
- added D26: 1N4448W, Diode_SMD:D_SOD-123, F.Cu at (614.1, -30.3)
- added D27: 1N4448W, Diode_SMD:D_SOD-123, F.Cu at (614.1, -20.2)
- added D28: 1N4448W, Diode_SMD:D_SOD-123, F.Cu at (614.1, -10.2)
- added D29: 1N4448W, Diode_SMD:D_SOD-123, F.Cu at (619.9, -43.7)
- added D3: 1N4448W, Diode_SMD:D_SOD-123, F.Cu at (602.5, -40.3)
- added D30: 1N4448W, Diode_SMD:D_SOD-123, F.Cu at (619.9, -33.6)
- added D31: 1N4448W, Diode_SMD:D_SOD-123, F.Cu at (602.5, -13.5)
- added D32: 1N4448W, Diode_SMD:D_SOD-123, F.Cu at (602.5, -10.2)
- added D33: 1N4448W, Diode_SMD:D_SOD-123, F.Cu at (602.5, -6.83)
- added D34: 1N4448W, Diode_SMD:D_SOD-123, F.Cu at (608.3, -47.0)
- added D35: 1N4448W, Diode_SMD:D_SOD-123, F.Cu at (608.3, -43.7)
- added D36: 1N4448W, Diode_SMD:D_SOD-123, F.Cu at (608.3, -33.6)
- added D37: 1N4448W, Diode_SMD:D_SOD-123, F.Cu at (608.3, -23.6)
- added D38: 1N4448W, Diode_SMD:D_SOD-123, F.Cu at (608.3, -13.5)
- added D39: 1N4448W, Diode_SMD:D_SOD-123, F.Cu at (614.1, -47.0)
- added D4: 1N4448W, Diode_SMD:D_SOD-123, F.Cu at (602.5, -37.0)
- added D40: 1N4448W, Diode_SMD:D_SOD-123, F.Cu at (614.1, -37.0)
- added D41: 1N4448W, Diode_SMD:D_SOD-123, F.Cu at (614.1, -26.9)
- added D42: 1N4448W, Diode_SMD:D_SOD-123, F.Cu at (614.1, -16.9)
- added D43: 1N4448W, Diode_SMD:D_SOD-123, F.Cu at (614.1, -6.83)
- added D44: 1N4448W, Diode_SMD:D_SOD-123, F.Cu at (619.9, -40.3)
- added D45: 1N4448W, Diode_SMD:D_SOD-123, F.Cu at (619.9, -30.3)
- added D46: 1N4448W, Diode_SMD:D_SOD-123, F.Cu at (619.9, -26.9)
- added D47: 1N4448W, Diode_SMD:D_SOD-123, F.Cu at (619.9, -23.6)
- added D48: 1N4448W, Diode_SMD:D_SOD-123, F.Cu at (619.9, -20.2)
- added D49: 1N4448W, Diode_SMD:D_SOD-123, F.Cu at (619.9, -16.9)
- added D5: 1N4448W, Diode_SMD:D_SOD-123, F.Cu at (602.5, -33.6)
- added D50: 1N4448W, Diode_SMD:D_SOD-123, F.Cu at (619.9, -13.5)
- added D51: 1N4448W, Diode_SMD:D_SOD-123, F.Cu at (619.9, -10.2)
- added D52: 1N4448W, Diode_SMD:D_SOD-123, F.Cu at (619.9, -6.83)
- added D53: 1N4448W, Diode_SMD:D_SOD-123, F.Cu at (625.7, -47.0)
- added D54: 1N4448W, Diode_SMD:D_SOD-123, F.Cu at (625.7, -43.7)
- added D55: 1N4448W, Diode_SMD:D_SOD-123, F.Cu at (625.7, -40.3)
- added D56: 1N4448W, Diode_SMD:D_SOD-123, F.Cu at (625.7, -37.0)
- added D57: 1N4448W, Diode_SMD:D_SOD-123, F.Cu at (625.7, -33.6)
- added D58: 1N4448W, Diode_SMD:D_SOD-123, F.Cu at (625.7, -30.3)
- added D59: 1N4448W, Diode_SMD:D_SOD-123, F.Cu at (625.7, -26.9)
- added D6: 1N4448W, Diode_SMD:D_SOD-123, F.Cu at (608.3, -40.3)
- added D60: 1N4448W, Diode_SMD:D_SOD-123, F.Cu at (625.7, -23.6)
- added D61: 1N4448W, Diode_SMD:D_SOD-123, F.Cu at (625.7, -20.2)
- added D62: 1N4448W, Diode_SMD:D_SOD-123, F.Cu at (625.7, -16.9)
- added D63: 1N4448W, Diode_SMD:D_SOD-123, F.Cu at (625.7, -13.5)
- added D64: 1N4448W, Diode_SMD:D_SOD-123, F.Cu at (625.7, -10.2)
- added D65: 1N4448W, Diode_SMD:D_SOD-123, F.Cu at (625.7, -6.83)
- added D66: 1N4448W, Diode_SMD:D_SOD-123, F.Cu at (631.5, -47.0)
- added D67: 1N4448W, Diode_SMD:D_SOD-123, F.Cu at (631.5, -43.7)
- added D68: 1N4448W, Diode_SMD:D_SOD-123, F.Cu at (631.5, -40.3)
- added D69: 1N4448W, Diode_SMD:D_SOD-123, F.Cu at (631.5, -37.0)
- added D7: 1N4448W, Diode_SMD:D_SOD-123, F.Cu at (608.3, -30.3)
- added D70: 1N4448W, Diode_SMD:D_SOD-123, F.Cu at (631.5, -33.6)
- added D71: 1N4448W, Diode_SMD:D_SOD-123, F.Cu at (631.5, -30.3)
- added D72: 1N4448W, Diode_SMD:D_SOD-123, F.Cu at (631.5, -26.9)
- added D73: 1N4448W, Diode_SMD:D_SOD-123, F.Cu at (631.5, -23.6)
- added D74: 1N4448W, Diode_SMD:D_SOD-123, F.Cu at (631.5, -20.2)
- added D75: 1N4448W, Diode_SMD:D_SOD-123, F.Cu at (631.5, -16.9)
- added D76: SK6812MINI, LED_SMD:LED_SK6812MINI_PLCC4_3.5x3.5mm_P1.75mm, F.Cu at (653.9, -46.2)
- added D77: SK6812MINI, LED_SMD:LED_SK6812MINI_PLCC4_3.5x3.5mm_P1.75mm, F.Cu at (639.9, -46.2)
- added D78: SK6812MINI, LED_SMD:LED_SK6812MINI_PLCC4_3.5x3.5mm_P1.75mm, F.Cu at (639.9, -41.1)
- added D79: SK6812MINI, LED_SMD:LED_SK6812MINI_PLCC4_3.5x3.5mm_P1.75mm, F.Cu at (639.9, -36.1)
- added D8: 1N4448W, Diode_SMD:D_SOD-123, F.Cu at (608.3, -20.2)
- added D80: SK6812MINI, LED_SMD:LED_SK6812MINI_PLCC4_3.5x3.5mm_P1.75mm, F.Cu at (639.9, -31.0)
- added D81: SK6812MINI, LED_SMD:LED_SK6812MINI_PLCC4_3.5x3.5mm_P1.75mm, F.Cu at (639.9, -26.0)
- added D82: SK6812MINI, LED_SMD:LED_SK6812MINI_PLCC4_3.5x3.5mm_P1.75mm, F.Cu at (639.9, -20.9)
- added D83: SK6812MINI, LED_SMD:LED_SK6812MINI_PLCC4_3.5x3.5mm_P1.75mm, F.Cu at (646.9, -46.2)
- added D84: SK6812MINI, LED_SMD:LED_SK6812MINI_PLCC4_3.5x3.5mm_P1.75mm, F.Cu at (653.9, -5.78)
- added D85: SK6812MINI, LED_SMD:LED_SK6812MINI_PLCC4_3.5x3.5mm_P1.75mm, F.Cu at (661.0, -46.2)
- added D86: SK6812MINI, LED_SMD:LED_SK6812MINI_PLCC4_3.5x3.5mm_P1.75mm, F.Cu at (661.0, -26.0)
- added D87: SK6812MINI, LED_SMD:LED_SK6812MINI_PLCC4_3.5x3.5mm_P1.75mm, F.Cu at (661.0, -5.78)
- added D88: SK6812MINI, LED_SMD:LED_SK6812MINI_PLCC4_3.5x3.5mm_P1.75mm, F.Cu at (639.9, -15.9)
- added D89: SK6812MINI, LED_SMD:LED_SK6812MINI_PLCC4_3.5x3.5mm_P1.75mm, F.Cu at (639.9, -10.8)
- added D9: 1N4448W, Diode_SMD:D_SOD-123, F.Cu at (608.3, -10.2)
- added D90: SK6812MINI, LED_SMD:LED_SK6812MINI_PLCC4_3.5x3.5mm_P1.75mm, F.Cu at (639.9, -5.78)
- added D91: SK6812MINI, LED_SMD:LED_SK6812MINI_PLCC4_3.5x3.5mm_P1.75mm, F.Cu at (639.9, -0.72)
- added D92: SK6812MINI, LED_SMD:LED_SK6812MINI_PLCC4_3.5x3.5mm_P1.75mm, F.Cu at (639.9, 4.33)
- added D93: SK6812MINI, LED_SMD:LED_SK6812MINI_PLCC4_3.5x3.5mm_P1.75mm, F.Cu at (639.9, 9.38)
- added D94: SK6812MINI, LED_SMD:LED_SK6812MINI_PLCC4_3.5x3.5mm_P1.75mm, F.Cu at (646.9, -41.1)
- added D95: SK6812MINI, LED_SMD:LED_SK6812MINI_PLCC4_3.5x3.5mm_P1.75mm, F.Cu at (646.9, -36.1)
- added D96: SK6812MINI, LED_SMD:LED_SK6812MINI_PLCC4_3.5x3.5mm_P1.75mm, F.Cu at (653.9, -0.72)
- added D97: SK6812MINI, LED_SMD:LED_SK6812MINI_PLCC4_3.5x3.5mm_P1.75mm, F.Cu at (661.0, -41.1)
- added D98: SK6812MINI, LED_SMD:LED_SK6812MINI_PLCC4_3.5x3.5mm_P1.75mm, F.Cu at (661.0, -20.9)
- added D99: SK6812MINI, LED_SMD:LED_SK6812MINI_PLCC4_3.5x3.5mm_P1.75mm, F.Cu at (661.0, -0.72)
- added REF**: Stabilizer_MX_2u, Button_Switch_Keyboard:Stabilizer_MX_2u, F.Cu at (349.9, 112.6)
- added REF**: Stabilizer_MX_2u, Button_Switch_Keyboard:Stabilizer_MX_2u, F.Cu at (220.8, 196.2)
- added REF**: Stabilizer_MX_2u, Button_Switch_Keyboard:Stabilizer_MX_2u, F.Cu at (159.2, 196.8)
- added REF**: Stabilizer_MX_2u, Button_Switch_Keyboard:Stabilizer_MX_2u, F.Cu at (347.5, 141.1)
- added SW1: Cherry, Button_Switch_Keyboard:SW_MX, F.Cu at (75.1, 89.6)
- added SW10: Cherry, Button_Switch_Keyboard:SW_MX, F.Cu at (205.5, 119.2)
- added SW11: Cherry, Button_Switch_Keyboard:SW_MX, F.Cu at (224.5, 118.2)
- added SW12: Cherry, Button_Switch_Keyboard:SW_MX, F.Cu at (243.5, 117.2)
- added SW13: Cherry, Button_Switch_Keyboard:SW_MX, F.Cu at (262.5, 116.2)
- added SW14: Cherry, Button_Switch_Keyboard:SW_MX, F.Cu at (281.6, 115.2)
- added SW15: Cherry, Button_Switch_Keyboard:SW_MX, F.Cu at (300.6, 114.2)
- added SW16: Cherry, Button_Switch_Keyboard:SW_MX, F.Cu at (319.6, 113.2)
- added SW17: Cherry, Button_Switch_Keyboard:SW_MX, F.Cu at (349.9, 112.6)
- added SW18: Cherry, Button_Switch_Keyboard:SW_MX, F.Cu at (70.1, 133.5)
- added SW19: Cherry, Button_Switch_Keyboard:SW_MX, F.Cu at (97.4, 134.2)
- added SW2: Cherry, Button_Switch_Keyboard:SW_MX, F.Cu at (94.1, 89.6)
- added SW20: Cherry, Button_Switch_Keyboard:SW_MX, F.Cu at (116.5, 135.2)
- added SW21: Cherry, Button_Switch_Keyboard:SW_MX, F.Cu at (135.5, 136.2)
- added SW22: Cherry, Button_Switch_Keyboard:SW_MX, F.Cu at (154.5, 137.2)
- added SW23: Cherry, Button_Switch_Keyboard:SW_MX, F.Cu at (173.5, 138.2)
- added SW24: Cherry, Button_Switch_Keyboard:SW_MX, F.Cu at (206.5, 138.2)
- added SW25: Cherry, Button_Switch_Keyboard:SW_MX, F.Cu at (225.5, 137.2)
- added SW26: Cherry, Button_Switch_Keyboard:SW_MX, F.Cu at (244.5, 136.2)
- added SW27: Cherry, Button_Switch_Keyboard:SW_MX, F.Cu at (263.5, 135.2)
- added SW28: Cherry, Button_Switch_Keyboard:SW_MX, F.Cu at (282.6, 134.2)
- added SW29: Cherry, Button_Switch_Keyboard:SW_MX, F.Cu at (301.6, 133.2)
- added SW3: Cherry, Button_Switch_Keyboard:SW_MX, F.Cu at (50.8, 108.5)
- added SW30: Cherry, Button_Switch_Keyboard:SW_MX, F.Cu at (320.6, 132.2)
- added SW31: Cherry, Button_Switch_Keyboard:SW_MX, F.Cu at (374.0, 134.7)
- added SW32: Cherry, Button_Switch_Keyboard:SW_MX, F.Cu at (67.7, 152.6)
- added SW33: Cherry, Button_Switch_Keyboard:SW_MX, F.Cu at (96.5, 153.2)
- added SW34: Cherry, Button_Switch_Keyboard:SW_MX, F.Cu at (115.5, 154.2)
- added SW35: Cherry, Button_Switch_Keyboard:SW_MX, F.Cu at (134.5, 155.2)
- added SW36: Cherry, Button_Switch_Keyboard:SW_MX, F.Cu at (153.5, 156.2)
- added SW37: Cherry, Button_Switch_Keyboard:SW_MX, F.Cu at (172.5, 157.2)
- added SW38: Cherry, Button_Switch_Keyboard:SW_MX, F.Cu at (207.5, 157.2)
- added SW39: Cherry, Button_Switch_Keyboard:SW_MX, F.Cu at (226.5, 156.2)
- added SW4: Cherry, Button_Switch_Keyboard:SW_MX, F.Cu at (74.9, 114.5)
- added SW40: Cherry, Button_Switch_Keyboard:SW_MX, F.Cu at (245.5, 155.2)
- added SW41: Cherry, Button_Switch_Keyboard:SW_MX, F.Cu at (264.5, 154.2)
- added SW42: Cherry, Button_Switch_Keyboard:SW_MX, F.Cu at (283.5, 153.2)
- added SW43: Cherry, Button_Switch_Keyboard:SW_MX, F.Cu at (302.6, 152.2)
- added SW44: Cherry, Button_Switch_Keyboard:SW_MX, F.Cu at (321.6, 151.2)
- added SW45: Cherry, Button_Switch_Keyboard:SW_MX, F.Cu at (347.5, 141.1)
- added SW46: Cherry, Button_Switch_Keyboard:SW_MX, F.Cu at (374.0, 153.8)
- added SW47: Cherry, Button_Switch_Keyboard:SW_MX, F.Cu at (72.5, 171.6)
- added SW48: Cherry, Button_Switch_Keyboard:SW_MX, F.Cu at (95.5, 172.3)
- added SW49: Cherry, Button_Switch_Keyboard:SW_MX, F.Cu at (114.5, 173.3)
- added SW5: Cherry, Button_Switch_Keyboard:SW_MX, F.Cu at (98.4, 115.2)
- added SW50: Cherry, Button_Switch_Keyboard:SW_MX, F.Cu at (133.5, 174.3)
- added SW51: Cherry, Button_Switch_Keyboard:SW_MX, F.Cu at (152.5, 175.2)
- added SW52: Cherry, Button_Switch_Keyboard:SW_MX, F.Cu at (171.6, 176.2)
- added SW53: Cherry, Button_Switch_Keyboard:SW_MX, F.Cu at (208.4, 176.2)
- added SW54: Cherry, Button_Switch_Keyboard:SW_MX, F.Cu at (227.5, 175.2)
- added SW55: Cherry, Button_Switch_Keyboard:SW_MX, F.Cu at (246.5, 174.3)
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Other:
- board outline added: 359.8 x 150.9 mm

Commit message: Place switch and leds
Parts:
- added C1: 100nF, Capacitor_SMD:C_0603_1608Metric_Pad1.08x0.95mm_HandSolder, B.Cu at (243.4, 125.8)
- added C10: 100nF, Capacitor_SMD:C_0603_1608Metric_Pad1.08x0.95mm_HandSolder, B.Cu at (265.4, 162.4)
- added C11: 100nF, Capacitor_SMD:C_0603_1608Metric_Pad1.08x0.95mm_HandSolder, B.Cu at (348.1, 150.2)
- added C12: 100nF, Capacitor_SMD:C_0603_1608Metric_Pad1.08x0.95mm_HandSolder, B.Cu at (224.6, 126.8)
- added C13: 100nF, Capacitor_SMD:C_0603_1608Metric_Pad1.08x0.95mm_HandSolder, B.Cu at (319.8, 121.8)
- added C14: 100nF, Capacitor_SMD:C_0603_1608Metric_Pad1.08x0.95mm_HandSolder, B.Cu at (373.8, 162.2)
- added C15: 100nF, Capacitor_SMD:C_0603_1608Metric_Pad1.08x0.95mm_HandSolder, B.Cu at (96.2, 161.8)
- added C16: 100nF, Capacitor_SMD:C_0603_1608Metric_Pad1.08x0.95mm_HandSolder, B.Cu at (74.6, 98.6)
- added C17: 100nF, Capacitor_SMD:C_0603_1608Metric_Pad1.08x0.95mm_HandSolder, B.Cu at (94.2, 98.0)
- added C18: 100nF, Capacitor_SMD:C_0603_1608Metric_Pad1.08x0.95mm_HandSolder, B.Cu at (152.8, 164.4)
- added C19: 100nF, Capacitor_SMD:C_0603_1608Metric_Pad1.08x0.95mm_HandSolder, B.Cu at (221.6, 206.8)
- added C2: 100nF, Capacitor_SMD:C_0603_1608Metric_Pad1.08x0.95mm_HandSolder, B.Cu at (349.4, 121.4)
- added C20: 100nF, Capacitor_SMD:C_0603_1608Metric_Pad1.08x0.95mm_HandSolder, B.Cu at (284.8, 161.4)
- added C21: 100nF, Capacitor_SMD:C_0603_1608Metric_Pad1.08x0.95mm_HandSolder, B.Cu at (226.6, 145.4)
- added C22: 100nF, Capacitor_SMD:C_0603_1608Metric_Pad1.08x0.95mm_HandSolder, B.Cu at (321.4, 141.2)
- added C23: 100nF, Capacitor_SMD:C_0603_1608Metric_Pad1.08x0.95mm_HandSolder, B.Cu at (206.0, 127.4)
- added C24: 100nF, Capacitor_SMD:C_0603_1608Metric_Pad1.08x0.95mm_HandSolder, B.Cu at (300.4, 122.6)
- added C25: 100nF, Capacitor_SMD:C_0603_1608Metric_Pad1.08x0.95mm_HandSolder, B.Cu at (158.5, 207.8)
- added C26: 100nF, Capacitor_SMD:C_0603_1608Metric_Pad1.08x0.95mm_HandSolder, B.Cu at (114.0, 182.6)
- added C27: 100nF, Capacitor_SMD:C_0603_1608Metric_Pad1.08x0.95mm_HandSolder, B.Cu at (174.0, 128.6)
- added C28: 100nF, Capacitor_SMD:C_0603_1608Metric_Pad1.08x0.95mm_HandSolder, B.Cu at (154.6, 127.4)
- added C29: 100nF, Capacitor_SMD:C_0603_1608Metric_Pad1.08x0.95mm_HandSolder, B.Cu at (135.6, 144.6)
- added C3: 100nF, Capacitor_SMD:C_0603_1608Metric_Pad1.08x0.95mm_HandSolder, B.Cu at (373.8, 181.6)
- added C30: 100nF, Capacitor_SMD:C_0603_1608Metric_Pad1.08x0.95mm_HandSolder, B.Cu at (259.4, 204.2)
- added C31: 100nF, Capacitor_SMD:C_0603_1608Metric_Pad1.08x0.95mm_HandSolder, B.Cu at (322.8, 160.2)
- added C32: 100nF, Capacitor_SMD:C_0603_1608Metric_Pad1.08x0.95mm_HandSolder, B.Cu at (206.8, 146.6)
- added C33: 100nF, Capacitor_SMD:C_0603_1608Metric_Pad1.08x0.95mm_HandSolder, B.Cu at (301.6, 142.0)
- added C34: 100nF, Capacitor_SMD:C_0603_1608Metric_Pad1.08x0.95mm_HandSolder, B.Cu at (243.4, 102.4)
- added C35: 100nF, Capacitor_SMD:C_0603_1608Metric_Pad1.08x0.95mm_HandSolder, B.Cu at (281.8, 123.6)
- added C36: 100nF, Capacitor_SMD:C_0603_1608Metric_Pad1.08x0.95mm_HandSolder, B.Cu at (122.2, 205.6)
- added C37: 100nF, Capacitor_SMD:C_0603_1608Metric_Pad1.08x0.95mm_HandSolder, B.Cu at (94.6, 181.2)
- added C38: 100nF, Capacitor_SMD:C_0603_1608Metric_Pad1.08x0.95mm_HandSolder, B.Cu at (170.4, 184.8)
- added C39: 100nF, Capacitor_SMD:C_0603_1608Metric_Pad1.08x0.95mm_HandSolder, B.Cu at (136.4, 126.2)
- added C4: 100nF, Capacitor_SMD:C_0603_1608Metric_Pad1.08x0.95mm_HandSolder, B.Cu at (96.8, 143.2)
- added C40: 100nF, Capacitor_SMD:C_0603_1608Metric_Pad1.08x0.95mm_HandSolder, B.Cu at (116.4, 143.6)
- added C41: 100nF, Capacitor_SMD:C_0603_1608Metric_Pad1.08x0.95mm_HandSolder, B.Cu at (282.4, 206.0)
- added C42: 100nF, Capacitor_SMD:C_0603_1608Metric_Pad1.08x0.95mm_HandSolder, B.Cu at (306.4, 179.8)
- added C43: 100nF, Capacitor_SMD:C_0603_1608Metric_Pad1.08x0.95mm_HandSolder, B.Cu at (246.6, 164.0)
- added C44: 100nF, Capacitor_SMD:C_0603_1608Metric_Pad1.08x0.95mm_HandSolder, B.Cu at (282.8, 142.8)
- added C45: 100nF, Capacitor_SMD:C_0603_1608Metric_Pad1.08x0.95mm_HandSolder, B.Cu at (205.0, 104.8)
- added C46: 100nF, Capacitor_SMD:C_0603_1608Metric_Pad1.08x0.95mm_HandSolder, B.Cu at (263.1, 125.2)
- added C47: 100nF, Capacitor_SMD:C_0603_1608Metric_Pad1.08x0.95mm_HandSolder, B.Cu at (360.8, 205.0)
- added C48: 100nF, Capacitor_SMD:C_0603_1608Metric_Pad1.08x0.95mm_HandSolder, B.Cu at (73.5, 180.8)
- added C49: 100nF, Capacitor_SMD:C_0603_1608Metric_Pad1.08x0.95mm_HandSolder, B.Cu at (116.2, 125.4)
- added C5: 100nF, Capacitor_SMD:C_0603_1608Metric_Pad1.08x0.95mm_HandSolder, B.Cu at (51.4, 117.0)
- added C50: 100nF, Capacitor_SMD:C_0603_1608Metric_Pad1.08x0.95mm_HandSolder, B.Cu at (97.0, 124.0)
- added C51: 100nF, Capacitor_SMD:C_0603_1608Metric_Pad1.08x0.95mm_HandSolder, B.Cu at (172.9, 147.0)
- added C52: 100nF, Capacitor_SMD:C_0603_1608Metric_Pad1.08x0.95mm_HandSolder, B.Cu at (322.8, 205.2)
- added C53: 100nF, Capacitor_SMD:C_0603_1608Metric_Pad1.08x0.95mm_HandSolder, B.Cu at (284.6, 181.2)
- added C54: 100nF, Capacitor_SMD:C_0603_1608Metric_Pad1.08x0.95mm_HandSolder, B.Cu at (227.4, 164.8)
- added C55: 100nF, Capacitor_SMD:C_0603_1608Metric_Pad1.08x0.95mm_HandSolder, B.Cu at (263.8, 144.2)
- added C56: 100nF, Capacitor_SMD:C_0603_1608Metric_Pad1.08x0.95mm_HandSolder, B.Cu at (224.0, 103.6)
- added C57: 100nF, Capacitor_SMD:C_0603_1608Metric_Pad1.08x0.95mm_HandSolder, B.Cu at (281.2, 101.4)
- added C58: 100nF, Capacitor_SMD:C_0603_1608Metric_Pad1.08x0.95mm_HandSolder, B.Cu at (342.0, 205.4)
- added C59: 100nF, Capacitor_SMD:C_0603_1608Metric_Pad1.08x0.95mm_HandSolder, B.Cu at (73.2, 204.2)
- added C6: 100nF, Capacitor_SMD:C_0603_1608Metric_Pad1.08x0.95mm_HandSolder, B.Cu at (75.0, 123.2)
- added C60: 100nF, Capacitor_SMD:C_0603_1608Metric_Pad1.08x0.95mm_HandSolder, B.Cu at (69.9, 141.6)
- added C61: 100nF, Capacitor_SMD:C_0603_1608Metric_Pad1.08x0.95mm_HandSolder, B.Cu at (48.1, 192.0)
- added C62: 100nF, Capacitor_SMD:C_0603_1608Metric_Pad1.08x0.95mm_HandSolder, B.Cu at (154.2, 145.8)
- added C63: 100nF, Capacitor_SMD:C_0603_1608Metric_Pad1.08x0.95mm_HandSolder, B.Cu at (152.2, 183.4)
- added C64: 100nF, Capacitor_SMD:C_0603_1608Metric_Pad1.08x0.95mm_HandSolder, B.Cu at (266.4, 182.2)
- added C65: 100nF, Capacitor_SMD:C_0603_1608Metric_Pad1.08x0.95mm_HandSolder, B.Cu at (209.0, 184.8)
- added C66: 100nF, Capacitor_SMD:C_0603_1608Metric_Pad1.08x0.95mm_HandSolder, B.Cu at (245.2, 145.0)
- added C67: 100nF, Capacitor_SMD:C_0603_1608Metric_Pad1.08x0.95mm_HandSolder, B.Cu at (373.6, 143.6)
- added C68: 100nF, Capacitor_SMD:C_0603_1608Metric_Pad1.08x0.95mm_HandSolder, B.Cu at (261.8, 102.2)
- added C69: 100nF, Capacitor_SMD:C_0603_1608Metric_Pad1.08x0.95mm_HandSolder, B.Cu at (341.8, 186.8)
- added C7: 100nF, Capacitor_SMD:C_0603_1608Metric_Pad1.08x0.95mm_HandSolder, B.Cu at (172.1, 166.8)
- added C70: 100nF, Capacitor_SMD:C_0603_1608Metric_Pad1.08x0.95mm_HandSolder, B.Cu at (96.3, 205.2)
- added C71: 100nF, Capacitor_SMD:C_0603_1608Metric_Pad1.08x0.95mm_HandSolder, B.Cu at (114.1, 162.4)
- added C72: 100nF, Capacitor_SMD:C_0603_1608Metric_Pad1.08x0.95mm_HandSolder, B.Cu at (68.0, 161.2)
- added C73: 100nF, Capacitor_SMD:C_0603_1608Metric_Pad1.08x0.95mm_HandSolder, B.Cu at (134.5, 163.8)
- added C74: 100nF, Capacitor_SMD:C_0603_1608Metric_Pad1.08x0.95mm_HandSolder, B.Cu at (132.6, 182.8)
- added C75: 100nF, Capacitor_SMD:C_0603_1608Metric_Pad1.08x0.95mm_HandSolder, B.Cu at (228.4, 184.6)
- added C76: 100nF, Capacitor_SMD:C_0603_1608Metric_Pad1.08x0.95mm_HandSolder, B.Cu at (206.6, 166.2)
- added C77: 100nF, Capacitor_SMD:C_0603_1608Metric_Pad1.08x0.95mm_HandSolder, B.Cu at (183.1, 208.8)
- added C8: 100nF, Capacitor_SMD:C_0603_1608Metric_Pad1.08x0.95mm_HandSolder, B.Cu at (247.2, 184.2)
- added C9: 100nF, Capacitor_SMD:C_0603_1608Metric_Pad1.08x0.95mm_HandSolder, B.Cu at (303.0, 161.2)
- added J1: PadExp Left, Connector_JST:JST_GH_SM12B-GHS-TB_1x12-1MP_P1.25mm_Horizontal, F.Cu at (372.9, 84.0)
- added J2: PadExp Right, Connector_JST:JST_GH_SM12B-GHS-TB_1x12-1MP_P1.25mm_Horizontal, F.Cu at (46.2, 84.0)
- added R1: 22R, Resistor_SMD:R_0603_1608Metric_Pad0.98x0.95mm_HandSolder, F.Cu at (265.4, 68.8)
- added R10: 22R, Resistor_SMD:R_0603_1608Metric_Pad0.98x0.95mm_HandSolder, F.Cu at (269.8, 78.8)
- added R11: 22R, Resistor_SMD:R_0603_1608Metric_Pad0.98x0.95mm_HandSolder, F.Cu at (274.1, 68.8)
- added R12: 22R, Resistor_SMD:R_0603_1608Metric_Pad0.98x0.95mm_HandSolder, F.Cu at (274.1, 71.3)
- added R13: 22R, Resistor_SMD:R_0603_1608Metric_Pad0.98x0.95mm_HandSolder, F.Cu at (274.1, 73.8)
- added R14: 22R, Resistor_SMD:R_0603_1608Metric_Pad0.98x0.95mm_HandSolder, F.Cu at (274.1, 76.3)
- added R15: 22R, Resistor_SMD:R_0603_1608Metric_Pad0.98x0.95mm_HandSolder, F.Cu at (274.1, 78.8)
- added R16: 22R, Resistor_SMD:R_0603_1608Metric_Pad0.98x0.95mm_HandSolder, F.Cu at (278.5, 68.8)
- added R17: 22R, Resistor_SMD:R_0603_1608Metric_Pad0.98x0.95mm_HandSolder, F.Cu at (278.5, 71.3)
- added R18: 22R, Resistor_SMD:R_0603_1608Metric_Pad0.98x0.95mm_HandSolder, F.Cu at (278.5, 73.8)
- added R19: 22R, Resistor_SMD:R_0603_1608Metric_Pad0.98x0.95mm_HandSolder, F.Cu at (278.5, 76.3)
- added R2: 22R, Resistor_SMD:R_0603_1608Metric_Pad0.98x0.95mm_HandSolder, F.Cu at (265.4, 71.3)
- added R20: 22R, Resistor_SMD:R_0603_1608Metric_Pad0.98x0.95mm_HandSolder, F.Cu at (278.5, 78.8)
- added R21: 22R, Resistor_SMD:R_0603_1608Metric_Pad0.98x0.95mm_HandSolder, B.Cu at (289.0, 97.0)
- added R3: 22R, Resistor_SMD:R_0603_1608Metric_Pad0.98x0.95mm_HandSolder, F.Cu at (265.4, 73.8)
- added R4: 22R, Resistor_SMD:R_0603_1608Metric_Pad0.98x0.95mm_HandSolder, F.Cu at (265.4, 76.3)
- added R5: 22R, Resistor_SMD:R_0603_1608Metric_Pad0.98x0.95mm_HandSolder, F.Cu at (265.4, 78.8)
- added R6: 22R, Resistor_SMD:R_0603_1608Metric_Pad0.98x0.95mm_HandSolder, F.Cu at (269.8, 68.8)
- added R7: 22R, Resistor_SMD:R_0603_1608Metric_Pad0.98x0.95mm_HandSolder, F.Cu at (269.8, 71.3)
- added R8: 22R, Resistor_SMD:R_0603_1608Metric_Pad0.98x0.95mm_HandSolder, F.Cu at (269.8, 73.8)
- added R9: 22R, Resistor_SMD:R_0603_1608Metric_Pad0.98x0.95mm_HandSolder, F.Cu at (269.8, 76.3)
- added U1: BlackPill_STLINK, Modules:BlackPill_STLINK, F.Cu at (330.0, 81.2)
- D1, D10, D100, D101, D102, D103, D104, D105, D106, D107, D108, D109, D11, D110, D111, D112, D113, D114, D115, D116, D117, D118, D119, D12, D120, D121, D122, D123, D124, D125, D126, D127, D128, D129, D13, D130, D131, D132, D133, D134, D135, D136, D137, D138, D139, D14, D140, D141, D142, D143, D144, D145, D146, D147, D148, D149, D15, D150, D151, D152, D16, D17, D18, D19, D2, D20, D21, D22, D23, D24, D25, D26, D27, D28, D29, D3, D30, D31, D32, D33, D34, D35, D36, D37, D38, D39, D4, D40, D41, D42, D43, D44, D45, D46, D47, D48, D49, D5, D50, D51, D52, D53, D54, D55, D56, D57, D58, D59, D6, D60, D61, D62, D63, D64, D65, D66, D67, D68, D69, D7, D70, D71, D72, D73, D74, D75, D76, D77, D78, D79, D8, D80, D81, D82, D83, D84, D85, D86, D87, D88, D89, D9, D90, D91, D92, D93, D94, D95, D96, D97, D98, D99: moved to B.Cu
- SW1, SW10, SW11, SW12, SW13, SW14, SW15, SW16, SW17, SW18, SW19, SW2, SW20, SW21, SW22, SW23, SW24, SW25, SW26, SW27, SW28, SW29, SW3, SW30, SW31, SW32, SW33, SW34, SW35, SW36, SW37, SW38, SW39, SW4, SW40, SW41, SW42, SW43, SW44, SW45, SW46, SW47, SW48, SW49, SW5, SW50, SW51, SW52, SW53, SW54, SW55, SW56, SW57, SW58, SW59, SW6, SW60, SW61, SW62, SW63, SW64, SW65, SW66, SW67, SW68, SW69, SW7, SW70, SW71, SW72, SW8, SW9: footprint Button_Switch_Keyboard:SW_MX -> Button_Switch_Keyboard:Kailh_socket_MX_LED
- moved D136 669.1 mm to (48.2, 188.1), turned to 180 degrees
- moved D137 649.0 mm to (72.5, 200.0), turned to 180 degrees
- moved D138 624.7 mm to (96.9, 200.7), turned to -3 degrees
- moved D61 622.1 mm to (39.0, 186.6), turned to 180 degrees
- moved D122 617.6 mm to (72.5, 176.6), turned to 180 degrees
- moved D78 609.0 mm to (50.8, 113.4), turned to 180 degrees
- moved D62 603.0 mm to (62.2, 197.6), turned to 180 degrees
- moved D139 600.2 mm to (121.7, 201.6), turned to -3 degrees
- moved D107 599.1 mm to (67.7, 157.5), turned to 180 degrees
- moved D124 597.5 mm to (114.2, 178.2), turned to -3 degrees
- moved D76 595.7 mm to (75.1, 94.5), turned to 180 degrees
- moved D123 590.1 mm to (95.2, 177.2), turned to -3 degrees
- moved D47 589.5 mm to (65.2, 176.0), turned to 180 degrees
- moved D79 586.0 mm to (74.9, 119.4), turned to 180 degrees
- moved D93 584.2 mm to (70.1, 138.5), turned to 180 degrees
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Connections:
- D147 pad 1: Net-(D147-DOUT) -> /ledsplate/led_out
- D148 pad 3: Net-(D147-DOUT) -> Net-(D148-DIN)
- D149 pad 1: Net-(D149-DOUT) -> Net-(D148-DIN)
- D149 pad 3: Net-(D148-DOUT) -> Net-(D149-DIN)
- D150 pad 1: Net-(D150-DOUT) -> Net-(D149-DIN)
- D150 pad 3: Net-(D149-DOUT) -> Net-(D150-DIN)
- D151 pad 1: Net-(D151-DOUT) -> Net-(D150-DIN)
- D151 pad 3: Net-(D150-DOUT) -> Net-(D151-DIN)
- D152 pad 1: /ledsplate/led_out -> Net-(D151-DIN)
- D152 pad 3: Net-(D151-DOUT) -> Net-(D152-DIN)
- D76 pad 3: Net-(D76-DIN) -> Net-(D148-DOUT)

Commit message: Continue routing
Parts:
- moved R21 38.6 mm to (327.5, 95.0)
- moved D76 19.0 mm to (94.1, 94.5), turned to 0 degrees
- moved D77 19.0 mm to (75.1, 94.5), turned to 0 degrees
- moved D9 15.2 mm to (165.1, 123.2), turned to -93 degrees
- moved D66 10.3 mm to (180.8, 203.2), turned to -90 degrees
- moved D24 10.0 mm to (197.5, 143.2)
- moved C48 8.04 mm to (67.2, 175.8)
- moved C59 7.90 mm to (67.2, 199.0)
- moved C25 7.87 mm to (153.8, 201.5)
- moved C7 7.75 mm to (167.0, 161.0)
- moved C36 7.65 mm to (116.5, 200.5)
- moved C26 7.51 mm to (109.0, 177.0)
- moved C27 7.51 mm to (169.0, 123.0)
- moved C54 7.50 mm to (221.2, 160.5)
- moved C39 7.50 mm to (131.0, 121.0)
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Routing:
- net Net-(D148-DOUT): track 0.00 -> 112.4 mm
- net +5V: track 0.00 -> 64.1 mm
- net Net-(D82-DOUT): track 0.00 -> 48.6 mm
- net Net-(D77-DOUT): track 0.00 -> 47.0 mm
- net Net-(D85-DOUT): track 0.00 -> 32.1 mm
- net Net-(D84-DOUT): track 0.00 -> 29.4 mm
- net Net-(D107-DOUT): track 0.00 -> 25.5 mm
- net Net-(D78-DOUT): track 0.00 -> 24.7 mm
- net Net-(D93-DOUT): track 0.00 -> 24.1 mm
- net Net-(D79-DOUT): track 0.00 -> 20.4 mm
- net Net-(D122-DOUT): track 0.00 -> 19.7 mm
- net Net-(D76-DOUT): track 0.00 -> 16.4 mm
- net Net-(D97-DOUT): track 0.00 -> 16.2 mm
- net Net-(D81-DOUT): track 0.00 -> 16.2 mm
- net Net-(D96-DOUT): track 0.00 -> 16.2 mm
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
Commit message: Continue routing
Parts:
- moved D145 38.1 mm to (322.8, 201.8)
- moved D147 38.1 mm to (360.9, 201.8)
- moved C41 8.89 mm to (277.2, 198.8)
- moved C8 8.06 mm to (241.5, 178.5)
- moved D72 7.89 mm to (351.8, 200.5), turned to -90 degrees
- moved C19 7.88 mm to (216.0, 201.2)
- moved C31 7.71 mm to (316.5, 155.8), turned to -177 degrees
- moved C11 7.69 mm to (342.2, 145.2)
- moved C75 7.63 mm to (222.5, 179.8)
- moved C43 7.58 mm to (240.5, 159.5)
- moved C22 7.54 mm to (315.5, 136.5)
- moved C64 7.54 mm to (260.5, 177.5)
- moved C46 7.34 mm to (257.5, 120.5)
- moved C20 7.28 mm to (278.5, 157.8)
- moved C66 7.26 mm to (239.5, 140.5)
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Connections:
- D108 pad 2: unconnected-(D108-VSS-Pad2) -> GND
- D109 pad 2: unconnected-(D109-VSS-Pad2) -> GND
- D110 pad 2: unconnected-(D110-VSS-Pad2) -> GND
- D111 pad 2: unconnected-(D111-VSS-Pad2) -> GND
- D96 pad 2: unconnected-(D96-VSS-Pad2) -> GND
- D97 pad 2: unconnected-(D97-VSS-Pad2) -> GND
- D98 pad 2: unconnected-(D98-VSS-Pad2) -> GND
- D99 pad 2: unconnected-(D99-VSS-Pad2) -> GND
Routing:
- net Net-(D106-DOUT): track 0.00 -> 381.5 mm
- net Net-(D92-DOUT): track 0.00 -> 356.1 mm
- net Net-(D121-DOUT): track 0.00 -> 214.0 mm
- net +5V: track 64.1 -> 0.00 mm
- net Net-(D105-DOUT): track 0.00 -> 53.1 mm
- net Net-(D144-DOUT): track 0.00 -> 39.7 mm
- net Net-(D142-DOUT): track 0.00 -> 35.9 mm
- net Net-(D127-DOUT): track 0.00 -> 34.4 mm
- net Net-(D133-DOUT): track 0.00 -> 34.3 mm
- net Net-(D120-DOUT): track 0.00 -> 32.5 mm
- net Net-(D141-DOUT): track 0.00 -> 31.9 mm
- net Net-(D98-DOUT): track 0.00 -> 31.6 mm
- net Net-(D82-DOUT): track 48.6 -> 17.8 mm
- net Net-(D134-DOUT): track 0.00 -> 30.3 mm
- net Net-(D91-DOUT): track 0.00 -> 30.1 mm
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
Commit message: Complete led wire
Parts:
- added R22: 22R, Resistor_SMD:R_0603_1608Metric_Pad0.98x0.95mm_HandSolder, B.Cu at (365.5, 202.0)
Connections:
- net /ledsplate/led_in renamed /led_w1_in
- D147 pad 1: /ledsplate/led_out -> /led_w1_out
Routing:
- net Net-(D135-DOUT): track 0.00 -> 397.6 mm
- net Net-(D121-DOUT): track 214.0 -> 398.4 mm
- net Net-(D136-DOUT): track 0.00 -> 30.1 mm
- net Net-(D146-DOUT): track 0.00 -> 16.5 mm
- net Net-(D145-DOUT): track 0.00 -> 16.5 mm
- net Net-(D97-DOUT): track 16.2 -> 32.4 mm
- net Net-(D126-DOUT): track 16.2 -> 0.00 mm
- net Net-(D112-DOUT): track 25.4 -> 33.3 mm
- net /led_w1_out: track 0.00 -> 2.97 mm
- net Net-(D127-DOUT): track 34.4 -> 35.4 mm
- net Net-(D122-DOUT): track 19.7 -> 20.3 mm
- net Net-(D129-DOUT): track 16.0 -> 16.6 mm
- net Net-(D130-DOUT): track 16.0 -> 16.6 mm

Commit message: Complete led wire
Parts:
- added R23: 22R, Resistor_SMD:R_0603_1608Metric_Pad0.98x0.95mm_HandSolder, F.Cu at (278.5, 81.8)
- added R23: 22R, Resistor_SMD:R_0603_1608Metric_Pad0.98x0.95mm_HandSolder, F.Cu at (356.4, 95.5)
- added R24: 22R, Resistor_SMD:R_0603_1608Metric_Pad0.98x0.95mm_HandSolder, F.Cu at (347.8, 97.0)
- added R24: 22R, Resistor_SMD:R_0603_1608Metric_Pad0.98x0.95mm_HandSolder, F.Cu at (356.4, 98.0)
Connections:
- D10 pad 2: Net-(D1-A) -> Net-(D10-A)
- D11 pad 2: Net-(D1-A) -> Net-(D10-A)
- D12 pad 2: Net-(D1-A) -> Net-(D10-A)
- D13 pad 2: Net-(D1-A) -> Net-(D10-A)
- D14 pad 2: Net-(D1-A) -> Net-(D10-A)
- D15 pad 2: Net-(D1-A) -> Net-(D10-A)
- D16 pad 2: Net-(D16-A) -> Net-(D10-A)
- D17 pad 2: Net-(D16-A) -> Net-(D10-A)
- D18 pad 2: Net-(D16-A) -> Net-(D18-A)
- D19 pad 2: Net-(D16-A) -> Net-(D18-A)
- D20 pad 2: Net-(D16-A) -> Net-(D18-A)
- D21 pad 2: Net-(D16-A) -> Net-(D18-A)
- D22 pad 2: Net-(D16-A) -> Net-(D18-A)
- D23 pad 2: Net-(D16-A) -> Net-(D18-A)
- D24 pad 2: Net-(D16-A) -> Net-(D18-A)
- D25 pad 2: Net-(D16-A) -> Net-(D18-A)
- D26 pad 2: Net-(D16-A) -> Net-(D18-A)
- D27 pad 2: Net-(D16-A) -> Net-(D18-A)
- D28 pad 2: Net-(D16-A) -> Net-(D18-A)
- D29 pad 2: Net-(D16-A) -> Net-(D18-A)
- D3 pad 2: Net-(D1-A) -> Net-(D10-A)
- D30 pad 2: Net-(D16-A) -> Net-(D18-A)
- D31 pad 2: Net-(D31-A) -> Net-(D18-A)
- D32 pad 2: Net-(D31-A) -> Net-(D32-A)
- D33 pad 2: Net-(D31-A) -> Net-(D32-A)
- D34 pad 2: Net-(D31-A) -> Net-(D32-A)
- D35 pad 2: Net-(D31-A) -> Net-(D32-A)
- D36 pad 2: Net-(D31-A) -> Net-(D32-A)
- D37 pad 2: Net-(D31-A) -> Net-(D32-A)
- D38 pad 2: Net-(D31-A) -> Net-(D32-A)
- D39 pad 2: Net-(D31-A) -> Net-(D32-A)
- D4 pad 2: Net-(D1-A) -> Net-(D10-A)
- D40 pad 2: Net-(D31-A) -> Net-(D32-A)
- D41 pad 2: Net-(D31-A) -> Net-(D32-A)
- D42 pad 2: Net-(D31-A) -> Net-(D32-A)
- D43 pad 2: Net-(D31-A) -> Net-(D32-A)
- D44 pad 2: Net-(D31-A) -> Net-(D32-A)
- D45 pad 2: Net-(D31-A) -> Net-(D32-A)
- D46 pad 2: Net-(D46-A) -> Net-(D32-A)
- D47 pad 2: Net-(D46-A) -> Net-(D47-A)
- D48 pad 2: Net-(D46-A) -> Net-(D47-A)
- D49 pad 2: Net-(D46-A) -> Net-(D47-A)
- D5 pad 2: Net-(D1-A) -> Net-(D10-A)
- D50 pad 2: Net-(D46-A) -> Net-(D47-A)
- D51 pad 2: Net-(D46-A) -> Net-(D47-A)
- D52 pad 2: Net-(D46-A) -> Net-(D47-A)
- D53 pad 2: Net-(D46-A) -> Net-(D47-A)
- D54 pad 2: Net-(D46-A) -> Net-(D47-A)
- D55 pad 2: Net-(D46-A) -> Net-(D47-A)
- D56 pad 2: Net-(D46-A) -> Net-(D47-A)
- D57 pad 2: Net-(D46-A) -> Net-(D47-A)
- D58 pad 2: Net-(D46-A) -> Net-(D47-A)
- D59 pad 2: Net-(D46-A) -> Net-(D47-A)
- D6 pad 2: Net-(D1-A) -> Net-(D10-A)
- D60 pad 2: Net-(D46-A) -> Net-(D47-A)
- D7 pad 2: Net-(D1-A) -> Net-(D10-A)
- D70 pad 2: Net-(D61-A) -> Net-(D70-A)
- D71 pad 2: Net-(D61-A) -> Net-(D70-A)
- D72 pad 2: Net-(D61-A) -> Net-(D70-A)
- D8 pad 2: Net-(D1-A) -> Net-(D10-A)
- D9 pad 2: Net-(D1-A) -> Net-(D10-A)
- J1 pad 10: /cl17 -> /cl18
- J1 pad 11: /cl18 -> /cl19
- J1 pad 12: /cl19 -> /cl20
- J1 pad 8: /cl15 -> /cl16
- J1 pad 9: /cl16 -> /cl17
- J2 pad 10: /cl17 -> /cl18
- J2 pad 11: /cl18 -> /cl19
- J2 pad 12: /cl19 -> /cl20
- J2 pad 8: /cl15 -> /cl16
- J2 pad 9: /cl16 -> /cl17
- R11 pad 1: unconnected-(R11-Pad1) -> /cl10
- R16 pad 2: Net-(D1-A) -> Net-(D10-A)
- R17 pad 2: Net-(D16-A) -> Net-(D18-A)
- R18 pad 2: Net-(D31-A) -> Net-(D32-A)
- R19 pad 2: Net-(D46-A) -> Net-(D47-A)
- R6 pad 1: unconnected-(R6-Pad1) -> /cl5
- SW1 pad 1: Net-(R1-Pad2) -> Net-(R2-Pad2)
- SW10 pad 1: Net-(R10-Pad2) -> Net-(R8-Pad2)
- SW11 pad 1: Net-(R11-Pad2) -> Net-(R9-Pad2)
- SW12 pad 1: Net-(R12-Pad2) -> Net-(R10-Pad2)
- SW13 pad 1: Net-(R13-Pad2) -> unconnected-(SW13-Pad1)
- SW14 pad 1: Net-(R14-Pad2) -> Net-(R12-Pad2)
- SW15 pad 1: Net-(R15-Pad2) -> Net-(R13-Pad2)
- SW16 pad 1: Net-(R1-Pad2) -> Net-(R14-Pad2)
- SW17 pad 1: Net-(R2-Pad2) -> Net-(R15-Pad2)
- SW18 pad 1: Net-(R3-Pad2) -> Net-(R2-Pad2)
- SW19 pad 1: Net-(R4-Pad2) -> Net-(R3-Pad2)
- SW2 pad 1: Net-(R2-Pad2) -> Net-(R3-Pad2)
- SW20 pad 1: Net-(R5-Pad2) -> Net-(R4-Pad2)
- SW21 pad 1: Net-(R6-Pad2) -> Net-(R5-Pad2)
- SW22 pad 1: Net-(R7-Pad2) -> Net-(R6-Pad2)
- SW23 pad 1: Net-(R8-Pad2) -> Net-(R7-Pad2)
- SW24 pad 1: Net-(R9-Pad2) -> Net-(R8-Pad2)
- SW25 pad 1: Net-(R10-Pad2) -> Net-(R9-Pad2)
- SW26 pad 1: Net-(R11-Pad2) -> Net-(R10-Pad2)
- SW27 pad 1: Net-(R12-Pad2) -> Net-(R11-Pad2)
- SW28 pad 1: Net-(R13-Pad2) -> Net-(R12-Pad2)
- SW29 pad 1: Net-(R14-Pad2) -> Net-(R13-Pad2)
- SW3 pad 1: Net-(R3-Pad2) -> Net-(R1-Pad2)
- SW30 pad 1: Net-(R15-Pad2) -> Net-(R14-Pad2)
- SW31 pad 1: Net-(R1-Pad2) -> Net-(R24-Pad2)
- SW4 pad 1: Net-(R4-Pad2) -> Net-(R2-Pad2)
- SW46 pad 1: Net-(R1-Pad2) -> Net-(R24-Pad2)
- SW5 pad 1: Net-(R5-Pad2) -> Net-(R3-Pad2)
- SW59 pad 1: Net-(R14-Pad2) -> Net-(R15-Pad2)
- SW6 pad 1: Net-(R6-Pad2) -> Net-(R4-Pad2)
- SW60 pad 1: Net-(R15-Pad2) -> Net-(R24-Pad2)
- SW65 pad 1: Net-(R5-Pad2) -> Net-(R6-Pad2)
- SW66 pad 1: Net-(R6-Pad2) -> Net-(R7-Pad2)
- SW67 pad 1: Net-(R7-Pad2) -> Net-(R8-Pad2)
- SW68 pad 1: Net-(R8-Pad2) -> Net-(R10-Pad2)
- SW69 pad 1: Net-(R9-Pad2) -> Net-(R11-Pad2)
- SW7 pad 1: Net-(R7-Pad2) -> Net-(R5-Pad2)
- SW70 pad 1: Net-(R10-Pad2) -> Net-(R14-Pad2)
- SW71 pad 1: Net-(R11-Pad2) -> Net-(R15-Pad2)
- SW72 pad 1: Net-(R12-Pad2) -> Net-(R24-Pad2)
- SW8 pad 1: Net-(R8-Pad2) -> Net-(R6-Pad2)
- SW9 pad 1: Net-(R9-Pad2) -> Net-(R7-Pad2)
- U1 pad 10: /cl19 -> /cl20
- U1 pad 31: unconnected-(U1-PA5-Pad31) -> /r-1
- U1 pad 6: unconnected-(U1-PA9-Pad6) -> /cl16
- U1 pad 7: /cl16 -> /cl17
- U1 pad 8: /cl17 -> /cl18
- U1 pad 9: /cl18 -> /cl19
Routing:
- net Net-(D10-A): track 0.00 -> 317.7 mm, vias 0 -> 2
- net Net-(R3-Pad2): track 0.00 -> 126.1 mm, vias 0 -> 6
- net Net-(R2-Pad2): track 0.00 -> 125.0 mm, vias 0 -> 6
- net Net-(R7-Pad2): track 0.00 -> 104.2 mm, vias 0 -> 5
- net Net-(R11-Pad2): track 0.00 -> 103.5 mm, vias 0 -> 5
- net Net-(R4-Pad2): track 0.00 -> 98.4 mm, vias 0 -> 5
- net Net-(R8-Pad2): track 0.00 -> 98.0 mm, vias 0 -> 5
- net Net-(R6-Pad2): track 0.00 -> 96.8 mm, vias 0 -> 5
- net Net-(R10-Pad2): track 0.00 -> 96.8 mm, vias 0 -> 5
- net Net-(R15-Pad2): track 0.00 -> 94.6 mm, vias 0 -> 4
- net Net-(R14-Pad2): track 0.00 -> 92.0 mm, vias 0 -> 4
- net Net-(R24-Pad2): track 0.00 -> 82.6 mm, vias 0 -> 4
- net Net-(R1-Pad2): track 0.00 -> 76.3 mm, vias 0 -> 2
- net Net-(R9-Pad2): track 0.00 -> 70.3 mm, vias 0 -> 4
- net Net-(R5-Pad2): track 0.00 -> 69.8 mm, vias 0 -> 4
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
Commit message: Continue routing
Parts:
- removed D73, D74, D75: 1N4448W, Diode_SMD:D_SOD-123
- moved C5 1.06 mm to (45.5, 112.5), turned to 180 degrees
Connections:
- D70 pad 2: Net-(D70-A) -> Net-(D61-A)
- D71 pad 2: Net-(D70-A) -> Net-(D61-A)
- D72 pad 2: Net-(D70-A) -> Net-(D61-A)
Routing:
- net GND: track 0.00 -> 2158.4 mm, vias 0 -> 154
- net +5V: track 0.00 -> 1556.5 mm, vias 0 -> 118
- net Net-(D61-A): track 0.00 -> 336.7 mm
- net Net-(D18-A): track 0.00 -> 326.9 mm
- net Net-(D47-A): track 0.00 -> 248.0 mm
- net Net-(D32-A): track 0.00 -> 168.0 mm
- net Net-(D126-DOUT): track 0.00 -> 16.8 mm
- net Net-(D97-DOUT): track 32.4 -> 16.2 mm
- net Net-(D46-K): track 0.00 -> 6.06 mm
- net Net-(D47-K): track 0.00 -> 6.01 mm
- net Net-(D53-K): track 0.00 -> 5.99 mm
- net Net-(D32-K): track 0.00 -> 5.98 mm
- net Net-(D25-K): track 0.00 -> 5.95 mm
- net Net-(D62-K): track 0.00 -> 5.93 mm
- net Net-(D61-K): track 0.00 -> 5.92 mm
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