File: isokey/isokey.kicad_pcb (KiCad board)
At the start: 2 copper layers, 363.8 x 153.8 mm, 392 parts, among them J1 PadExp Left, J2 PadExp Right, Q1 BSS138, SW1 Cherry, SW10 Cherry, SW11 Cherry, SW12 Cherry, SW13 Cherry, SW14 Cherry, SW15 Cherry, SW16 Cherry, SW17 Cherry, SW18 Cherry, SW19 Cherry, SW2 Cherry, SW20 Cherry, SW21 Cherry, SW22 Cherry, SW23 Cherry, SW24 Cherry, SW25 Cherry, SW26 Cherry, SW27 Cherry, SW28 Cherry, SW29 Cherry, SW3 Cherry, SW30 Cherry, SW31 Cherry, SW32 Cherry, SW33 Cherry, SW34 Cherry, SW35 Cherry, SW36 Cherry, SW37 Cherry, SW38 Cherry, SW39 Cherry, SW4 Cherry, SW40 Cherry, SW41 Cherry, SW42 Cherry, SW43 Cherry, SW44 Cherry, SW45 Cherry, SW46 Cherry, SW47 Cherry, SW48 Cherry, SW49 Cherry, SW5 Cherry, SW50 Cherry, SW51 Cherry, SW52 Cherry, SW53 Cherry, SW54 Cherry, SW55 Cherry, SW56 Cherry, SW57 Cherry, SW58 Cherry, SW59 Cherry, SW6 Cherry, SW60 Cherry, SW61 Cherry, SW62 Cherry, SW63 Cherry, SW64 Cherry, SW65 Cherry, SW67 Cherry, SW68 Cherry, SW69 Cherry, SW7 Cherry, SW70 Cherry, SW71 Cherry, SW72 Cherry, SW73 RotaryEncoder_Switch, SW74 RotaryEncoder_Switch, SW8 Cherry, SW9 Cherry, U1 BlackPill_STLINK, U4 TLV73318PDBV

Commit message: WIP
Parts:
- removed C34, C45, C56, C57, C68, C77: 100nF, Capacitor_SMD:C_0603_1608Metric_Pad1.08x0.95mm_HandSolder
- removed D148, D149, D150, D151, D152: SK6812MINI, LED_SMD:LED_SK6812MINI_PLCC4_3.5x3.5mm_P1.75mm
- added H1: StabilizerHoles, Button_Switch_Keyboard:Stabilizer_MX_2u, F.Cu at (349.9, 112.6)
- added H2: StabilizerHoles, Button_Switch_Keyboard:Stabilizer_MX_2u, F.Cu at (346.6, 141.1)
- added H3: StabilizerHoles, Button_Switch_Keyboard:Stabilizer_MX_2u, F.Cu at (222.6, 197.0)
- added H4: StabilizerHoles, Button_Switch_Keyboard:Stabilizer_MX_2u, F.Cu at (157.7, 197.6)
- C78, C79, C80, C81, C82, C83, C85, Q1, R26, R35, R59, R60, R61: moved to B.Cu
- R36: value NP -> 10k; moved to B.Cu
- U2: value ~ -> LP5569
- moved D155 204.7 mm to (392.9, 110.6), turned to 90 degrees
- moved D154 201.6 mm to (382.0, 121.4), turned to 180 degrees
- moved D156 189.2 mm to (382.2, 99.5), turned to 180 degrees
- moved D153 187.9 mm to (371.1, 110.4), turned to 90 degrees
- moved C78 179.7 mm to (201.4, 198.3), turned to 90 degrees
- moved D164 175.3 mm to (190.0, 211.0), turned to 180 degrees
- moved C81 168.3 mm to (204.2, 202.8), turned to -135 degrees
- moved R36 164.7 mm to (203.1, 198.3), turned to 90 degrees
- moved D160 160.4 mm to (181.0, 207.8), turned to 135 degrees
- moved U3 157.6 mm to (201.5, 201.7), turned to -135 degrees
- moved D162 152.7 mm to (199.0, 207.8), turned to -135 degrees
- moved C85 145.7 mm to (199.5, 198.3), turned to 90 degrees
- moved D167 145.4 mm to (199.0, 189.8), turned to 135 degrees
- moved D161 140.2 mm to (181.0, 189.8), turned to 45 degrees
- moved D166 129.2 mm to (190.0, 169.6), turned to 90 degrees
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Connections:
- D76 pad 3: Net-(D148-DOUT) -> Net-(D76-DIN)
- R21 pad 2: Net-(D152-DIN) -> Net-(D76-DIN)
- R26 pad 1: +3.3V -> +1V8
- R35 pad 1: +3.3V -> +1V8
- R35 pad 2: /Led_EN -> Net-(U2-EN/PWM)
- R36 pad 1: /Led_EN -> +1V8
- R36 pad 2: GND -> Net-(U3-EN/PWM)
- SW15 pad 1: /sw0_c -> /cl12
- SW29 pad 1: /sw0_c -> /cl12
- SW43 pad 1: /sw0_c -> /cl12
- SW58 pad 1: /sw0_c -> /cl12
- SW73 pad S1: /sw0_c -> /cl12
- SW74 pad S1: /sw1_c -> /cl6
- U2 pad 11: Net-(D73-K) -> Net-(D157-K)
- U2 pad 12: Net-(D74-K) -> Net-(D158-K)
- U2 pad 13: Net-(D75-K) -> Net-(D73-K)
- U2 pad 14: Net-(D153-K) -> Net-(D74-K)
- U2 pad 15: Net-(D154-K) -> Net-(D75-K)
- U2 pad 16: Net-(D155-K) -> Net-(D153-K)
- U2 pad 17: Net-(D156-K) -> Net-(D154-K)
- U2 pad 18: Net-(D157-K) -> Net-(D155-K)
- U2 pad 19: Net-(D158-K) -> Net-(D156-K)
- U2 pad 20: unconnected-(U2-ADDR-Pad20) -> GND
- U2 pad 5: /Led_EN -> Net-(U2-EN/PWM)
- U3 pad 14: Net-(D164-K) -> Net-(D163-K)
- U3 pad 15: Net-(D163-K) -> Net-(D159-K)
- U3 pad 16: Net-(D162-K) -> Net-(D161-K)
- U3 pad 17: Net-(D161-K) -> Net-(D160-K)
- U3 pad 18: Net-(D160-K) -> Net-(D164-K)
- U3 pad 19: Net-(D159-K) -> Net-(D162-K)
- U3 pad 20: unconnected-(U3-ADDR-Pad20) -> +5V
- U3 pad 5: /Led_EN -> Net-(U3-EN/PWM)
Routing:
- net (no net): track 308.8 -> 0.00 mm
- net /ENC1B: track 104.8 -> 409.1 mm, vias 1 -> 2
- net /cl6: track 0.00 -> 265.0 mm, vias 0 -> 6
- net /cl17: track 0.00 -> 262.0 mm
- net /port_id: track 0.00 -> 259.0 mm
- net /led_SCL: track 0.00 -> 220.8 mm, vias 0 -> 5
- net /led_SDA: track 0.00 -> 206.6 mm, vias 0 -> 5
- net /cl9: track 0.00 -> 205.5 mm
- net +3.3V: track 88.5 -> 275.5 mm, vias 1 -> 5
- net +5V: track 2093.2 -> 2265.6 mm, vias 151 -> 162
- net /sw1_c: track 170.2 -> 0.00 mm, vias 4 -> 0
- net /c15: track 0.00 -> 169.3 mm, vias 0 -> 1
- net /cl16: track 0.00 -> 169.1 mm, vias 0 -> 1
- net /c14: track 0.00 -> 168.4 mm, vias 0 -> 1
- net /ENC1A: track 108.4 -> 265.8 mm, vias 1 -> 2
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
Commit message: Complete routing
Parts:
- R25, R27, U4: moved to B.Cu
- moved C84 67.4 mm to (357.4, 88.3)
- moved U4 63.0 mm to (356.5, 90.9)
- moved C87 62.4 mm to (359.6, 90.2), turned to 90 degrees
- moved R28 62.0 mm to (353.4, 88.3)
- moved C86 56.4 mm to (355.3, 90.3), turned to 90 degrees
- moved R25 28.9 mm to (325.8, 73.1), turned to -90 degrees
- moved R27 28.1 mm to (324.1, 73.1), turned to -90 degrees
- moved R60 27.8 mm to (301.6, 92.3), turned to 0 degrees
- moved Q1 27.6 mm to (301.6, 89.3), turned to -90 degrees
- moved R59 27.4 mm to (301.6, 86.3), turned to 0 degrees
- moved R61 27.2 mm to (301.7, 84.6), turned to 180 degrees
- moved R21 26.0 mm to (301.6, 94.0), turned to 0 degrees
- moved R26 24.6 mm to (311.7, 87.8), turned to -90 degrees
- moved C79 22.4 mm to (307.4, 86.9), turned to 180 degrees
- moved R35 21.2 mm to (310.0, 87.8), turned to -90 degrees
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Connections:
- J1 pad 10: /c14 -> /cl14
- J1 pad 11: /c15 -> /cl15
- J2 pad 10: /c14 -> /cl14
- J2 pad 11: /c15 -> /cl15
- R1 pad 1: /cl17 -> /cl3
- R10 pad 1: /cl8 -> /cl11
- R11 pad 1: /cl7 -> /cl10
- R12 pad 1: /r-1 -> /cl9
- R13 pad 1: /r4 -> /cl8
- R14 pad 1: /r3 -> /cl7
- R15 pad 1: /r2 -> /cl6
- R16 pad 1: /r1 -> /cl5
- R17 pad 1: /r0 -> /cl4
- R18 pad 1: /cl6 -> /cl14
- R19 pad 1: /cl5 -> /cl17
- R2 pad 1: /cl16 -> /cl2
- R20 pad 1: /cl4 -> /cl0
- R23 pad 1: /cl3 -> /cl15
- R24 pad 1: /cl2 -> /cl16
- R3 pad 1: /cl15 -> /cl1
- R37 pad 1: /cl1 -> /cl13
- R38 pad 1: /cl0 -> /cl12
- R4 pad 1: /cl14 -> /r-1
- R5 pad 1: /cl13 -> /r4
- R6 pad 1: /cl12 -> /r3
- R7 pad 1: /cl11 -> /r2
- R8 pad 1: /cl10 -> /r1
- R9 pad 1: /cl9 -> /r0
- U2 pad 11: Net-(D157-K) -> Net-(D155-K)
- U2 pad 12: Net-(D158-K) -> Net-(D154-K)
- U2 pad 13: Net-(D73-K) -> Net-(D153-K)
- U2 pad 14: Net-(D74-K) -> Net-(D156-K)
- U2 pad 15: Net-(D75-K) -> Net-(D157-K)
- U2 pad 16: Net-(D153-K) -> Net-(D158-K)
- U2 pad 17: Net-(D154-K) -> Net-(D73-K)
- U2 pad 18: Net-(D155-K) -> Net-(D74-K)
- U2 pad 19: Net-(D156-K) -> Net-(D75-K)
Routing:
- net +5V: track 2265.6 -> 2728.4 mm, vias 162 -> 181
- net /cl15: track 83.0 -> 541.8 mm, vias 4 -> 12
- net /cl14: track 98.2 -> 549.8 mm, vias 4 -> 9
- net GND: track 3307.6 -> 3699.3 mm, vias 290 -> 314
- net +3.3V: track 275.5 -> 522.5 mm, vias 5 -> 14
- net /r-1: track 183.8 -> 417.9 mm, vias 3 -> 6
- net /cl0: track 289.3 -> 496.6 mm, vias 6 -> 9
- net /cl16: track 169.1 -> 375.3 mm, vias 1 -> 2
- net +1V8: track 112.9 -> 308.7 mm, vias 3 -> 5
- net /c15: track 169.3 -> 0.00 mm, vias 1 -> 0
- net /c14: track 168.4 -> 0.00 mm, vias 1 -> 0
- net /led_SDA: track 206.6 -> 364.7 mm, vias 5 -> 8
- net /led_SCL: track 220.8 -> 374.7 mm, vias 5 -> 8
- net /Led_CLK: track 97.0 -> 216.7 mm, vias 0 -> 2
- net /Led_INT: track 100.7 -> 219.1 mm, vias 1 -> 2
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Other:
- outline, holes or cut-outs redrawn

Commit message: Move left con
Parts:
- moved C95 7.07 mm to (51.5, 75.7)
- moved J1 3.74 mm to (45.0, 83.5)
- moved R63 3.74 mm to (53.0, 92.2)
Routing:
- net GND: track 3699.3 -> 3689.7 mm, vias 314 -> 313
- net +5V: track 2728.4 -> 2720.8 mm, vias 181 -> 182
- net /r2: track 565.8 -> 561.9 mm
- net /r4: track 663.1 -> 659.3 mm
- net /r0: track 473.6 -> 469.9 mm
- net /r-1: track 417.9 -> 414.2 mm
- net /r3: track 589.3 -> 585.6 mm
- net /r1: track 523.0 -> 519.4 mm
- net /port_id: track 373.3 -> 376.3 mm
- net /cl17: track 377.0 -> 379.7 mm
- net /cl16: track 375.3 -> 377.7 mm
- net /cl15: track 541.8 -> 544.1 mm
- net /cl0: track 496.6 -> 495.4 mm
- net Net-(U1-PA7): track 4.32 -> 5.48 mm
- net /cl14: track 549.8 -> 550.8 mm
Other:
- board outline removed
