File: isokey/isokey.kicad_pcb (KiCad board)
At the start: 2 copper layers, 336 parts, among them J1 PadExp Right, J2 PadExp Left, Q1 BSS138, SW1 Cherry, SW10 Cherry, SW11 Cherry, SW12 Cherry, SW13 Cherry, SW14 Cherry, SW15 Cherry, SW16 Cherry, SW17 Cherry, SW18 Cherry, SW19 Cherry, SW2 Cherry, SW20 Cherry, SW21 Cherry, SW22 Cherry, SW23 Cherry, SW24 Cherry, SW25 Cherry, SW26 Cherry, SW27 Cherry, SW28 Cherry, SW29 Cherry, SW3 Cherry, SW30 Cherry, SW31 Cherry, SW32 Cherry, SW33 Cherry, SW34 Cherry, SW35 Cherry, SW36 Cherry, SW37 Cherry, SW38 Cherry, SW39 Cherry, SW4 Cherry, SW40 Cherry, SW41 Cherry, SW42 Cherry, SW43 Cherry, SW44 Cherry, SW45 Cherry, SW46 Cherry, SW47 Cherry, SW48 Cherry, SW5 Cherry, SW6 Cherry, SW7 Cherry, SW8 Cherry, SW9 Cherry, U1 BlackPill_STLINK, U3 TLV73318PDBV, U4 LP5569

Commit message: Continue routing
Parts:
- removed C38, C63, C64, C65, C66, C67, C68, C69, C70, C71, C72, C73, C74, C75, C76, C77, C78, C79, C80, C81, C82, C83: 100nF, Capacitor_SMD:C_0603_1608Metric_Pad1.08x0.95mm_HandSolder
- removed D100, D74, D79, D80, D81, D82, D83, D84, D85, D86, D87, D88, D89, D90, D91, D92, D93, D94, D95, D96, D97, D98, D99: SK6812MINI, LED_SMD:LED_SK6812MINI_PLCC4_3.5x3.5mm_P1.75mm
- removed the U1 at (190.0, -37.0)
- removed the U1 at (168.5, -38.0)
- added U1: BlackPill_STLINK, Module:BlackPill_doble_top-bot, F.Cu at (222.4, -40.8)
- C15, C16, C18, C19, C21, C22, C24, C25, C28, C32, C33, C39, C42, C45, C48, C51, C52, C54, C55, C56, C61, C62, D119, D26, D28: moved to B.Cu
- D27, D29: moved to F.Cu
- D30, D32, D34, D36, D38, D40, D41, D42, D44, D48, D50, D52, D54, D56, D58, D60, D62, D64, D66, D68, D72, D75, D76, D78: value SK6812MINI -> SK6812MINI-E; moved to B.Cu
- D31, D33, D35, D37, D39, D43, D45, D46, D47, D49, D51, D53, D55, D57, D59, D61, D63, D65, D67, D69, D70, D71, D73, D77: value SK6812MINI -> SK6812MINI-E
- moved R38 329.8 mm to (196.4, 10.5)
- moved R39 329.0 mm to (196.6, 12.3)
- moved C8 317.0 mm to (203.5, 13.8), turned to 180 degrees
- moved R33 312.3 mm to (209.4, 13.8)
- moved R40 309.7 mm to (201.3, -5.71)
- moved C9 309.6 mm to (209.4, 11.3)
- moved R35 309.4 mm to (203.5, 11.3)
- moved C10 277.6 mm to (191.9, -13.9)
- moved C11 277.6 mm to (191.9, -10.9)
- moved C12 277.6 mm to (191.9, -7.84)
- moved C13 277.6 mm to (191.9, -4.83)
- moved U3 277.6 mm to (202.4, -14.7)
- moved R31 273.0 mm to (236.6, -20.5), turned to 180 degrees
- moved R18 271.0 mm to (240.1, -25.6), turned to 180 degrees
- moved R20 268.8 mm to (240.1, -23.0), turned to 180 degrees
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Connections:
- D31 pad 1: Net-(D31-DOUT) -> Net-(D30-DOUT)
- D31 pad 3: Net-(D30-DOUT) -> Net-(D30-DIN)
- D32 pad 3: Net-(D31-DOUT) -> Net-(D30-DOUT)
- D33 pad 1: Net-(D33-DOUT) -> Net-(D32-DOUT)
- D33 pad 3: Net-(D32-DOUT) -> Net-(D30-DOUT)
- D34 pad 3: Net-(D33-DOUT) -> Net-(D32-DOUT)
- D35 pad 1: Net-(D35-DOUT) -> Net-(D34-DOUT)
- D35 pad 3: Net-(D34-DOUT) -> Net-(D32-DOUT)
- D36 pad 3: Net-(D35-DOUT) -> Net-(D34-DOUT)
- D37 pad 1: Net-(D37-DOUT) -> Net-(D36-DOUT)
- D37 pad 3: Net-(D36-DOUT) -> Net-(D34-DOUT)
- D38 pad 3: Net-(D37-DOUT) -> Net-(D36-DOUT)
- D39 pad 1: Net-(D39-DOUT) -> Net-(D38-DOUT)
- D39 pad 3: Net-(D38-DOUT) -> Net-(D36-DOUT)
- D40 pad 3: Net-(D39-DOUT) -> Net-(D38-DOUT)
- D45 pad 1: Net-(D45-DOUT) -> Net-(D40-DOUT)
- D45 pad 3: Net-(D44-DOUT) -> Net-(D38-DOUT)
- D46 pad 1: Net-(D46-DOUT) -> Net-(D41-DOUT)
- D46 pad 3: Net-(D45-DOUT) -> Net-(D40-DOUT)
- D47 pad 1: Net-(D47-DOUT) -> Net-(D42-DOUT)
- D47 pad 3: Net-(D46-DOUT) -> Net-(D41-DOUT)
- D48 pad 1: Net-(D48-DOUT) -> Net-(D43-DOUT)
- D48 pad 3: Net-(D47-DOUT) -> Net-(D42-DOUT)
- D49 pad 1: Net-(D49-DOUT) -> Net-(D44-DOUT)
- D49 pad 3: Net-(D48-DOUT) -> Net-(D43-DOUT)
- D50 pad 3: Net-(D49-DOUT) -> Net-(D44-DOUT)
- D55 pad 1: Net-(D55-DOUT) -> Net-(D50-DOUT)
- D55 pad 3: Net-(D54-DOUT) -> Net-(D44-DOUT)
- D56 pad 1: Net-(D56-DOUT) -> Net-(D51-DOUT)
- D56 pad 3: Net-(D55-DOUT) -> Net-(D50-DOUT)
- D57 pad 1: Net-(D57-DOUT) -> Net-(D52-DOUT)
- D57 pad 3: Net-(D56-DOUT) -> Net-(D51-DOUT)
- D58 pad 1: Net-(D58-DOUT) -> Net-(D53-DOUT)
- D58 pad 3: Net-(D57-DOUT) -> Net-(D52-DOUT)
- D59 pad 1: Net-(D59-DOUT) -> Net-(D54-DOUT)
- D59 pad 3: Net-(D58-DOUT) -> Net-(D53-DOUT)
- D60 pad 3: Net-(D59-DOUT) -> Net-(D54-DOUT)
- D65 pad 1: Net-(D65-DOUT) -> Net-(D60-DOUT)
- D65 pad 3: Net-(D64-DOUT) -> Net-(D54-DOUT)
- D66 pad 1: Net-(D66-DOUT) -> Net-(D61-DOUT)
- D66 pad 3: Net-(D65-DOUT) -> Net-(D60-DOUT)
- D67 pad 1: Net-(D67-DOUT) -> Net-(D62-DOUT)
- D67 pad 3: Net-(D66-DOUT) -> Net-(D61-DOUT)
- D68 pad 1: Net-(D68-DOUT) -> Net-(D63-DOUT)
- D68 pad 3: Net-(D67-DOUT) -> Net-(D62-DOUT)
- D69 pad 1: Net-(D69-DOUT) -> Net-(D64-DOUT)
- D69 pad 3: Net-(D68-DOUT) -> Net-(D63-DOUT)
- D70 pad 3: Net-(D69-DOUT) -> Net-(D64-DOUT)
- D73 pad 1: Net-(D73-DOUT) -> /led_w1_out
- D75 pad 1: Net-(D75-DOUT) -> Net-(D70-DOUT)
- D75 pad 3: Net-(D74-DOUT) -> Net-(D64-DOUT)
- D76 pad 1: Net-(D76-DOUT) -> Net-(D71-DOUT)
- D76 pad 3: Net-(D75-DOUT) -> Net-(D70-DOUT)
- D77 pad 1: Net-(D77-DOUT) -> Net-(D72-DOUT)
- D77 pad 3: Net-(D76-DOUT) -> Net-(D71-DOUT)
- D78 pad 1: Net-(D78-DOUT) -> /led_w1_out
- D78 pad 3: Net-(D77-DOUT) -> Net-(D72-DOUT)
Routing:
- net GND: track 0.00 -> 826.7 mm, vias 0 -> 93
- net +5V: track 0.00 -> 746.9 mm, vias 0 -> 46
- net /cl3: track 0.00 -> 129.6 mm, vias 0 -> 9
- net /cl4: track 0.00 -> 124.9 mm, vias 0 -> 9
- net /sw0_r: track 0.00 -> 100.7 mm, vias 0 -> 7
- net /cl1: track 0.00 -> 100.7 mm, vias 0 -> 7
- net /cl2: track 0.00 -> 99.1 mm, vias 0 -> 7
- net /r0: track 0.00 -> 98.1 mm, vias 0 -> 5
- net /r3: track 0.00 -> 98.0 mm, vias 0 -> 5
- net /r1: track 0.00 -> 98.0 mm, vias 0 -> 5
- net /r2: track 0.00 -> 90.1 mm, vias 0 -> 5
- net +3.3V: track 0.00 -> 37.0 mm
- net Net-(D72-DOUT): track 0.00 -> 25.8 mm, vias 0 -> 3
- net Net-(D63-DOUT): track 0.00 -> 25.3 mm, vias 0 -> 4
- net Net-(D62-DOUT): track 0.00 -> 25.3 mm, vias 0 -> 4
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Other:
- board outline added: 4.6 x 4.6 mm

Commit message: Continue routing
Parts:
- removed J1: PadExp Right, Connector_JST:JST_GH_SM14B-GHS-TB_1x14-1MP_P1.25mm_Horizontal
- removed J2: PadExp Left, Connector_JST:JST_GH_SM14B-GHS-TB_1x14-1MP_P1.25mm_Horizontal
- removed R43: 22R, Resistor_SMD:R_0603_1608Metric_Pad0.98x0.95mm_HandSolder
- added TP1: CL6, TestPoint:Testpoint_Pad_1.0x2.0mm, F.Cu at (345.5, 11.5)
- added TP10: GND, TestPoint:Testpoint_Pad_1.0x2.0mm, F.Cu at (345.5, -47.7)
- added TP11: W1, TestPoint:Testpoint_Pad_1.0x2.0mm, F.Cu at (345.5, 21.0)
- added TP2: CL7, TestPoint:Testpoint_Pad_1.0x2.0mm, F.Cu at (345.5, 13.0)
- added TP3: CL8, TestPoint:Testpoint_Pad_1.0x2.0mm, F.Cu at (345.5, 14.5)
- added TP4: CL9, TestPoint:Testpoint_Pad_1.0x2.0mm, F.Cu at (345.5, 16.0)
- added TP5: +5V, TestPoint:Testpoint_Pad_1.0x2.0mm, F.Cu at (345.6, -49.2)
- added TP6: GND, TestPoint:Testpoint_Pad_1.0x2.0mm, F.Cu at (345.5, -28.8)
- added TP7: CL10, TestPoint:Testpoint_Pad_1.0x2.0mm, F.Cu at (345.5, 17.5)
- added TP8: ID, TestPoint:Testpoint_Pad_1.0x2.0mm, F.Cu at (345.5, 19.5)
- added TP9: +5V, TestPoint:Testpoint_Pad_1.0x2.0mm, F.Cu at (345.5, -30.2)
- C59, C60: moved to B.Cu
- moved R12 182.8 mm to (339.6, 22.3), turned to 0 degrees
- moved U2 99.5 mm to (230.1, -4.30)
- moved R11 54.3 mm to (256.8, -81.0)
- moved D131 37.5 mm to (243.2, 33.5), turned to -150 degrees
- moved D133 36.3 mm to (279.1, 26.5), turned to -75 degrees
- moved D25 33.3 mm to (210.4, 21.9)
- moved C85 33.1 mm to (152.3, -9.66)
- moved C88 33.1 mm to (152.3, -7.15)
- moved D115 33.1 mm to (141.6, -9.62)
- moved D116 33.1 mm to (141.6, -7.03)
- moved D117 33.1 mm to (141.6, -4.44)
- moved D118 33.1 mm to (141.6, -1.85)
- moved R40 33.1 mm to (170.2, 5.67)
- moved R45 33.1 mm to (152.3, -4.64)
- moved R46 33.1 mm to (152.3, -2.13)
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Connections:
- R12 pad 2: /port_id -> /led_w1_out
- R13 pad 1: /cl9 -> unconnected-(R13-Pad1)
- R15 pad 1: /cl10 -> unconnected-(R15-Pad1)
- R17 pad 1: /cl11 -> unconnected-(R17-Pad1)
- R19 pad 1: /r0 -> unconnected-(R19-Pad1)
- R2 pad 1: /cl4 -> unconnected-(R2-Pad1)
- R21 pad 1: /r1 -> unconnected-(R21-Pad1)
- R23 pad 1: /r2 -> unconnected-(R23-Pad1)
- R24 pad 2: /~{CS} -> unconnected-(R24-Pad2)
- R25 pad 1: /r3 -> unconnected-(R25-Pad1)
- R26 pad 2: /SCLK -> unconnected-(R26-Pad2)
- R27 pad 1: /r4 -> unconnected-(R27-Pad1)
- R28 pad 2: /MISO -> unconnected-(R28-Pad2)
- R29 pad 1: /r-1 -> unconnected-(R29-Pad1)
- R30 pad 2: /MOSI -> /r0
- R31 pad 1: /cl1 -> unconnected-(R31-Pad1)
- R32 pad 1: /cl2 -> unconnected-(R32-Pad1)
- R34 pad 1: /cl3 -> unconnected-(R34-Pad1)
- R4 pad 1: /cl5 -> unconnected-(R4-Pad1)
- R5 pad 1: /cl6 -> unconnected-(R5-Pad1)
- R7 pad 1: /cl7 -> unconnected-(R7-Pad1)
- R9 pad 1: /cl8 -> unconnected-(R9-Pad1)
Routing:
- net /cl4: track 124.9 -> 213.9 mm
- net /cl2: track 99.1 -> 181.7 mm, vias 7 -> 9
- net /cl3: track 129.6 -> 195.8 mm
- net /cl1: track 100.7 -> 159.6 mm, vias 7 -> 9
- net Net-(D70-DOUT): track 0.00 -> 36.5 mm, vias 0 -> 1
- net +5V: track 746.9 -> 781.2 mm, vias 46 -> 51
- net Net-(D44-DOUT): track 0.00 -> 33.5 mm, vias 0 -> 3
- net Net-(D38-DOUT): track 8.77 -> 29.0 mm, vias 2 -> 3
- net Net-(D54-DOUT): track 8.77 -> 28.8 mm, vias 2 -> 3
- net /r0: track 98.1 -> 109.0 mm
- net Net-(D71-DOUT): track 16.6 -> 27.2 mm, vias 2 -> 3
- net Net-(D131-K): track 0.00 -> 8.66 mm
- net Net-(D133-K): track 0.00 -> 8.55 mm
- net Net-(D132-K): track 0.00 -> 6.02 mm
- net /sw0_r: track 100.7 -> 106.7 mm
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
Commit message: Continue routing
Parts:
- removed R1, R10, R18, R20, R22, R28, R3, R30, R8: 22R, Resistor_SMD:R_0603_1608Metric_Pad0.98x0.95mm_HandSolder
- added R43: 22R, Resistor_SMD:R_0603_1608Metric_Pad0.98x0.95mm_HandSolder, B.Cu at (246.2, -65.8)
- added R48: 22R, Resistor_SMD:R_0603_1608Metric_Pad0.98x0.95mm_HandSolder, F.Cu at (246.2, -7.00)
- added R49: 22R, Resistor_SMD:R_0603_1608Metric_Pad0.98x0.95mm_HandSolder, B.Cu at (246.2, -7.00)
- added R50: 22R, Resistor_SMD:R_0603_1608Metric_Pad0.98x0.95mm_HandSolder, F.Cu at (246.2, -5.25)
- added R51: 22R, Resistor_SMD:R_0603_1608Metric_Pad0.98x0.95mm_HandSolder, B.Cu at (246.2, -5.25)
- added R52: 22R, Resistor_SMD:R_0603_1608Metric_Pad0.98x0.95mm_HandSolder, F.Cu at (246.2, -3.50)
- added R53: 22R, Resistor_SMD:R_0603_1608Metric_Pad0.98x0.95mm_HandSolder, B.Cu at (246.2, -3.50)
- added R54: 22R, Resistor_SMD:R_0603_1608Metric_Pad0.98x0.95mm_HandSolder, F.Cu at (246.2, -1.75)
- added R55: 22R, Resistor_SMD:R_0603_1608Metric_Pad0.98x0.95mm_HandSolder, B.Cu at (246.2, -1.75)
- added R56: 22R, Resistor_SMD:R_0603_1608Metric_Pad0.98x0.95mm_HandSolder, B.Cu at (246.2, 0.00)
- added R57: 22R, Resistor_SMD:R_0603_1608Metric_Pad0.98x0.95mm_HandSolder, F.Cu at (246.2, 0.00)
- R15, R2, R21, R25, R27, R31, R34, R5, R9: moved to B.Cu
- moved R35 88.1 mm to (246.2, -65.8), turned to 180 degrees
- moved R33 86.1 mm to (246.2, -64.0), turned to 180 degrees
- moved C1 53.1 mm to (216.7, -91.7)
- moved C4 53.1 mm to (217.5, -85.5)
- moved C2 53.1 mm to (220.8, -96.2)
- moved C3 53.1 mm to (216.7, -88.7)
- moved R6 44.7 mm to (244.2, -82.8)
- moved R19 44.6 mm to (246.2, -8.75)
- moved R36 43.1 mm to (218.5, -78.3)
- moved C7 43.1 mm to (220.5, -78.8)
- moved R37 43.1 mm to (221.0, -78.3)
- moved R31 42.1 mm to (246.2, -62.2)
- moved R21 42.0 mm to (246.2, -8.75)
- moved R14 40.0 mm to (205.6, -31.2)
- moved R16 40.0 mm to (205.6, -28.6)
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Connections:
- D25 pad 1: unconnected-(D25-K-Pad1) -> /sw0_r
- R13 pad 1: unconnected-(R13-Pad1) -> /r2
- R13 pad 2: Net-(U1-PA5) -> unconnected-(R13-Pad2)
- R15 pad 1: unconnected-(R15-Pad1) -> /r3
- R15 pad 2: Net-(U1-PA6) -> unconnected-(R15-Pad2)
- R17 pad 1: unconnected-(R17-Pad1) -> /r3
- R17 pad 2: Net-(U1-PA7) -> unconnected-(R17-Pad2)
- R19 pad 1: unconnected-(R19-Pad1) -> /r4
- R19 pad 2: Net-(U1-PA8) -> unconnected-(R19-Pad2)
- R2 pad 1: unconnected-(R2-Pad1) -> /r0
- R2 pad 2: Net-(U1-PA0) -> unconnected-(R2-Pad2)
- R21 pad 1: unconnected-(R21-Pad1) -> /r4
- R21 pad 2: Net-(U1-PA9) -> unconnected-(R21-Pad2)
- R23 pad 1: unconnected-(R23-Pad1) -> /cl0
- R23 pad 2: Net-(U1-PA10) -> unconnected-(R23-Pad2)
- R24 pad 2: unconnected-(R24-Pad2) -> /ENC1A
- R25 pad 1: unconnected-(R25-Pad1) -> /cl0
- R25 pad 2: Net-(U1-PA11) -> unconnected-(R25-Pad2)
- R26 pad 2: unconnected-(R26-Pad2) -> /ENC1B
- R27 pad 1: unconnected-(R27-Pad1) -> /cl1
- R27 pad 2: Net-(U1-PA12) -> unconnected-(R27-Pad2)
- R29 pad 1: unconnected-(R29-Pad1) -> /cl1
- R29 pad 2: Net-(U1-PA15) -> unconnected-(R29-Pad2)
- R31 pad 1: unconnected-(R31-Pad1) -> /cl2
- R31 pad 2: Net-(U1-PC13) -> unconnected-(R31-Pad2)
- R32 pad 1: unconnected-(R32-Pad1) -> /cl2
- R32 pad 2: Net-(U1-PC14) -> unconnected-(R32-Pad2)
- R33 pad 1: /PA13 -> /cl3
- R33 pad 2: /ENC1A -> unconnected-(R33-Pad2)
- R34 pad 1: unconnected-(R34-Pad1) -> /cl3
- R34 pad 2: Net-(U1-PC15) -> unconnected-(R34-Pad2)
- R35 pad 1: /PA14 -> /cl4
- R35 pad 2: /ENC1B -> unconnected-(R35-Pad2)
- R4 pad 1: unconnected-(R4-Pad1) -> /r0
- R4 pad 2: Net-(U1-PA1) -> unconnected-(R4-Pad2)
- R5 pad 1: unconnected-(R5-Pad1) -> /r1
- R5 pad 2: Net-(U1-PA2) -> unconnected-(R5-Pad2)
- R7 pad 1: unconnected-(R7-Pad1) -> /r1
- R7 pad 2: Net-(U1-PA3) -> unconnected-(R7-Pad2)
- R9 pad 1: unconnected-(R9-Pad1) -> /r2
- R9 pad 2: Net-(U1-PA4) -> unconnected-(R9-Pad2)
- RSW1 pad S1: /cl6 -> /cl0
- RSW1 pad S2: /sw1_r -> /sw0_r
- SW1 pad 2: /sw0_r -> /cl0
- SW11 pad 2: /sw0_r -> /cl0
- SW12 pad 1: /sw0_r -> /cl0
- SW2 pad 1: /sw0_r -> /cl0
- SW21 pad 2: /sw0_r -> /cl0
- SW22 pad 1: /sw0_r -> /cl0
- SW31 pad 2: /sw0_r -> /cl0
- SW32 pad 1: /sw0_r -> /cl0
- U1 pad 10: Net-(U1-PA15) -> unconnected-(U1-PA15-Pad10)
- U1 pad 12: Net-(U1-PB4) -> unconnected-(U1-PB4-Pad12)
- U1 pad 13: Net-(U1-PB5) -> unconnected-(U1-PB5-Pad13)
- U1 pad 16: Net-(U1-PB8) -> unconnected-(U1-PB8-Pad16)
- U1 pad 17: Net-(U1-PB9) -> unconnected-(U1-PB9-Pad17)
- U1 pad 22: Net-(U1-PC13) -> unconnected-(U1-PC13-Pad22)
- U1 pad 23: Net-(U1-PC14) -> unconnected-(U1-PC14-Pad23)
- U1 pad 24: Net-(U1-PC15) -> unconnected-(U1-PC15-Pad24)
- U1 pad 26: Net-(U1-PA0) -> unconnected-(U1-PA0-Pad26)
- U1 pad 27: Net-(U1-PA1) -> unconnected-(U1-PA1-Pad27)
- U1 pad 28: Net-(U1-PA2) -> unconnected-(U1-PA2-Pad28)
- U1 pad 29: Net-(U1-PA3) -> unconnected-(U1-PA3-Pad29)
- U1 pad 3: Net-(U1-PB14) -> unconnected-(U1-PB14-Pad3)
- U1 pad 30: Net-(U1-PA4) -> unconnected-(U1-PA4-Pad30)
- U1 pad 31: Net-(U1-PA5) -> unconnected-(U1-PA5-Pad31)
- U1 pad 32: Net-(U1-PA6) -> unconnected-(U1-PA6-Pad32)
- U1 pad 33: Net-(U1-PA7) -> unconnected-(U1-PA7-Pad33)
- U1 pad 34: Net-(U1-PB0) -> unconnected-(U1-PB0-Pad34)
- U1 pad 35: Net-(U1-PB1) -> unconnected-(U1-PB1-Pad35)
- U1 pad 37: Net-(U1-PB10) -> unconnected-(U1-PB10-Pad37)
- U1 pad 4: Net-(U1-PB15) -> unconnected-(U1-PB15-Pad4)
- U1 pad 5: Net-(U1-PA8) -> unconnected-(U1-PA8-Pad5)
- U1 pad 6: Net-(U1-PA9) -> unconnected-(U1-PA9-Pad6)
- U1 pad 7: Net-(U1-PA10) -> unconnected-(U1-PA10-Pad7)
- U1 pad 8: Net-(U1-PA11) -> unconnected-(U1-PA11-Pad8)
- U1 pad 9: Net-(U1-PA12) -> unconnected-(U1-PA12-Pad9)
Routing:
- net /cl0: track 0.00 -> 107.7 mm, vias 0 -> 8
- net /sw0_r: track 106.7 -> 0.00 mm, vias 7 -> 0
- net Net-(R11-Pad1): track 0.00 -> 100.8 mm, vias 0 -> 1
- net /cl10: track 0.00 -> 99.5 mm, vias 0 -> 1
- net /cl9: track 0.00 -> 98.5 mm, vias 0 -> 1
- net /cl8: track 0.00 -> 98.1 mm, vias 0 -> 1
- net /cl7: track 0.00 -> 97.6 mm, vias 0 -> 1
- net /cl6: track 0.00 -> 97.4 mm, vias 0 -> 1
- net Net-(U1-PB5): track 24.3 -> 0.00 mm, vias 1 -> 0
- net Net-(U1-PB15): track 24.3 -> 0.00 mm, vias 1 -> 0
- net Net-(U1-PA8): track 24.3 -> 0.00 mm, vias 1 -> 0
- net Net-(U1-PB4): track 24.3 -> 0.00 mm, vias 1 -> 0
- net Net-(U1-PB14): track 24.3 -> 0.00 mm, vias 1 -> 0
- net Net-(U1-PA15): track 24.3 -> 0.00 mm, vias 1 -> 0
- net Net-(U1-PA12): track 24.3 -> 0.00 mm, vias 1 -> 0
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
Commit message: Continue routing
Parts:
- removed Q1: BSS138, Package_TO_SOT_SMD:SOT-23-3
- removed R14, R16, R24, R26: 22R, Resistor_SMD:R_0603_1608Metric_Pad0.98x0.95mm_HandSolder
- added C38: 1uF, Capacitor_SMD:C_0805_2012Metric, B.Cu at (231.9, -13.2)
- added C63: 10uF, Capacitor_SMD:C_1206_3216Metric, B.Cu at (234.4, -12.7)
- added C64: 1uF, Capacitor_SMD:C_0805_2012Metric, B.Cu at (245.2, -68.0)
- added C65: 10uF, Capacitor_SMD:C_1206_3216Metric, B.Cu at (330.0, -29.8)
- added C66: 10uF, Capacitor_SMD:C_1206_3216Metric, F.Cu at (253.8, 14.0)
- added C67: 10uF, Capacitor_SMD:C_1206_3216Metric, F.Cu at (250.5, -69.0)
- added C68: 100nF, Capacitor_SMD:C_0603_1608Metric_Pad1.08x0.95mm_HandSolder, F.Cu at (202.3, -9.40)
- added C69: 100nF, Capacitor_SMD:C_0603_1608Metric_Pad1.08x0.95mm_HandSolder, B.Cu at (202.3, -9.40)
- added D74: 1N4448W, Diode_SMD:D_SOD-123, F.Cu at (177.7, 54.6)
- added JP1: SolderJumper_3_Open_line, Jumper:SolderJumper-3_P2.0mm_Open_TrianglePad1.0x1.5mm_NumberLabels, F.Cu at (230.6, -63.5)
- added JP10: SolderJumper_3_Open_line, Jumper:SolderJumper-3_P2.0mm_Open_TrianglePad1.0x1.5mm_NumberLabels, F.Cu at (230.6, -43.2)
- added JP11: SolderJumper_3_Open_line, Jumper:SolderJumper-3_P2.0mm_Open_TrianglePad1.0x1.5mm_NumberLabels, F.Cu at (230.6, -40.6)
- added JP12: SolderJumper_3_Open_line, Jumper:SolderJumper-3_P2.0mm_Open_TrianglePad1.0x1.5mm_NumberLabels, F.Cu at (230.6, -38.1)
- added JP13: SolderJumper_3_Open_line, Jumper:SolderJumper-3_P2.0mm_Open_TrianglePad1.0x1.5mm_NumberLabels, F.Cu at (230.6, -35.6)
- added JP14: SolderJumper_3_Open_line, Jumper:SolderJumper-3_P2.0mm_Open_TrianglePad1.0x1.5mm_NumberLabels, F.Cu at (230.6, -33.0)
- added JP15: SolderJumper_3_Open_line, Jumper:SolderJumper-3_P2.0mm_Open_TrianglePad1.0x1.5mm_NumberLabels, F.Cu at (230.6, -30.5)
- added JP16: SolderJumper_3_Open_line, Jumper:SolderJumper-3_P2.0mm_Open_TrianglePad1.0x1.5mm_NumberLabels, F.Cu at (230.6, -27.9)
- added JP17: SolderJumper_3_Open_line, Jumper:SolderJumper-3_P2.0mm_Open_TrianglePad1.0x1.5mm_NumberLabels, F.Cu at (230.6, -25.4)
- added JP18: SolderJumper_3_Open_line, Jumper:SolderJumper-3_P2.0mm_Open_TrianglePad1.0x1.5mm_NumberLabels, F.Cu at (230.6, -22.9)
- added JP19: SolderJumper_3_Open_line, Jumper:SolderJumper-3_P2.0mm_Open_TrianglePad1.0x1.5mm_NumberLabels, F.Cu at (230.6, -20.3)
- added JP2: SolderJumper_3_Open_line, Jumper:SolderJumper-3_P2.0mm_Open_TrianglePad1.0x1.5mm_NumberLabels, F.Cu at (230.6, -66.0)
- added JP20: SolderJumper_3_Open_line, Jumper:SolderJumper-3_P2.0mm_Open_TrianglePad1.0x1.5mm_NumberLabels, F.Cu at (230.6, -17.8)
- added JP21: SolderJumper_3_Open_line, Jumper:SolderJumper-3_P2.0mm_Open_TrianglePad1.0x1.5mm_NumberLabels, B.Cu at (234.6, -17.8)
- added JP22: SolderJumper_3_Open_line, Jumper:SolderJumper-3_P2.0mm_Open_TrianglePad1.0x1.5mm_NumberLabels, B.Cu at (234.6, -20.3)
- added JP23: SolderJumper_3_Open_line, Jumper:SolderJumper-3_P2.0mm_Open_TrianglePad1.0x1.5mm_NumberLabels, B.Cu at (234.6, -22.9)
- added JP24: SolderJumper_3_Open_line, Jumper:SolderJumper-3_P2.0mm_Open_TrianglePad1.0x1.5mm_NumberLabels, B.Cu at (234.6, -25.4)
- added JP25: SolderJumper_3_Open_line, Jumper:SolderJumper-3_P2.0mm_Open_TrianglePad1.0x1.5mm_NumberLabels, B.Cu at (234.6, -27.9)
- added JP26: SolderJumper_3_Open_line, Jumper:SolderJumper-3_P2.0mm_Open_TrianglePad1.0x1.5mm_NumberLabels, B.Cu at (234.6, -30.5)
- added JP27: SolderJumper_3_Open_line, Jumper:SolderJumper-3_P2.0mm_Open_TrianglePad1.0x1.5mm_NumberLabels, B.Cu at (234.6, -33.0)
- added JP28: SolderJumper_3_Open_line, Jumper:SolderJumper-3_P2.0mm_Open_TrianglePad1.0x1.5mm_NumberLabels, B.Cu at (234.6, -35.6)
- added JP29: SolderJumper_3_Open_line, Jumper:SolderJumper-3_P2.0mm_Open_TrianglePad1.0x1.5mm_NumberLabels, B.Cu at (234.6, -38.1)
- added JP3: SolderJumper_3_Open_line, Jumper:SolderJumper-3_P2.0mm_Open_TrianglePad1.0x1.5mm_NumberLabels, F.Cu at (230.6, -61.0)
- added JP30: SolderJumper_3_Open_line, Jumper:SolderJumper-3_P2.0mm_Open_TrianglePad1.0x1.5mm_NumberLabels, B.Cu at (234.6, -40.6)
- added JP31: SolderJumper_3_Open_line, Jumper:SolderJumper-3_P2.0mm_Open_TrianglePad1.0x1.5mm_NumberLabels, B.Cu at (234.6, -43.2)
- added JP32: SolderJumper_3_Open_line, Jumper:SolderJumper-3_P2.0mm_Open_TrianglePad1.0x1.5mm_NumberLabels, B.Cu at (234.6, -45.7)
- added JP33: SolderJumper_3_Open_line, Jumper:SolderJumper-3_P2.0mm_Open_TrianglePad1.0x1.5mm_NumberLabels, B.Cu at (234.6, -48.3)
- added JP34: SolderJumper_3_Open_line, Jumper:SolderJumper-3_P2.0mm_Open_TrianglePad1.0x1.5mm_NumberLabels, B.Cu at (234.6, -50.8)
- added JP35: SolderJumper_3_Open_line, Jumper:SolderJumper-3_P2.0mm_Open_TrianglePad1.0x1.5mm_NumberLabels, B.Cu at (234.6, -53.3)
- added JP36: SolderJumper_3_Open_line, Jumper:SolderJumper-3_P2.0mm_Open_TrianglePad1.0x1.5mm_NumberLabels, B.Cu at (234.6, -55.9)
- added JP37: SolderJumper_3_Open_line, Jumper:SolderJumper-3_P2.0mm_Open_TrianglePad1.0x1.5mm_NumberLabels, B.Cu at (234.6, -58.4)
- added JP38: SolderJumper_3_Open_line, Jumper:SolderJumper-3_P2.0mm_Open_TrianglePad1.0x1.5mm_NumberLabels, B.Cu at (234.6, -61.0)
- added JP39: SolderJumper_3_Open_line, Jumper:SolderJumper-3_P2.0mm_Open_TrianglePad1.0x1.5mm_NumberLabels, B.Cu at (234.6, -63.5)
- added JP4: SolderJumper_3_Open_line, Jumper:SolderJumper-3_P2.0mm_Open_TrianglePad1.0x1.5mm_NumberLabels, F.Cu at (230.6, -58.4)
- added JP40: SolderJumper_3_Open_line, Jumper:SolderJumper-3_P2.0mm_Open_TrianglePad1.0x1.5mm_NumberLabels, B.Cu at (234.6, -66.0)
- added JP43: SolderJumper_3_Open_line, Jumper:SolderJumper-3_P2.0mm_Open_TrianglePad1.0x1.5mm_NumberLabels, F.Cu at (176.8, 61.9)
- added JP44: SolderJumper_3_Open_line, Jumper:SolderJumper-3_P2.0mm_Open_TrianglePad1.0x1.5mm_NumberLabels, F.Cu at (176.8, 65.5)
- added JP5: SolderJumper_3_Open_line, Jumper:SolderJumper-3_P2.0mm_Open_TrianglePad1.0x1.5mm_NumberLabels, F.Cu at (230.6, -55.9)
- added JP6: SolderJumper_3_Open_line, Jumper:SolderJumper-3_P2.0mm_Open_TrianglePad1.0x1.5mm_NumberLabels, F.Cu at (230.6, -53.3)
- added JP7: SolderJumper_3_Open_line, Jumper:SolderJumper-3_P2.0mm_Open_TrianglePad1.0x1.5mm_NumberLabels, F.Cu at (230.6, -50.8)
- added JP8: SolderJumper_3_Open_line, Jumper:SolderJumper-3_P2.0mm_Open_TrianglePad1.0x1.5mm_NumberLabels, F.Cu at (230.6, -48.3)
- added JP9: SolderJumper_3_Open_line, Jumper:SolderJumper-3_P2.0mm_Open_TrianglePad1.0x1.5mm_NumberLabels, F.Cu at (230.6, -45.7)
- added M1: JOYSTICK-PSP1000, SparkFun-Electromechanical:JOYSTICK-PSP1000, F.Cu at (174.2, 82.4)
- added Q2: BSS138, Package_TO_SOT_SMD:SOT-23-3, B.Cu at (244.7, -44.4)
- added Q3: BSS138, Package_TO_SOT_SMD:SOT-23-3, F.Cu at (244.7, -44.4)
- added R1: 4k7, Resistor_SMD:R_0603_1608Metric_Pad0.98x0.95mm_HandSolder, F.Cu at (244.3, -47.0)
- added R10: 22R, Resistor_SMD:R_0603_1608Metric_Pad0.98x0.95mm_HandSolder, B.Cu at (242.8, -7.50)
- added R18: 10k, Resistor_SMD:R_0603_1608Metric_Pad0.98x0.95mm_HandSolder, F.Cu at (124.2, -6.05)
- added R20: 4k7, Resistor_SMD:R_0603_1608Metric_Pad0.98x0.95mm_HandSolder, B.Cu at (244.3, -47.0)
- added R22: 10k, Resistor_SMD:R_0603_1608Metric_Pad0.98x0.95mm_HandSolder, B.Cu at (245.3, -41.5)
- added R28: 22R, Resistor_SMD:R_0603_1608Metric_Pad0.98x0.95mm_HandSolder, B.Cu at (247.8, -46.2)
- added R3: 10k, Resistor_SMD:R_0603_1608Metric_Pad0.98x0.95mm_HandSolder, F.Cu at (245.3, -41.5)
- added R30: 22R, Resistor_SMD:R_0603_1608Metric_Pad0.98x0.95mm_HandSolder, B.Cu at (245.3, -39.9)
- added R58: 22R, Resistor_SMD:R_0603_1608Metric_Pad0.98x0.95mm_HandSolder, F.Cu at (189.5, -20.7)
- added R59: 22R, Resistor_SMD:R_0603_1608Metric_Pad0.98x0.95mm_HandSolder, F.Cu at (189.5, -18.1)
- added R60: 22R, Resistor_SMD:R_0603_1608Metric_Pad0.98x0.95mm_HandSolder, F.Cu at (189.5, -15.6)
- added R61: 22R, Resistor_SMD:R_0603_1608Metric_Pad0.98x0.95mm_HandSolder, B.Cu at (193.6, -9.70)
- added R62: 22R, Resistor_SMD:R_0603_1608Metric_Pad0.98x0.95mm_HandSolder, F.Cu at (193.6, -9.70)
- added R63: 22R, Resistor_SMD:R_0603_1608Metric_Pad0.98x0.95mm_HandSolder, B.Cu at (193.5, -11.9)
- added R64: 22R, Resistor_SMD:R_0603_1608Metric_Pad0.98x0.95mm_HandSolder, F.Cu at (193.5, -11.9)
- added R8: 22R, Resistor_SMD:R_0603_1608Metric_Pad0.98x0.95mm_HandSolder, B.Cu at (341.5, 21.0)
- added U6: JOYSTICKPTH, SparkFun-Electromechanical:JOYSTICK, F.Cu at (221.8, 34.8)
- added U7: JOYSTICKPTH, SparkFun-Electromechanical:JOYSTICK, B.Cu at (221.8, 34.8)
- C5, C6, C8, R39, R40: moved to B.Cu
- R41: value 4k7 -> 10k
- R42: value 10k -> 22R
- U1: footprint Module:BlackPill_doble_top-bot -> Module:BlackPill
- moved C4 125.5 mm to (330.0, -29.8), turned to -90 degrees
- moved C5 104.0 mm to (253.8, 14.0), turned to 0 degrees
- moved C7 100.0 mm to (189.7, 16.4)
- moved R36 98.4 mm to (191.9, 16.4)
- moved R37 98.4 mm to (194.4, 16.4)
- moved R41 92.3 mm to (197.4, -9.40)
- moved C2 84.6 mm to (234.4, -12.7), turned to -90 degrees
- moved R42 82.7 mm to (189.5, -23.2)
- moved C1 79.9 mm to (231.9, -13.2), turned to -90 degrees
- moved R11 74.8 mm to (242.8, -7.50)
- moved C85 52.1 mm to (104.5, -30.5)
- moved C88 52.1 mm to (104.5, -28.0)
- moved R45 52.1 mm to (104.5, -25.5)
- moved R46 52.1 mm to (104.5, -23.0)
- moved R47 52.1 mm to (104.5, -20.5)
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Connections:
- C9 pad 1: /ENC1A -> /ENC1B
- R11 pad 2: /port_id -> /pc14
- R13 pad 2: unconnected-(R13-Pad2) -> /pb4
- R15 pad 2: unconnected-(R15-Pad2) -> /pa2
- R17 pad 2: unconnected-(R17-Pad2) -> /pa2
- R19 pad 2: unconnected-(R19-Pad2) -> /pc13
- R2 pad 2: unconnected-(R2-Pad2) -> /pb0
- R21 pad 2: unconnected-(R21-Pad2) -> /pc13
- R23 pad 2: unconnected-(R23-Pad2) -> /pb2
- R25 pad 2: unconnected-(R25-Pad2) -> /pb2
- R27 pad 2: unconnected-(R27-Pad2) -> /pa8
- R29 pad 2: unconnected-(R29-Pad2) -> /pa8
- R31 pad 2: unconnected-(R31-Pad2) -> /pb10
- R32 pad 2: unconnected-(R32-Pad2) -> /pb10
- R33 pad 2: unconnected-(R33-Pad2) -> /pb15
- R34 pad 2: unconnected-(R34-Pad2) -> /pb15
- R35 pad 2: unconnected-(R35-Pad2) -> /pb14
- R39 pad 1: /ENC1A -> /ENC1B
- R4 pad 2: unconnected-(R4-Pad2) -> /pb0
- R40 pad 1: Net-(U3-EN) -> /ENC1A
- R41 pad 1: /led_w1_in -> /ENC1A
- R41 pad 2: +5V -> +3.3V
- R42 pad 1: /led_w1 -> /led_SCL
- R42 pad 2: +3.3V -> /pb6
- R43 pad 2: unconnected-(R43-Pad2) -> /pb14
- R48 pad 2: unconnected-(R48-Pad2) -> /pb5
- R49 pad 2: unconnected-(R49-Pad2) -> /pb5
- R5 pad 2: unconnected-(R5-Pad2) -> /pa3
- R50 pad 2: unconnected-(R50-Pad2) -> /pa1
- R51 pad 2: unconnected-(R51-Pad2) -> /pa1
- R52 pad 2: unconnected-(R52-Pad2) -> /pa0
- R53 pad 2: unconnected-(R53-Pad2) -> /pa0
- R54 pad 2: unconnected-(R54-Pad2) -> /pb8
- R55 pad 2: unconnected-(R55-Pad2) -> /pb8
- R56 pad 2: unconnected-(R56-Pad2) -> /pc15
- R57 pad 2: unconnected-(R57-Pad2) -> /pc15
- R6 pad 1: Net-(U1-PB3) -> /led_w1
- R6 pad 2: /led_w1 -> /pb3
- R7 pad 2: unconnected-(R7-Pad2) -> /pa3
- R9 pad 2: unconnected-(R9-Pad2) -> /pb4
- TP1 pad 1: /cl6 -> /cl5
- TP2 pad 1: /cl7 -> /cl6
- TP3 pad 1: /cl8 -> /cl7
- TP4 pad 1: /cl9 -> /cl8
- TP7 pad 1: /cl10 -> /cl9
- U1 pad 1: Net-(U1-PB12) -> /1
- U1 pad 10: unconnected-(U1-PA15-Pad10) -> /10
- U1 pad 11: Net-(U1-PB3) -> /11
- U1 pad 12: unconnected-(U1-PB4-Pad12) -> /12
- U1 pad 13: unconnected-(U1-PB5-Pad13) -> /13
- U1 pad 14: Net-(U1-PB6) -> /14
- U1 pad 15: Net-(U1-PB7) -> /15
- U1 pad 16: unconnected-(U1-PB8-Pad16) -> /16
- U1 pad 17: unconnected-(U1-PB9-Pad17) -> /17
- U1 pad 18: +5V -> /18
- U1 pad 19: GND -> /19
- U1 pad 2: Net-(U1-PB13) -> /2
- U1 pad 20: +3.3V -> /20
- U1 pad 21: unconnected-(U1-VBAT-Pad21) -> /21
- U1 pad 22: unconnected-(U1-PC13-Pad22) -> /22
- U1 pad 23: unconnected-(U1-PC14-Pad23) -> /23
- U1 pad 24: unconnected-(U1-PC15-Pad24) -> /24
- U1 pad 25: unconnected-(U1-~{RESET}-Pad25) -> /25
- U1 pad 26: unconnected-(U1-PA0-Pad26) -> /26
- U1 pad 27: unconnected-(U1-PA1-Pad27) -> /27
- U1 pad 28: unconnected-(U1-PA2-Pad28) -> /28
- U1 pad 29: unconnected-(U1-PA3-Pad29) -> /29
- U1 pad 3: unconnected-(U1-PB14-Pad3) -> /3
- U1 pad 30: unconnected-(U1-PA4-Pad30) -> /30
- U1 pad 31: unconnected-(U1-PA5-Pad31) -> /31
- U1 pad 32: unconnected-(U1-PA6-Pad32) -> /32
- U1 pad 33: unconnected-(U1-PA7-Pad33) -> /33
- U1 pad 34: unconnected-(U1-PB0-Pad34) -> /34
- U1 pad 35: unconnected-(U1-PB1-Pad35) -> /35
- U1 pad 36: /port_id -> /36
- U1 pad 37: unconnected-(U1-PB10-Pad37) -> /37
- U1 pad 38: +3.3V -> /38
- U1 pad 39: GND -> /39
- U1 pad 4: unconnected-(U1-PB15-Pad4) -> /4
- U1 pad 40: +5V -> /40
- U1 pad 5: unconnected-(U1-PA8-Pad5) -> /5
- U1 pad 6: unconnected-(U1-PA9-Pad6) -> /6
- U1 pad 7: unconnected-(U1-PA10-Pad7) -> /7
- U1 pad 8: unconnected-(U1-PA11-Pad8) -> /8
- U1 pad 9: unconnected-(U1-PA12-Pad9) -> /9
Routing:
- net GND: track 831.0 -> 1128.7 mm, vias 97 -> 127
- net /r4: track 0.00 -> 144.8 mm, vias 0 -> 8
- net +5V: track 781.2 -> 924.3 mm, vias 51 -> 66
- net /cl5: track 0.00 -> 141.3 mm, vias 0 -> 2
- net /cl10: track 99.5 -> 0.00 mm, vias 1 -> 0
- net +3.3V: track 32.5 -> 130.8 mm, vias 0 -> 10
- net Net-(D64-DOUT): track 0.00 -> 43.6 mm, vias 0 -> 5
- net /pc15: track 0.00 -> 43.4 mm, vias 0 -> 2
- net /cl6: track 97.4 -> 140.6 mm, vias 1 -> 2
- net /r3: track 109.4 -> 152.1 mm, vias 6 -> 7
- net /pa0: track 0.00 -> 41.3 mm, vias 0 -> 2
- net /pc14: track 0.00 -> 38.5 mm, vias 0 -> 3
- net /pb8: track 0.00 -> 37.1 mm, vias 0 -> 3
- net /pc13: track 0.00 -> 36.5 mm, vias 0 -> 2
- net /cl7: track 97.6 -> 129.9 mm, vias 1 -> 2
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