File: isokey/isokey.kicad_pcb (KiCad board)
At the start: 2 copper layers, 4.6 x 4.6 mm, 367 parts, among them M1 JOYSTICK-PSP1000, Q2 BSS138, Q3 BSS138, SW1 Cherry, SW10 Cherry, SW11 Cherry, SW12 Cherry, SW13 Cherry, SW14 Cherry, SW15 Cherry, SW16 Cherry, SW17 Cherry, SW18 Cherry, SW19 Cherry, SW2 Cherry, SW20 Cherry, SW21 Cherry, SW22 Cherry, SW23 Cherry, SW24 Cherry, SW25 Cherry, SW26 Cherry, SW27 Cherry, SW28 Cherry, SW29 Cherry, SW3 Cherry, SW30 Cherry, SW31 Cherry, SW32 Cherry, SW33 Cherry, SW34 Cherry, SW35 Cherry, SW36 Cherry, SW37 Cherry, SW38 Cherry, SW39 Cherry, SW4 Cherry, SW40 Cherry, SW41 Cherry, SW42 Cherry, SW43 Cherry, SW44 Cherry, SW45 Cherry, SW46 Cherry, SW47 Cherry, SW48 Cherry, SW5 Cherry, SW6 Cherry, SW7 Cherry, SW8 Cherry, SW9 Cherry, U1 BlackPill_STLINK, U3 TLV73318PDBV, U4 LP5569, U6 JOYSTICKPTH, U7 JOYSTICKPTH

Commit message: Complete routing
Parts:
- removed C12, C13, C84, C86: 1uF, Capacitor_SMD:C_0805_2012Metric
- removed C85: 100nF, Capacitor_SMD:C_0603_1608Metric_Pad1.08x0.95mm_HandSolder
- removed D101, D102, D103, D104, D105, D106, D107, D108, D109: LED, LED_SMD:LED_0603_1608Metric_Pad1.05x0.95mm_HandSolder
- removed H1, H2, H3: StabilizerHoles, Button_Switch_Keyboard:Stabilizer_MX_2u
- removed M1: JOYSTICK-PSP1000, SparkFun-Electromechanical:JOYSTICK-PSP1000
- removed R45: 10k, Resistor_SMD:R_0603_1608Metric_Pad0.98x0.95mm_HandSolder
- removed U4: LP5569, Package_DFN_QFN:WQFN-24-1EP_4x4mm_P0.5mm_EP2.45x2.45mm_ThermalVias
- added C70: 100nF, Capacitor_SMD:C_0603_1608Metric_Pad1.08x0.95mm_HandSolder, F.Cu at (197.1, 22.7)
- added C71: 1uF, Capacitor_SMD:C_0805_2012Metric, F.Cu at (214.7, 11.4)
- added C72: 100nF, Capacitor_SMD:C_0603_1608Metric_Pad1.08x0.95mm_HandSolder, F.Cu at (222.6, 14.2)
- added C73: 1uF, Capacitor_SMD:C_0805_2012Metric, F.Cu at (232.1, 44.8)
- added C74: 1uF, Capacitor_SMD:C_0805_2012Metric, F.Cu at (213.6, 17.1)
- added C75: 1uF, Capacitor_SMD:C_0805_2012Metric, B.Cu at (232.8, 6.00)
- added D79: LED, LED_SMD:LED_0603_1608Metric_Pad1.05x0.95mm_HandSolder, F.Cu at (214.9, 22.8)
- added D80: LED, LED_SMD:LED_0603_1608Metric_Pad1.05x0.95mm_HandSolder, F.Cu at (218.1, -13.6)
- added D81: LED, LED_SMD:LED_0603_1608Metric_Pad1.05x0.95mm_HandSolder, F.Cu at (218.1, -26.3)
- added D82: LED, LED_SMD:LED_0603_1608Metric_Pad1.05x0.95mm_HandSolder, F.Cu at (218.1, -39.0)
- added D83: LED, LED_SMD:LED_0603_1608Metric_Pad1.05x0.95mm_HandSolder, F.Cu at (218.1, -51.7)
- added D84: LED, LED_SMD:LED_0603_1608Metric_Pad1.05x0.95mm_HandSolder, F.Cu at (228.6, 46.8)
- added D85: LED, LED_SMD:LED_0603_1608Metric_Pad1.05x0.95mm_HandSolder, F.Cu at (218.7, 48.9)
- added D86: LED, LED_SMD:LED_0603_1608Metric_Pad1.05x0.95mm_HandSolder, F.Cu at (207.3, 43.4)
- added D87: LED, LED_SMD:LED_0603_1608Metric_Pad1.05x0.95mm_HandSolder, F.Cu at (207.0, 30.9)
- added J1: PJ-320A-4P, Connector_Audio:Jack_3.5mm_PJ320E_Horizontal, F.Cu at (232.5, -64.2)
- added J2: PJ-320A-4P, Connector_Audio:Jack_3.5mm_PJ320E_Horizontal, B.Cu at (232.5, -68.8)
- added JP41: SolderJumper_3_Open_line, Jumper:SolderJumper-3_P2.0mm_Open_TrianglePad1.0x1.5mm_NumberLabels, B.Cu at (198.6, 20.4)
- added JP42: SolderJumper_3_Open_line, Jumper:SolderJumper-3_P2.0mm_Open_TrianglePad1.0x1.5mm_NumberLabels, F.Cu at (198.6, 20.4)
- added JP45: SolderJumper_3_Open_line, Jumper:SolderJumper-3_P2.0mm_Open_TrianglePad1.0x1.5mm_NumberLabels, B.Cu at (203.9, 17.7)
- added JP46: SolderJumper_3_Open_line, Jumper:SolderJumper-3_P2.0mm_Open_TrianglePad1.0x1.5mm_NumberLabels, F.Cu at (203.9, 17.7)
- added JP47: SolderJumper_3_Open_line, Jumper:SolderJumper-3_P2.0mm_Open_TrianglePad1.0x1.5mm_NumberLabels, B.Cu at (238.8, -68.9)
- added JP48: SolderJumper_3_Open_line, Jumper:SolderJumper-3_P2.0mm_Open_TrianglePad1.0x1.5mm_NumberLabels, B.Cu at (238.8, -64.1)
- added JP49: SolderJumper_3_Open_line, Jumper:SolderJumper-3_P2.0mm_Open_TrianglePad1.0x1.5mm_NumberLabels, F.Cu at (238.8, -68.9)
- added JP50: SolderJumper_3_Open_line, Jumper:SolderJumper-3_P2.0mm_Open_TrianglePad1.0x1.5mm_NumberLabels, F.Cu at (238.8, -64.1)
- added R14: 10k, Resistor_SMD:R_0603_1608Metric_Pad0.98x0.95mm_HandSolder, B.Cu at (208.4, 13.5)
- added R16: 10k, Resistor_SMD:R_0603_1608Metric_Pad0.98x0.95mm_HandSolder, B.Cu at (206.8, 14.4)
- added R24: 10k, Resistor_SMD:R_0603_1608Metric_Pad0.98x0.95mm_HandSolder, F.Cu at (221.0, 15.1)
- added R26: 10k, Resistor_SMD:R_0603_1608Metric_Pad0.98x0.95mm_HandSolder, F.Cu at (215.9, 13.5)
- added R65: 10k, Resistor_SMD:R_0603_1608Metric_Pad0.98x0.95mm_HandSolder, F.Cu at (215.9, 19.0)
- added U8: ~, Package_DFN_QFN:WQFN-24-1EP_4x4mm_P0.5mm_EP2.45x2.45mm_ThermalVias, F.Cu at (219.8, 9.20)
- added U9: TLV73318PDBV, Package_TO_SOT_SMD:SOT-23-5, F.Cu at (218.5, 17.5)
- C10, C7, C87, C88, C89, D110, D111, D112, D113, D114, D115, D116, D117, D118, JP44, R18, R46, R47, R58, R60, U3, U5: moved to B.Cu
- moved D115 142.0 mm to (228.6, 46.8), turned to 30 degrees
- moved D116 134.5 mm to (218.7, 48.9), turned to -15 degrees
- moved C89 132.2 mm to (232.1, 44.8), turned to 30 degrees
- moved C88 130.5 mm to (229.4, 9.95), turned to -60 degrees
- moved R46 130.4 mm to (230.9, 9.05), turned to 120 degrees
- moved R47 129.7 mm to (231.8, 4.30), turned to -150 degrees
- moved C87 126.0 mm to (230.6, 2.40), turned to 30 degrees
- moved D114 123.0 mm to (218.1, -51.7), turned to 90 degrees
- moved D117 122.9 mm to (207.3, 43.4), turned to -60 degrees
- moved C10 120.8 mm to (235.9, 4.20), turned to -150 degrees
- moved D113 120.6 mm to (218.1, -39.0), turned to 90 degrees
- moved D112 119.0 mm to (218.1, -26.3), turned to 90 degrees
- moved D110 119.0 mm to (214.9, 22.8), turned to 30 degrees
- moved D118 118.9 mm to (207.0, 30.9), turned to 75 degrees
- moved D111 118.3 mm to (218.1, -13.6), turned to 90 degrees
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Connections:
- D110 pad 1: Net-(D110-K) -> /led_driver/l8
- D111 pad 1: Net-(D111-K) -> /led_driver/l0
- D112 pad 1: Net-(D112-K) -> /led_driver/l1
- D113 pad 1: Net-(D113-K) -> /led_driver/l2
- D114 pad 1: Net-(D114-K) -> /led_driver/l3
- D115 pad 1: Net-(D115-K) -> /led_driver/l4
- D116 pad 1: Net-(D116-K) -> /led_driver/l5
- D117 pad 1: Net-(D117-K) -> /led_driver/l6
- D118 pad 1: Net-(D118-K) -> /led_driver/l7
- JP43 pad 1: +3.3V -> /Interfaces/h1
- JP43 pad 2: /Interfaces/Vb -> GND
- JP43 pad 3: /Interfaces/Vt -> +3.3V
- JP44 pad 1: GND -> /Interfaces/h3
- JP44 pad 2: /Interfaces/gb -> +3.3V
- JP44 pad 3: /Interfaces/gt -> GND
- R15 pad 2: /pa2 -> /pa7
- R17 pad 2: /pa2 -> /pa7
- R5 pad 2: /pa3 -> /pa6
- R7 pad 2: /pa3 -> /pa6
- RSW1 pad S1: /cl0 -> /sw0_r
- RSW1 pad S2: /sw0_r -> /cl0
- U2 pad 1: GND -> Net-(JP42-A)
- U2 pad 2: +3.3V -> Net-(JP41-A)
- U2 pad 3: /led_SCL -> Net-(JP45-A)
- U2 pad 4: /led_SDA -> Net-(JP46-A)
- U5 pad 11: Net-(D118-K) -> /led_driver/l8
- U5 pad 12: Net-(D117-K) -> /led_driver/l7
- U5 pad 13: Net-(D116-K) -> /led_driver/l6
- U5 pad 14: Net-(D115-K) -> /led_driver/l5
- U5 pad 15: Net-(D114-K) -> /led_driver/l4
- U5 pad 16: Net-(D113-K) -> /led_driver/l3
- U5 pad 17: Net-(D112-K) -> /led_driver/l2
- U5 pad 18: Net-(D111-K) -> /led_driver/l1
- U5 pad 19: Net-(D110-K) -> /led_driver/l0
- U5 pad 6: /Led_CLK -> unconnected-(U5-CLK-Pad6)
- U6 pad H1: /Interfaces/Vt -> /Interfaces/h1
- U6 pad H2: /pa3 -> /pa5
- U6 pad H3: /Interfaces/gt -> /Interfaces/h3
- U6 pad V2: /pa2 -> /pb1
- U7 pad H1: /Interfaces/gb -> /Interfaces/h3
- U7 pad H2: /pa3 -> /pa5
- U7 pad H3: /Interfaces/Vb -> /Interfaces/h1
- U7 pad V2: /pa2 -> /pb1
Routing:
- net +5V: track 924.3 -> 1200.6 mm, vias 66 -> 86
- net +3.3V: track 130.8 -> 344.5 mm, vias 10 -> 23
- net GND: track 1128.7 -> 1300.9 mm, vias 127 -> 143
- net /Led_INT: track 0.00 -> 136.3 mm, vias 0 -> 6
- net /pb1: track 9.49 -> 138.5 mm, vias 1 -> 2
- net /led_driver/l4: track 0.00 -> 81.6 mm, vias 0 -> 2
- net /pa5: track 9.49 -> 87.2 mm
- net /cl0: track 109.4 -> 186.3 mm, vias 8 -> 10
- net /ENC1B: track 0.00 -> 71.9 mm, vias 0 -> 5
- net /led_driver/l5: track 0.00 -> 70.1 mm, vias 0 -> 2
- net /led_driver/l3: track 0.00 -> 68.0 mm, vias 0 -> 2
- net /pb12: track 0.00 -> 63.1 mm, vias 1 -> 2
- net /pb7: track 0.00 -> 60.1 mm, vias 1 -> 4
- net /pb13: track 0.00 -> 60.0 mm, vias 1 -> 2
- net /pb6: track 0.00 -> 59.9 mm, vias 1 -> 3
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
Commit message: move oled
Parts:
- moved C10 205.8 mm to (113.2, 169.5)
- moved C11 205.8 mm to (94.1, 180.5)
- moved C22 205.8 mm to (163.6, 131.5)
- moved C24 205.8 mm to (131.1, 149.6)
- moved C25 205.8 mm to (150.2, 149.6)
- moved C28 205.8 mm to (207.3, 149.6)
- moved C29 205.8 mm to (144.3, 169.5)
- moved C30 205.8 mm to (163.5, 169.6)
- moved C32 205.8 mm to (201.5, 169.5)
- moved C33 205.8 mm to (219.8, 169.5)
- moved C36 205.8 mm to (166.3, 190.6)
- moved C4 205.8 mm to (207.3, 135.6)
- moved C47 205.8 mm to (163.6, 131.5)
- moved C49 205.8 mm to (131.1, 149.6)
- moved C50 205.8 mm to (150.2, 149.6)
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Routing:
- net GND: track 1300.9 -> 1331.4 mm, vias 143 -> 146
- net /ENC1B: track 71.9 -> 57.4 mm
- net +3.3V: track 344.5 -> 336.0 mm
- net +5V: track 1200.6 -> 1207.9 mm
- net Net-(JP45-A): track 2.64 -> 4.22 mm
- net Net-(JP41-A): track 4.03 -> 2.66 mm
- net Net-(JP46-A): track 4.20 -> 3.50 mm
