File: isokey/keyplate.kicad_sch (KiCad schematic)
At the start: 144 parts

Commit message: WIP
Changed lines of the file:
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@@
   (junction (at 68.58 77.47) (diameter 0) (color 0 0 0 0)
   )
-  (junction (at 121.92 147.32) (diameter 0) (color 0 0 0 0)
-  )
   (junction (at 203.2 107.95) (diameter 0) (color 0 0 0 0)
   )
   (junction (at 110.49 129.54) (diameter 0) (color 0 0 0 0)
   )
-  (junction (at 191.77 41.91) (diameter 0) (color 0 0 0 0)
-  )
   (junction (at 231.14 120.65) (diameter 0) (color 0 0 0 0)
   )
@@
     (stroke (width 0) (type default))
   )
-  (wire (pts (xy 121.92 147.32) (xy 121.92 149.86))
+  (wire (pts (xy 121.92 129.54) (xy 121.92 149.86))
     (stroke (width 0) (type default))
   )
@@
     (stroke (width 0) (type default))
   )
-  (wire (pts (xy 191.77 41.91) (xy 191.77 64.77))
+  (wire (pts (xy 191.77 35.56) (xy 191.77 64.77))
     (stroke (width 0) (type default))
   )
@@
     (stroke (width 0) (type default))
   )
-  (wire (pts (xy 121.92 129.54) (xy 121.92 147.32))
-    (stroke (width 0) (type default))
-  )
   (wire (pts (xy 110.49 107.95) (xy 110.49 129.54))
     (stroke (width 0) (type default))
@@
     (stroke (width 0) (type default))
   )
-  (wire (pts (xy 191.77 41.91) (xy 195.58 41.91))
-    (stroke (width 0) (type default))
-  )
   (wire (pts (xy 110.49 64.77) (xy 110.49 86.36))
     (stroke (width 0) (type default))
@@
     (stroke (width 0) (type default))
   )
-  (wire (pts (xy 121.92 147.32) (xy 124.46 147.32))
-    (stroke (width 0) (type default))
-  )
   (wire (pts (xy 173.99 99.06) (xy 185.42 99.06))
     (stroke (width 0) (type default))
@@
   )
   (wire (pts (xy 45.72 142.24) (xy 68.58 142.24))
-    (stroke (width 0) (type default))
-  )
-  (wire (pts (xy 191.77 35.56) (xy 191.77 41.91))
     (stroke (width 0) (type default))
   )
@@
     (effects (font (size 1.27 1.27)) (justify left))
   )
-  (hierarchical_label "sw1_c" (shape input) (at 124.46 147.32 0) (fields_autoplaced)
-    (effects (font (size 1.27 1.27)) (justify left))
-  )
-  (hierarchical_label "sw0_c" (shape input) (at 195.58 41.91 0) (fields_autoplaced)
-    (effects (font (size 1.27 1.27)) (justify left))
-  )

Commit message: isokey: start splitting
Parts:
- removed D? (x72): 1N4448W, Diode_SMD:D_SOD-123, symbol Diode:1N4448W
- removed SW? (x70): Cherry, Button_Switch_Keyboard:Kailh_socket_MX_LED, symbol Switch:SW_Push_45deg
- added D? (x48): 1N4448W, Diode_SMD:D_SOD-123, symbol Diode:1N4448W
- added SW? (x47): Cherry, Button_Switch_Keyboard:Kailh_socket_MX_LED, symbol Switch:SW_Push_45deg
Connections:
- net cl0: now also SW?.1, SW?.1, SW?.1, SW?.2, SW?.2, SW?.2, SW?.2
- net cl1: now also SW?.1, SW?.1, SW?.1, SW?.1, SW?.1, SW?.2, SW?.2, SW?.2, SW?.2, SW?.2
- net cl2: now also SW?.1, SW?.1, SW?.1, SW?.1, SW?.1, SW?.2, SW?.2, SW?.2, SW?.2, SW?.2
- net cl3: now also SW?.1, SW?.1, SW?.1, SW?.1, SW?.1, SW?.2, SW?.2, SW?.2, SW?.2, SW?.2
- net cl4: now also SW?.1, SW?.1, SW?.1, SW?.1, SW?.1, SW?.2, SW?.2, SW?.2, SW?.2, SW?.2
- net r0: now also D?.2 (A), D?.2 (A), D?.2 (A), D?.2 (A), D?.2 (A), D?.2 (A), D?.2 (A), D?.2 (A), D?.2 (A)
- net r1: now also D?.2 (A), D?.2 (A), D?.2 (A), D?.2 (A), D?.2 (A), D?.2 (A), D?.2 (A), D?.2 (A), D?.2 (A), D?.2 (A)
- net r2: now also D?.2 (A), D?.2 (A), D?.2 (A), D?.2 (A), D?.2 (A), D?.2 (A), D?.2 (A), D?.2 (A), D?.2 (A), D?.2 (A)
- net r3: now also D?.2 (A), D?.2 (A), D?.2 (A), D?.2 (A), D?.2 (A), D?.2 (A), D?.2 (A), D?.2 (A), D?.2 (A), D?.2 (A)
- net r4: now also D?.2 (A), D?.2 (A), D?.2 (A), D?.2 (A), D?.2 (A), D?.2 (A), D?.2 (A), D?.2 (A), D?.2 (A)
- new net: D?.1 (K), SW?.2 (x23)
- new net: D?.1 (K), SW?.1 (x24)

Commit message: Continue routing
Connections:
- net sw0_r: now reaches D?.1 (K)
Changed lines of the file:
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@@
     (company "IsoKey - asterix24@gmail.com")
   )
-  (junction (at 52.07 149.86) (diameter 0) (color 0 0 0 0)
-  )
   (junction (at 98.425 120.65) (diameter 0) (color 0 0 0 0)
   )
@@
     (stroke (width 0) (type default))
   )
-  (wire (pts (xy 52.07 149.86) (xy 52.07 193.04))
-    (stroke (width 0) (type default))
-  )
   (wire (pts (xy 103.505 129.54) (xy 103.505 149.86))
     (stroke (width 0) (type default))
@@
     (stroke (width 0) (type default))
   )
-  (wire (pts (xy 52.07 129.54) (xy 52.07 149.86))
+  (wire (pts (xy 52.07 129.54) (xy 52.07 193.04))
     (stroke (width 0) (type default))
   )
@@
     (stroke (width 0) (type default))
   )
+  (wire (pts (xy 47.625 154.94) (xy 56.515 154.94))
+    (stroke (width 0) (type default))
+  )
   (wire (pts (xy 81.28 162.56) (xy 91.44 162.56))
     (stroke (width 0) (type default))
@@
   )
   (wire (pts (xy 98.425 77.47) (xy 108.585 77.47))
-    (stroke (width 0) (type default))
-  )
-  (wire (pts (xy 52.07 149.86) (xy 53.975 149.86))
     (stroke (width 0) (type default))
   )
@@
     (effects (font (size 1.27 1.27)) (justify left))
   )
-  (hierarchical_label "sw0_r" (shape input) (at 53.975 149.86 0) (fields_autoplaced)
-    (effects (font (size 1.27 1.27)) (justify left))
+  (hierarchical_label "sw0_r" (shape input) (at 47.625 154.94 180) (fields_autoplaced)
+    (effects (font (size 1.27 1.27)) (justify right))
   )
   (hierarchical_label "r1" (shape input) (at 29.845 99.06 180) (fields_autoplaced)

Commit message: Continue routing
Parts:
- added D?: 1N4448W, Diode_SMD:D_SOD-123, symbol Diode:1N4448W
Connections:
- net r4: now also D?.2 (A)
- net sw0_r: now also D?.1 (K)
Changed lines of the file:
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@@
   (junction (at 57.15 142.24) (diameter 0) (color 0 0 0 0)
   )
+  (junction (at 49.276 154.94) (diameter 0) (color 0 0 0 0)
+  )
   (junction (at 46.99 99.06) (diameter 0) (color 0 0 0 0)
   )
@@
   (junction (at 52.07 86.36) (diameter 0) (color 0 0 0 0)
   )
+  (junction (at 49.276 162.56) (diameter 0) (color 0 0 0 0)
+  )
   (junction (at 69.215 64.77) (diameter 0) (color 0 0 0 0)
   )
@@
     (stroke (width 0) (type default))
   )
-  (wire (pts (xy 47.625 154.94) (xy 56.515 154.94))
+  (wire (pts (xy 47.625 154.94) (xy 49.276 154.94))
     (stroke (width 0) (type default))
   )
@@
     (stroke (width 0) (type default))
   )
-  (wire (pts (xy 29.845 162.56) (xy 56.515 162.56))
+  (wire (pts (xy 29.845 162.56) (xy 49.276 162.56))
     (stroke (width 0) (type default))
   )
@@
     (stroke (width 0) (type default))
   )
+  (wire (pts (xy 49.276 154.94) (xy 56.515 154.94))
+    (stroke (width 0) (type default))
+  )
   (wire (pts (xy 52.07 64.77) (xy 52.07 86.36))
     (stroke (width 0) (type default))
@@
   )
   (wire (pts (xy 120.65 64.77) (xy 120.65 86.36))
+    (stroke (width 0) (type default))
+  )
+  (wire (pts (xy 49.276 162.56) (xy 56.515 162.56))
     (stroke (width 0) (type default))
   )
@@
         )
       )
+    )
+  )
+  (symbol (lib_id "Diode:1N4448W") (at 49.276 158.75 270) (unit 1)
+    (in_bom yes) (on_board yes) (dnp no)
+    (property "Reference" "D?" (at 42.672 159.004 90)
+      (effects (font (size 1.27 1.27)) (justify left))
+    )
+    (property "Value" "1N4448W" (at 51.816 160.02 90)
+      (effects (font (size 1.27 1.27)) (justify left) hide)
+    )
+    (property "Footprint" "Diode_SMD:D_SOD-123" (at 44.831 158.75 0)
+      (effects (font (size 1.27 1.27)) hide)
+    )
+    (property "Datasheet" "https://www.vishay.com/docs/85722/1n4448w.pdf" (at 49.276 158.75 0)
+      (effects (font (size 1.27 1.27)) hide)
+    )
+    (property "Sim.Device" "D" (at 49.276 158.75 0)
+      (effects (font (size 1.27 1.27)) hide)
+    )
+    (property "Sim.Pins" "1=K 2=A" (at 49.276 158.75 0)
+      (effects (font (size 1.27 1.27)) hide)
+    )
+    (pin "1")
+    (pin "2")
+    (instances
+      (project "isokey"
+        (path "/b0c352a4-2db1-45ff-8668-f2efdeb7d408"
+          (reference "D?") (unit 1)
+        )
+        (path "/b0c352a4-2db1-45ff-8668-f2efdeb7d408/fdcf2c12-f432-4cc9-a99f-9b8019eb8ce2"
+          (reference "D74") (unit 1)
+        )
+        (path "/b0c352a4-2db1-45ff-8668-f2efdeb7d408/870755d2-ff44-4c69-82b3-4018370ecd52"
+          (reference "D?") (unit 1)
+        )
+      )
