File: isokey/isokey_frame.kicad_pcb (KiCad board)
At the start: 2 copper layers, 363.8 x 161.1 mm, 385 parts, among them J1 PadExp Left, J2 PadExp Right, Q1 BSS138, SW1 Cherry, SW10 Cherry, SW11 Cherry, SW12 Cherry, SW13 Cherry, SW14 Cherry, SW15 Cherry, SW16 Cherry, SW17 Cherry, SW18 Cherry, SW19 Cherry, SW2 Cherry, SW20 Cherry, SW21 Cherry, SW22 Cherry, SW23 Cherry, SW24 Cherry, SW25 Cherry, SW26 Cherry, SW27 Cherry, SW28 Cherry, SW29 Cherry, SW3 Cherry, SW30 Cherry, SW31 Cherry, SW32 Cherry, SW33 Cherry, SW34 Cherry, SW35 Cherry, SW36 Cherry, SW37 Cherry, SW38 Cherry, SW39 Cherry, SW4 Cherry, SW40 Cherry, SW41 Cherry, SW42 Cherry, SW43 Cherry, SW44 Cherry, SW45 Cherry, SW46 Cherry, SW47 Cherry, SW48 Cherry, SW49 Cherry, SW5 Cherry, SW50 Cherry, SW51 Cherry, SW52 Cherry, SW53 Cherry, SW54 Cherry, SW55 Cherry, SW56 Cherry, SW57 Cherry, SW58 Cherry, SW59 Cherry, SW6 Cherry, SW60 Cherry, SW61 Cherry, SW62 Cherry, SW63 Cherry, SW64 Cherry, SW65 Cherry, SW67 Cherry, SW68 Cherry, SW69 Cherry, SW7 Cherry, SW70 Cherry, SW71 Cherry, SW72 Cherry, SW73 RotaryEncoder_Switch, SW74 RotaryEncoder_Switch, SW8 Cherry, SW9 Cherry, U1 BlackPill_STLINK, U2 LP5569, U4 TLV73318PDBV

Commit message: complete routing
Other:
- board size 363.8 x 161.1 mm -> 348 x 144.4 mm

Commit message: Fix for output file
Parts:
- removed C1, C10, C11, C12, C13, C14, C15, C16, C17, C18, C19, C2, C20, C21, C22, C23, C24, C25, C26, C27, C28, C29, C3, C30, C31, C32, C33, C35, C36, C37, C38, C39, C4, C40, C41, C42, C43, C44, C46, C47, C48, C49, C5, C50, C51, C52, C53, C54, C55, C58, C59, C6, C60, C61, C62, C63, C64, C65, C67, C69, C7, C70, C71, C72, C73, C74, C75, C76, C78, C79, C8, C9, C92, C93, C96, C97, C98: 100nF, Capacitor_SMD:C_0603_1608Metric_Pad1.08x0.95mm_HandSolder
- removed C80, C81, C82, C83, C84, C85, C86, C87, C88, C89: 1uF, Capacitor_SMD:C_0805_2012Metric
- removed C90, C91, C94, C95: 10uF, Capacitor_SMD:C_1206_3216Metric
- removed D1, D10, D11, D12, D13, D14, D15, D16, D169, D17, D18, D19, D2, D20, D21, D22, D23, D24, D25, D26, D27, D28, D29, D3, D30, D31, D32, D33, D34, D35, D36, D37, D38, D39, D4, D40, D41, D42, D43, D44, D45, D46, D47, D48, D49, D5, D50, D51, D52, D53, D54, D55, D56, D57, D58, D59, D6, D60, D61, D62, D63, D64, D65, D66, D67, D68, D69, D7, D70, D71, D72, D8, D9: 1N4448W, Diode_SMD:D_SOD-123
- removed D100, D101, D102, D103, D104, D105, D106, D107, D108, D109, D110, D111, D112, D113, D114, D115, D116, D117, D118, D119, D120, D121, D122, D123, D124, D125, D126, D127, D128, D129, D130, D131, D132, D133, D134, D135, D136, D137, D138, D139, D140, D142, D143, D144, D145, D146, D147, D76, D77, D78, D79, D80, D81, D82, D83, D84, D85, D86, D87, D88, D89, D90, D91, D92, D93, D94, D95, D96, D97, D98, D99: SK6812MINI, LED_SMD:LED_SK6812MINI_PLCC4_3.5x3.5mm_P1.75mm
- removed D153, D154, D155, D156, D157, D158, D159, D160, D161, D162, D163, D164, D165, D166, D167, D73, D74, D75: LED, LED_SMD:LED_0603_1608Metric_Pad1.05x0.95mm_HandSolder
- removed H1, H2, H3, H4: StabilizerHoles, Button_Switch_Keyboard:Stabilizer_MX_2u
- removed J1: PadExp Left, Connector_JST:JST_GH_SM14B-GHS-TB_1x14-1MP_P1.25mm_Horizontal
- removed J2: PadExp Right, Connector_JST:JST_GH_SM14B-GHS-TB_1x14-1MP_P1.25mm_Horizontal
- removed Q1: BSS138, Package_TO_SOT_SMD:SOT-23-3
- removed R1, R10, R11, R12, R13, R14, R15, R16, R17, R18, R19, R2, R20, R21, R22, R23, R24, R29, R3, R30, R33, R34, R37, R38, R4, R46, R5, R6, R61, R63, R66, R67, R7, R8, R9: 22R, Resistor_SMD:R_0603_1608Metric_Pad0.98x0.95mm_HandSolder
- removed R25, R26, R27, R28, R31, R32, R35, R36, R59, R64, R65: 10k, Resistor_SMD:R_0603_1608Metric_Pad0.98x0.95mm_HandSolder
- removed R60: 4k7, Resistor_SMD:R_0603_1608Metric_Pad0.98x0.95mm_HandSolder
- removed SW1, SW10, SW11, SW12, SW13, SW14, SW15, SW16, SW17, SW18, SW19, SW2, SW20, SW21, SW22, SW23, SW24, SW25, SW26, SW27, SW28, SW29, SW3, SW30, SW31, SW32, SW33, SW34, SW35, SW36, SW37, SW38, SW39, SW4, SW40, SW41, SW42, SW43, SW44, SW45, SW46, SW47, SW48, SW49, SW5, SW50, SW51, SW52, SW53, SW54, SW55, SW56, SW57, SW58, SW59, SW6, SW60, SW61, SW62, SW63, SW64, SW65, SW67, SW68, SW69, SW7, SW70, SW71, SW72, SW8, SW9: Cherry, Button_Switch_Keyboard:Kailh_socket_MX_LED
- removed SW73, SW74: RotaryEncoder_Switch, Rotary_Encoder:RotaryEncoder_Alps_EC12E-Switch_Vertical_H20mm_CircularMountingHoles
- removed U1: BlackPill_STLINK, Module:BlackPill
- removed U2: LP5569, Package_DFN_QFN:WQFN-24-1EP_4x4mm_P0.5mm_EP2.45x2.45mm_ThermalVias
- removed U3: ~, Package_DFN_QFN:WQFN-24-1EP_4x4mm_P0.5mm_EP2.45x2.45mm_ThermalVias
- removed U4: TLV73318PDBV, Package_TO_SOT_SMD:SOT-23-5
- removed U5: ~, Display:OLED_Display_128x32_SSD1306_i2c
Routing:
- net GND: track 3717.6 -> 0.00 mm, vias 306 -> 0
- net +5V: track 2718.7 -> 0.00 mm, vias 181 -> 0
- net /r4: track 655.7 -> 0.00 mm, vias 5 -> 0
- net /r3: track 585.1 -> 0.00 mm, vias 7 -> 0
- net /r2: track 559.9 -> 0.00 mm, vias 7 -> 0
- net /cl14: track 553.4 -> 0.00 mm, vias 9 -> 0
- net /cl15: track 544.0 -> 0.00 mm, vias 12 -> 0
- net +3.3V: track 524.5 -> 0.00 mm, vias 15 -> 0
- net /r1: track 522.5 -> 0.00 mm, vias 7 -> 0
- net /cl0: track 494.2 -> 0.00 mm, vias 9 -> 0
- net /r0: track 473.6 -> 0.00 mm, vias 7 -> 0
- net /r-1: track 411.1 -> 0.00 mm, vias 6 -> 0
- net Net-(D121-DOUT): track 398.1 -> 0.00 mm
- net Net-(D135-DOUT): track 395.1 -> 0.00 mm
- net /cl1: track 387.9 -> 0.00 mm, vias 7 -> 0
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Other:
- board size 348 x 144.4 mm -> 363.8 x 149.2 mm
- board text added: "DB"
- board text added: "Rev.A"

Commit message: Reoder prj. Complete routing fix drc.
Parts:
- added C1: 1uF, Capacitor_SMD:C_0805_2012Metric, F.Cu at (107.7, 161.2)
- added C10: 1uF, Capacitor_SMD:C_0805_2012Metric, B.Cu at (113.2, 169.5)
- added C11: 1uF, Capacitor_SMD:C_0805_2012Metric, F.Cu at (94.1, 180.5)
- added C14: 100nF, Capacitor_SMD:C_0603_1608Metric_Pad1.08x0.95mm_HandSolder, F.Cu at (131.1, 111.5)
- added C15: 100nF, Capacitor_SMD:C_0603_1608Metric_Pad1.08x0.95mm_HandSolder, B.Cu at (150.3, 111.5)
- added C16: 100nF, Capacitor_SMD:C_0603_1608Metric_Pad1.08x0.95mm_HandSolder, B.Cu at (169.2, 111.5)
- added C17: 100nF, Capacitor_SMD:C_0603_1608Metric_Pad1.08x0.95mm_HandSolder, F.Cu at (188.3, 111.5)
- added C18: 100nF, Capacitor_SMD:C_0603_1608Metric_Pad1.08x0.95mm_HandSolder, B.Cu at (207.3, 111.5)
- added C19: 100nF, Capacitor_SMD:C_0603_1608Metric_Pad1.08x0.95mm_HandSolder, B.Cu at (219.8, 131.5)
- added C2: 10uF, Capacitor_SMD:C_1206_3216Metric, F.Cu at (105.4, 160.6)
- added C20: 100nF, Capacitor_SMD:C_0603_1608Metric_Pad1.08x0.95mm_HandSolder, F.Cu at (201.7, 131.4)
- added C21: 100nF, Capacitor_SMD:C_0603_1608Metric_Pad1.08x0.95mm_HandSolder, B.Cu at (182.6, 131.4)
- added C22: 100nF, Capacitor_SMD:C_0603_1608Metric_Pad1.08x0.95mm_HandSolder, B.Cu at (163.6, 131.5)
- added C23: 100nF, Capacitor_SMD:C_0603_1608Metric_Pad1.08x0.95mm_HandSolder, F.Cu at (144.6, 131.4)
- added C24: 100nF, Capacitor_SMD:C_0603_1608Metric_Pad1.08x0.95mm_HandSolder, B.Cu at (131.1, 149.6)
- added C25: 100nF, Capacitor_SMD:C_0603_1608Metric_Pad1.08x0.95mm_HandSolder, B.Cu at (150.2, 149.6)
- added C26: 100nF, Capacitor_SMD:C_0603_1608Metric_Pad1.08x0.95mm_HandSolder, F.Cu at (169.2, 149.6)
- added C27: 100nF, Capacitor_SMD:C_0603_1608Metric_Pad1.08x0.95mm_HandSolder, F.Cu at (188.3, 149.6)
- added C28: 100nF, Capacitor_SMD:C_0603_1608Metric_Pad1.08x0.95mm_HandSolder, B.Cu at (207.3, 149.6)
- added C29: 100nF, Capacitor_SMD:C_0603_1608Metric_Pad1.08x0.95mm_HandSolder, F.Cu at (144.3, 169.5)
- added C3: 1uF, Capacitor_SMD:C_0805_2012Metric, F.Cu at (116.9, 98.8)
- added C30: 100nF, Capacitor_SMD:C_0603_1608Metric_Pad1.08x0.95mm_HandSolder, F.Cu at (163.5, 169.6)
- added C31: 100nF, Capacitor_SMD:C_0603_1608Metric_Pad1.08x0.95mm_HandSolder, F.Cu at (182.4, 169.5)
- added C32: 100nF, Capacitor_SMD:C_0603_1608Metric_Pad1.08x0.95mm_HandSolder, B.Cu at (201.5, 169.5)
- added C33: 100nF, Capacitor_SMD:C_0603_1608Metric_Pad1.08x0.95mm_HandSolder, B.Cu at (219.8, 169.5)
- added C34: 100nF, Capacitor_SMD:C_0603_1608Metric_Pad1.08x0.95mm_HandSolder, F.Cu at (112.9, 187.5)
- added C35: 100nF, Capacitor_SMD:C_0603_1608Metric_Pad1.08x0.95mm_HandSolder, F.Cu at (142.2, 194.9)
- added C36: 100nF, Capacitor_SMD:C_0603_1608Metric_Pad1.08x0.95mm_HandSolder, F.Cu at (166.3, 190.6)
- added C37: 100nF, Capacitor_SMD:C_0603_1608Metric_Pad1.08x0.95mm_HandSolder, F.Cu at (190.2, 190.6)
- added C38: 1uF, Capacitor_SMD:C_0805_2012Metric, B.Cu at (107.7, 161.2)
- added C39: 100nF, Capacitor_SMD:C_0603_1608Metric_Pad1.08x0.95mm_HandSolder, B.Cu at (131.1, 111.5)
- added C4: 10uF, Capacitor_SMD:C_1206_3216Metric, F.Cu at (207.3, 135.6)
- added C40: 100nF, Capacitor_SMD:C_0603_1608Metric_Pad1.08x0.95mm_HandSolder, F.Cu at (150.3, 111.5)
- added C41: 100nF, Capacitor_SMD:C_0603_1608Metric_Pad1.08x0.95mm_HandSolder, F.Cu at (169.2, 111.5)
- added C42: 100nF, Capacitor_SMD:C_0603_1608Metric_Pad1.08x0.95mm_HandSolder, B.Cu at (188.3, 111.5)
- added C43: 100nF, Capacitor_SMD:C_0603_1608Metric_Pad1.08x0.95mm_HandSolder, F.Cu at (207.3, 111.5)
- added C44: 100nF, Capacitor_SMD:C_0603_1608Metric_Pad1.08x0.95mm_HandSolder, F.Cu at (219.8, 131.5)
- added C45: 100nF, Capacitor_SMD:C_0603_1608Metric_Pad1.08x0.95mm_HandSolder, B.Cu at (201.7, 131.4)
- added C46: 100nF, Capacitor_SMD:C_0603_1608Metric_Pad1.08x0.95mm_HandSolder, F.Cu at (182.6, 131.4)
- added C47: 100nF, Capacitor_SMD:C_0603_1608Metric_Pad1.08x0.95mm_HandSolder, F.Cu at (163.6, 131.5)
- added C48: 100nF, Capacitor_SMD:C_0603_1608Metric_Pad1.08x0.95mm_HandSolder, B.Cu at (144.6, 131.4)
- added C49: 100nF, Capacitor_SMD:C_0603_1608Metric_Pad1.08x0.95mm_HandSolder, F.Cu at (131.1, 149.6)
- added C5: 10uF, Capacitor_SMD:C_1206_3216Metric, B.Cu at (130.4, 179.5)
- added C50: 100nF, Capacitor_SMD:C_0603_1608Metric_Pad1.08x0.95mm_HandSolder, F.Cu at (150.2, 149.6)
- added C51: 100nF, Capacitor_SMD:C_0603_1608Metric_Pad1.08x0.95mm_HandSolder, B.Cu at (169.2, 149.6)
- added C52: 100nF, Capacitor_SMD:C_0603_1608Metric_Pad1.08x0.95mm_HandSolder, B.Cu at (188.3, 149.6)
- added C53: 100nF, Capacitor_SMD:C_0603_1608Metric_Pad1.08x0.95mm_HandSolder, F.Cu at (207.3, 149.6)
- added C54: 100nF, Capacitor_SMD:C_0603_1608Metric_Pad1.08x0.95mm_HandSolder, B.Cu at (144.3, 169.5)
- added C55: 100nF, Capacitor_SMD:C_0603_1608Metric_Pad1.08x0.95mm_HandSolder, B.Cu at (163.5, 169.6)
- added C56: 100nF, Capacitor_SMD:C_0603_1608Metric_Pad1.08x0.95mm_HandSolder, B.Cu at (182.4, 169.5)
- added C57: 100nF, Capacitor_SMD:C_0603_1608Metric_Pad1.08x0.95mm_HandSolder, F.Cu at (201.5, 169.5)
- added C58: 100nF, Capacitor_SMD:C_0603_1608Metric_Pad1.08x0.95mm_HandSolder, F.Cu at (219.8, 169.5)
- added C59: 100nF, Capacitor_SMD:C_0603_1608Metric_Pad1.08x0.95mm_HandSolder, B.Cu at (112.9, 187.5)
- added C6: 10uF, Capacitor_SMD:C_1206_3216Metric, B.Cu at (121.9, 98.8)
- added C60: 100nF, Capacitor_SMD:C_0603_1608Metric_Pad1.08x0.95mm_HandSolder, B.Cu at (142.2, 194.9)
- added C61: 100nF, Capacitor_SMD:C_0603_1608Metric_Pad1.08x0.95mm_HandSolder, B.Cu at (166.3, 190.6)
- added C62: 100nF, Capacitor_SMD:C_0603_1608Metric_Pad1.08x0.95mm_HandSolder, B.Cu at (190.2, 190.6)
- added C63: 10uF, Capacitor_SMD:C_1206_3216Metric, B.Cu at (105.4, 160.6)
- added C64: 1uF, Capacitor_SMD:C_0805_2012Metric, B.Cu at (116.9, 98.8)
- added C65: 10uF, Capacitor_SMD:C_1206_3216Metric, B.Cu at (207.3, 135.6)
- added C66: 10uF, Capacitor_SMD:C_1206_3216Metric, F.Cu at (130.4, 179.5)
- added C67: 10uF, Capacitor_SMD:C_1206_3216Metric, F.Cu at (121.9, 98.8)
- added C68: 100nF, Capacitor_SMD:C_0603_1608Metric_Pad1.08x0.95mm_HandSolder, F.Cu at (97.4, 187.1)
- added C69: 100nF, Capacitor_SMD:C_0603_1608Metric_Pad1.08x0.95mm_HandSolder, B.Cu at (97.4, 187.1)
- added C7: 100nF, Capacitor_SMD:C_0603_1608Metric_Pad1.08x0.95mm_HandSolder, B.Cu at (74.5, 188.0)
- added C70: 100nF, Capacitor_SMD:C_0603_1608Metric_Pad1.08x0.95mm_HandSolder, F.Cu at (74.5, 188.0)
- added C71: 1uF, Capacitor_SMD:C_0805_2012Metric, F.Cu at (92.0, 176.7)
- added C72: 100nF, Capacitor_SMD:C_0603_1608Metric_Pad1.08x0.95mm_HandSolder, F.Cu at (100.0, 179.5)
- added C73: 1uF, Capacitor_SMD:C_0805_2012Metric, F.Cu at (109.4, 210.1)
- added C74: 1uF, Capacitor_SMD:C_0805_2012Metric, F.Cu at (90.9, 182.4)
- added C75: 1uF, Capacitor_SMD:C_0805_2012Metric, B.Cu at (110.1, 171.3)
- added C8: 100nF, Capacitor_SMD:C_0603_1608Metric_Pad1.08x0.95mm_HandSolder, B.Cu at (87.0, 192.1)
- added C87: 1uF, Capacitor_SMD:C_0805_2012Metric, B.Cu at (107.9, 167.7)
- added C88: 100nF, Capacitor_SMD:C_0603_1608Metric_Pad1.08x0.95mm_HandSolder, B.Cu at (106.7, 175.3)
- added C89: 1uF, Capacitor_SMD:C_0805_2012Metric, B.Cu at (109.4, 210.1)
- added C9: 100nF, Capacitor_SMD:C_0603_1608Metric_Pad1.08x0.95mm_HandSolder, F.Cu at (87.0, 192.1)
- added D1: 1N4448W, Diode_SMD:D_SOD-123, B.Cu at (146.7, 112.1)
- added D10: 1N4448W, Diode_SMD:D_SOD-123, F.Cu at (221.1, 112.1)
- added D11: 1N4448W, Diode_SMD:D_SOD-123, B.Cu at (146.7, 131.1)
- added D110: LED, LED_SMD:LED_0603_1608Metric_Pad1.05x0.95mm_HandSolder, B.Cu at (92.2, 188.1)
- added D111: LED, LED_SMD:LED_0603_1608Metric_Pad1.05x0.95mm_HandSolder, B.Cu at (95.4, 151.7)
- added D112: LED, LED_SMD:LED_0603_1608Metric_Pad1.05x0.95mm_HandSolder, B.Cu at (95.4, 139.0)
- added D113: LED, LED_SMD:LED_0603_1608Metric_Pad1.05x0.95mm_HandSolder, B.Cu at (95.4, 126.3)
- added D114: LED, LED_SMD:LED_0603_1608Metric_Pad1.05x0.95mm_HandSolder, B.Cu at (95.4, 113.6)
- added D115: LED, LED_SMD:LED_0603_1608Metric_Pad1.05x0.95mm_HandSolder, B.Cu at (105.9, 212.1)
- added D116: LED, LED_SMD:LED_0603_1608Metric_Pad1.05x0.95mm_HandSolder, B.Cu at (96.0, 214.2)
- added D117: LED, LED_SMD:LED_0603_1608Metric_Pad1.05x0.95mm_HandSolder, B.Cu at (84.6, 208.7)
- added D118: LED, LED_SMD:LED_0603_1608Metric_Pad1.05x0.95mm_HandSolder, B.Cu at (84.3, 196.2)
- added D119: 1N4448W, Diode_SMD:D_SOD-123, B.Cu at (221.1, 150.2)
- added D12: 1N4448W, Diode_SMD:D_SOD-123, F.Cu at (146.7, 131.1)
- added D120: 1N4448W, Diode_SMD:D_SOD-123, F.Cu at (221.1, 150.2)
- added D121: 1N4448W, Diode_SMD:D_SOD-123, B.Cu at (146.7, 169.2)
- added D122: 1N4448W, Diode_SMD:D_SOD-123, F.Cu at (146.7, 169.2)
- added D123: 1N4448W, Diode_SMD:D_SOD-123, B.Cu at (165.8, 169.2)
- added D124: 1N4448W, Diode_SMD:D_SOD-123, F.Cu at (165.8, 169.2)
- added D125: 1N4448W, Diode_SMD:D_SOD-123, B.Cu at (184.8, 169.2)
- added D126: 1N4448W, Diode_SMD:D_SOD-123, F.Cu at (184.8, 169.2)
- added D127: 1N4448W, Diode_SMD:D_SOD-123, B.Cu at (203.9, 169.2)
- added D128: 1N4448W, Diode_SMD:D_SOD-123, F.Cu at (203.9, 169.2)
- added D129: 1N4448W, Diode_SMD:D_SOD-123, B.Cu at (222.1, 169.2)
- added D13: 1N4448W, Diode_SMD:D_SOD-123, B.Cu at (165.8, 131.1)
- added D130: 1N4448W, Diode_SMD:D_SOD-123, F.Cu at (222.1, 169.2)
- added D131: 1N4448W, Diode_SMD:D_SOD-123, B.Cu at (120.5, 198.8)
- added D132: 1N4448W, Diode_SMD:D_SOD-123, F.Cu at (120.5, 198.8)
- added D133: 1N4448W, Diode_SMD:D_SOD-123, B.Cu at (156.5, 191.8)
- added D134: 1N4448W, Diode_SMD:D_SOD-123, F.Cu at (156.5, 191.8)
- added D135: 1N4448W, Diode_SMD:D_SOD-123, B.Cu at (181.9, 191.1)
- added D136: 1N4448W, Diode_SMD:D_SOD-123, F.Cu at (181.9, 191.1)
- added D137: 1N4448W, Diode_SMD:D_SOD-123, B.Cu at (205.8, 191.1)
- added D138: 1N4448W, Diode_SMD:D_SOD-123, F.Cu at (205.8, 191.1)
- added D14: 1N4448W, Diode_SMD:D_SOD-123, F.Cu at (165.8, 131.1)
- added D15: 1N4448W, Diode_SMD:D_SOD-123, B.Cu at (184.8, 131.1)
- added D16: 1N4448W, Diode_SMD:D_SOD-123, F.Cu at (184.8, 131.1)
- added D17: 1N4448W, Diode_SMD:D_SOD-123, B.Cu at (203.9, 131.1)
- added D18: 1N4448W, Diode_SMD:D_SOD-123, F.Cu at (203.9, 131.1)
- added D19: 1N4448W, Diode_SMD:D_SOD-123, B.Cu at (222.1, 131.1)
- added D2: 1N4448W, Diode_SMD:D_SOD-123, F.Cu at (146.7, 112.1)
- added D20: 1N4448W, Diode_SMD:D_SOD-123, F.Cu at (222.1, 131.1)
- added D21: 1N4448W, Diode_SMD:D_SOD-123, B.Cu at (146.7, 150.2)
- added D22: 1N4448W, Diode_SMD:D_SOD-123, F.Cu at (146.7, 150.2)
- added D23: 1N4448W, Diode_SMD:D_SOD-123, B.Cu at (165.8, 150.2)
- added D24: 1N4448W, Diode_SMD:D_SOD-123, F.Cu at (165.8, 150.2)
- added D25: 1N4448W, Diode_SMD:D_SOD-123, B.Cu at (114.0, 206.2)
- added D26: 1N4448W, Diode_SMD:D_SOD-123, B.Cu at (184.8, 150.2)
- added D27: 1N4448W, Diode_SMD:D_SOD-123, F.Cu at (184.8, 150.2)
- added D28: 1N4448W, Diode_SMD:D_SOD-123, B.Cu at (203.9, 150.2)
- added D29: 1N4448W, Diode_SMD:D_SOD-123, F.Cu at (203.9, 150.2)
- added D3: 1N4448W, Diode_SMD:D_SOD-123, B.Cu at (165.8, 112.1)
- added D30: SK6812MINI-E, LED_SMD:LED_SK6812MINI_PLCC4_3.5x3.5mm_P1.75mm, B.Cu at (138.3, 112.3)
- added D31: SK6812MINI-E, LED_SMD:LED_SK6812MINI_PLCC4_3.5x3.5mm_P1.75mm, F.Cu at (138.3, 112.3)
- added D32: SK6812MINI-E, LED_SMD:LED_SK6812MINI_PLCC4_3.5x3.5mm_P1.75mm, B.Cu at (157.4, 112.3)
- added D33: SK6812MINI-E, LED_SMD:LED_SK6812MINI_PLCC4_3.5x3.5mm_P1.75mm, F.Cu at (157.4, 112.3)
- added D34: SK6812MINI-E, LED_SMD:LED_SK6812MINI_PLCC4_3.5x3.5mm_P1.75mm, B.Cu at (176.4, 112.3)
- added D35: SK6812MINI-E, LED_SMD:LED_SK6812MINI_PLCC4_3.5x3.5mm_P1.75mm, F.Cu at (176.4, 112.3)
- added D36: SK6812MINI-E, LED_SMD:LED_SK6812MINI_PLCC4_3.5x3.5mm_P1.75mm, B.Cu at (195.5, 112.3)
- added D37: SK6812MINI-E, LED_SMD:LED_SK6812MINI_PLCC4_3.5x3.5mm_P1.75mm, F.Cu at (195.5, 112.3)
- added D38: SK6812MINI-E, LED_SMD:LED_SK6812MINI_PLCC4_3.5x3.5mm_P1.75mm, B.Cu at (214.5, 112.3)
- added D39: SK6812MINI-E, LED_SMD:LED_SK6812MINI_PLCC4_3.5x3.5mm_P1.75mm, F.Cu at (214.5, 112.3)
- added D4: 1N4448W, Diode_SMD:D_SOD-123, F.Cu at (165.8, 112.1)
- added D40: SK6812MINI-E, LED_SMD:LED_SK6812MINI_PLCC4_3.5x3.5mm_P1.75mm, B.Cu at (214.5, 131.4)
- added D41: SK6812MINI-E, LED_SMD:LED_SK6812MINI_PLCC4_3.5x3.5mm_P1.75mm, B.Cu at (195.5, 131.4)
- added D42: SK6812MINI-E, LED_SMD:LED_SK6812MINI_PLCC4_3.5x3.5mm_P1.75mm, B.Cu at (176.4, 131.4)
- added D43: SK6812MINI-E, LED_SMD:LED_SK6812MINI_PLCC4_3.5x3.5mm_P1.75mm, F.Cu at (157.4, 131.4)
- added D44: SK6812MINI-E, LED_SMD:LED_SK6812MINI_PLCC4_3.5x3.5mm_P1.75mm, B.Cu at (138.3, 131.4)
- added D45: SK6812MINI-E, LED_SMD:LED_SK6812MINI_PLCC4_3.5x3.5mm_P1.75mm, F.Cu at (214.5, 131.4)
- added D46: SK6812MINI-E, LED_SMD:LED_SK6812MINI_PLCC4_3.5x3.5mm_P1.75mm, F.Cu at (195.5, 131.4)
- added D47: SK6812MINI-E, LED_SMD:LED_SK6812MINI_PLCC4_3.5x3.5mm_P1.75mm, F.Cu at (176.4, 131.4)
- added D48: SK6812MINI-E, LED_SMD:LED_SK6812MINI_PLCC4_3.5x3.5mm_P1.75mm, B.Cu at (157.4, 131.4)
- added D49: SK6812MINI-E, LED_SMD:LED_SK6812MINI_PLCC4_3.5x3.5mm_P1.75mm, F.Cu at (138.3, 131.4)
- added D5: 1N4448W, Diode_SMD:D_SOD-123, B.Cu at (184.8, 112.1)
- added D50: SK6812MINI-E, LED_SMD:LED_SK6812MINI_PLCC4_3.5x3.5mm_P1.75mm, B.Cu at (138.3, 150.4)
- added D51: SK6812MINI-E, LED_SMD:LED_SK6812MINI_PLCC4_3.5x3.5mm_P1.75mm, F.Cu at (157.4, 150.4)
- added D52: SK6812MINI-E, LED_SMD:LED_SK6812MINI_PLCC4_3.5x3.5mm_P1.75mm, B.Cu at (176.4, 150.4)
- added D53: SK6812MINI-E, LED_SMD:LED_SK6812MINI_PLCC4_3.5x3.5mm_P1.75mm, F.Cu at (195.5, 150.4)
- added D54: SK6812MINI-E, LED_SMD:LED_SK6812MINI_PLCC4_3.5x3.5mm_P1.75mm, B.Cu at (214.5, 150.4)
- added D55: SK6812MINI-E, LED_SMD:LED_SK6812MINI_PLCC4_3.5x3.5mm_P1.75mm, F.Cu at (138.3, 150.4)
- added D56: SK6812MINI-E, LED_SMD:LED_SK6812MINI_PLCC4_3.5x3.5mm_P1.75mm, B.Cu at (157.4, 150.4)
- added D57: SK6812MINI-E, LED_SMD:LED_SK6812MINI_PLCC4_3.5x3.5mm_P1.75mm, F.Cu at (176.4, 150.4)
- added D58: SK6812MINI-E, LED_SMD:LED_SK6812MINI_PLCC4_3.5x3.5mm_P1.75mm, B.Cu at (195.5, 150.4)
- added D59: SK6812MINI-E, LED_SMD:LED_SK6812MINI_PLCC4_3.5x3.5mm_P1.75mm, F.Cu at (214.5, 150.4)
- added D6: 1N4448W, Diode_SMD:D_SOD-123, F.Cu at (184.8, 112.1)
- added D60: SK6812MINI-E, LED_SMD:LED_SK6812MINI_PLCC4_3.5x3.5mm_P1.75mm, B.Cu at (214.5, 169.5)
- added D61: SK6812MINI-E, LED_SMD:LED_SK6812MINI_PLCC4_3.5x3.5mm_P1.75mm, F.Cu at (195.5, 169.5)
- added D62: SK6812MINI-E, LED_SMD:LED_SK6812MINI_PLCC4_3.5x3.5mm_P1.75mm, B.Cu at (176.4, 169.5)
- added D63: SK6812MINI-E, LED_SMD:LED_SK6812MINI_PLCC4_3.5x3.5mm_P1.75mm, F.Cu at (157.4, 169.5)
- added D64: SK6812MINI-E, LED_SMD:LED_SK6812MINI_PLCC4_3.5x3.5mm_P1.75mm, B.Cu at (138.3, 169.5)
- added D65: SK6812MINI-E, LED_SMD:LED_SK6812MINI_PLCC4_3.5x3.5mm_P1.75mm, F.Cu at (214.5, 169.5)
- added D66: SK6812MINI-E, LED_SMD:LED_SK6812MINI_PLCC4_3.5x3.5mm_P1.75mm, B.Cu at (195.5, 169.5)
- added D67: SK6812MINI-E, LED_SMD:LED_SK6812MINI_PLCC4_3.5x3.5mm_P1.75mm, F.Cu at (176.4, 169.5)
- added D68: SK6812MINI-E, LED_SMD:LED_SK6812MINI_PLCC4_3.5x3.5mm_P1.75mm, B.Cu at (157.4, 169.5)
- added D69: SK6812MINI-E, LED_SMD:LED_SK6812MINI_PLCC4_3.5x3.5mm_P1.75mm, F.Cu at (138.3, 169.5)
- added D7: 1N4448W, Diode_SMD:D_SOD-123, B.Cu at (203.9, 112.1)
- added D70: SK6812MINI-E, LED_SMD:LED_SK6812MINI_PLCC4_3.5x3.5mm_P1.75mm, F.Cu at (116.8, 192.6)
- added D71: SK6812MINI-E, LED_SMD:LED_SK6812MINI_PLCC4_3.5x3.5mm_P1.75mm, F.Cu at (149.1, 194.0)
- added D72: SK6812MINI-E, LED_SMD:LED_SK6812MINI_PLCC4_3.5x3.5mm_P1.75mm, B.Cu at (173.5, 191.4)
- added D73: SK6812MINI-E, LED_SMD:LED_SK6812MINI_PLCC4_3.5x3.5mm_P1.75mm, F.Cu at (197.4, 191.4)
- added D74: 1N4448W, Diode_SMD:D_SOD-123, F.Cu at (114.0, 206.2)
- added D75: SK6812MINI-E, LED_SMD:LED_SK6812MINI_PLCC4_3.5x3.5mm_P1.75mm, B.Cu at (116.8, 192.6)
- added D76: SK6812MINI-E, LED_SMD:LED_SK6812MINI_PLCC4_3.5x3.5mm_P1.75mm, B.Cu at (149.1, 194.0)
- added D77: SK6812MINI-E, LED_SMD:LED_SK6812MINI_PLCC4_3.5x3.5mm_P1.75mm, F.Cu at (173.5, 191.4)
- added D78: SK6812MINI-E, LED_SMD:LED_SK6812MINI_PLCC4_3.5x3.5mm_P1.75mm, B.Cu at (197.4, 191.4)
- added D79: LED, LED_SMD:LED_0603_1608Metric_Pad1.05x0.95mm_HandSolder, F.Cu at (92.2, 188.1)
- added D8: 1N4448W, Diode_SMD:D_SOD-123, F.Cu at (203.9, 112.1)
- added D80: LED, LED_SMD:LED_0603_1608Metric_Pad1.05x0.95mm_HandSolder, F.Cu at (95.4, 151.7)
- added D81: LED, LED_SMD:LED_0603_1608Metric_Pad1.05x0.95mm_HandSolder, F.Cu at (95.4, 139.0)
- added D82: LED, LED_SMD:LED_0603_1608Metric_Pad1.05x0.95mm_HandSolder, F.Cu at (95.4, 126.3)
- added D83: LED, LED_SMD:LED_0603_1608Metric_Pad1.05x0.95mm_HandSolder, F.Cu at (95.4, 113.6)
- added D84: LED, LED_SMD:LED_0603_1608Metric_Pad1.05x0.95mm_HandSolder, F.Cu at (105.9, 212.1)
- added D85: LED, LED_SMD:LED_0603_1608Metric_Pad1.05x0.95mm_HandSolder, F.Cu at (96.0, 214.2)
- added D86: LED, LED_SMD:LED_0603_1608Metric_Pad1.05x0.95mm_HandSolder, F.Cu at (84.6, 208.7)
- added D87: LED, LED_SMD:LED_0603_1608Metric_Pad1.05x0.95mm_HandSolder, F.Cu at (84.3, 196.2)
- added D9: 1N4448W, Diode_SMD:D_SOD-123, B.Cu at (221.1, 112.1)
- added G***: LOGO, footprints:logo_15x15, F.Cu at (122.8, 161.3)
- added G***: LOGO, footprints:logo_15x15, B.Cu at (124.1, 166.2)
- added H1: MountingHole_Pad, MountingHole:MountingHole_2.5mm_Pad_TopBottom, F.Cu at (221.5, 199.4)
- added H2: MountingHole_Pad, MountingHole:MountingHole_2.5mm_Pad_TopBottom, F.Cu at (98.3, 220.9)
- added H3: MountingHole_Pad, MountingHole:MountingHole_2.5mm_Pad_TopBottom, F.Cu at (74.3, 196.9)
- added H4: StabilizerHoles, Button_Switch_Keyboard:Stabilizer_MX_2u, F.Cu at (121.2, 190.1)
- added H5: MountingHole_Pad, MountingHole:MountingHole_2.5mm_Pad_TopBottom, F.Cu at (90.3, 163.9)
- added H6: MountingHole_Pad, MountingHole:MountingHole_2.5mm_Pad_TopBottom, F.Cu at (91.3, 104.9)
- added H7: MountingHole_Pad, MountingHole:MountingHole_2.5mm_Pad_TopBottom, F.Cu at (221.5, 92.4)
- added J1: PJ-320A-4P, Connector_Audio:Jack_3.5mm_PJ320E_Horizontal, F.Cu at (109.8, 101.1)
- added J2: PJ-320A-4P, Connector_Audio:Jack_3.5mm_PJ320E_Horizontal, B.Cu at (109.8, 96.5)
- added JP1: SolderJumper_3_Open_line, Jumper:SolderJumper-3_P2.0mm_Open_TrianglePad1.0x1.5mm_NumberLabels, F.Cu at (108.0, 109.8)
- added JP10: SolderJumper_3_Open_line, Jumper:SolderJumper-3_P2.0mm_Open_TrianglePad1.0x1.5mm_NumberLabels, F.Cu at (108.0, 130.1)
- added JP11: SolderJumper_3_Open_line, Jumper:SolderJumper-3_P2.0mm_Open_TrianglePad1.0x1.5mm_NumberLabels, F.Cu at (108.0, 132.7)
- added JP12: SolderJumper_3_Open_line, Jumper:SolderJumper-3_P2.0mm_Open_TrianglePad1.0x1.5mm_NumberLabels, F.Cu at (108.0, 135.2)
- added JP13: SolderJumper_3_Open_line, Jumper:SolderJumper-3_P2.0mm_Open_TrianglePad1.0x1.5mm_NumberLabels, F.Cu at (108.0, 137.7)
- added JP14: SolderJumper_3_Open_line, Jumper:SolderJumper-3_P2.0mm_Open_TrianglePad1.0x1.5mm_NumberLabels, F.Cu at (108.0, 140.3)
- added JP15: SolderJumper_3_Open_line, Jumper:SolderJumper-3_P2.0mm_Open_TrianglePad1.0x1.5mm_NumberLabels, F.Cu at (108.0, 142.8)
- added JP16: SolderJumper_3_Open_line, Jumper:SolderJumper-3_P2.0mm_Open_TrianglePad1.0x1.5mm_NumberLabels, F.Cu at (108.0, 145.4)
- added JP17: SolderJumper_3_Open_line, Jumper:SolderJumper-3_P2.0mm_Open_TrianglePad1.0x1.5mm_NumberLabels, F.Cu at (108.0, 147.9)
- added JP18: SolderJumper_3_Open_line, Jumper:SolderJumper-3_P2.0mm_Open_TrianglePad1.0x1.5mm_NumberLabels, F.Cu at (108.0, 150.4)
- added JP19: SolderJumper_3_Open_line, Jumper:SolderJumper-3_P2.0mm_Open_TrianglePad1.0x1.5mm_NumberLabels, F.Cu at (108.0, 153.0)
- added JP2: SolderJumper_3_Open_line, Jumper:SolderJumper-3_P2.0mm_Open_TrianglePad1.0x1.5mm_NumberLabels, F.Cu at (108.0, 107.3)
- added JP20: SolderJumper_3_Open_line, Jumper:SolderJumper-3_P2.0mm_Open_TrianglePad1.0x1.5mm_NumberLabels, F.Cu at (108.0, 155.5)
- added JP21: SolderJumper_3_Open_line, Jumper:SolderJumper-3_P2.0mm_Open_TrianglePad1.0x1.5mm_NumberLabels, B.Cu at (112.0, 155.5)
- added JP22: SolderJumper_3_Open_line, Jumper:SolderJumper-3_P2.0mm_Open_TrianglePad1.0x1.5mm_NumberLabels, B.Cu at (112.0, 153.0)
- added JP23: SolderJumper_3_Open_line, Jumper:SolderJumper-3_P2.0mm_Open_TrianglePad1.0x1.5mm_NumberLabels, B.Cu at (112.0, 150.4)
- added JP24: SolderJumper_3_Open_line, Jumper:SolderJumper-3_P2.0mm_Open_TrianglePad1.0x1.5mm_NumberLabels, B.Cu at (112.0, 147.9)
- added JP25: SolderJumper_3_Open_line, Jumper:SolderJumper-3_P2.0mm_Open_TrianglePad1.0x1.5mm_NumberLabels, B.Cu at (112.0, 145.4)
- added JP26: SolderJumper_3_Open_line, Jumper:SolderJumper-3_P2.0mm_Open_TrianglePad1.0x1.5mm_NumberLabels, B.Cu at (112.0, 142.8)
- added JP27: SolderJumper_3_Open_line, Jumper:SolderJumper-3_P2.0mm_Open_TrianglePad1.0x1.5mm_NumberLabels, B.Cu at (112.0, 140.3)
- added JP28: SolderJumper_3_Open_line, Jumper:SolderJumper-3_P2.0mm_Open_TrianglePad1.0x1.5mm_NumberLabels, B.Cu at (112.0, 137.7)
- added JP29: SolderJumper_3_Open_line, Jumper:SolderJumper-3_P2.0mm_Open_TrianglePad1.0x1.5mm_NumberLabels, B.Cu at (112.0, 135.2)
- added JP3: SolderJumper_3_Open_line, Jumper:SolderJumper-3_P2.0mm_Open_TrianglePad1.0x1.5mm_NumberLabels, F.Cu at (108.0, 112.3)
- added JP30: SolderJumper_3_Open_line, Jumper:SolderJumper-3_P2.0mm_Open_TrianglePad1.0x1.5mm_NumberLabels, B.Cu at (112.0, 132.7)
- added JP31: SolderJumper_3_Open_line, Jumper:SolderJumper-3_P2.0mm_Open_TrianglePad1.0x1.5mm_NumberLabels, B.Cu at (112.0, 130.1)
- added JP32: SolderJumper_3_Open_line, Jumper:SolderJumper-3_P2.0mm_Open_TrianglePad1.0x1.5mm_NumberLabels, B.Cu at (112.0, 127.6)
- added JP33: SolderJumper_3_Open_line, Jumper:SolderJumper-3_P2.0mm_Open_TrianglePad1.0x1.5mm_NumberLabels, B.Cu at (112.0, 125.0)
- added JP34: SolderJumper_3_Open_line, Jumper:SolderJumper-3_P2.0mm_Open_TrianglePad1.0x1.5mm_NumberLabels, B.Cu at (112.0, 122.5)
- added JP35: SolderJumper_3_Open_line, Jumper:SolderJumper-3_P2.0mm_Open_TrianglePad1.0x1.5mm_NumberLabels, B.Cu at (112.0, 120.0)
- added JP36: SolderJumper_3_Open_line, Jumper:SolderJumper-3_P2.0mm_Open_TrianglePad1.0x1.5mm_NumberLabels, B.Cu at (112.0, 117.4)
- added JP37: SolderJumper_3_Open_line, Jumper:SolderJumper-3_P2.0mm_Open_TrianglePad1.0x1.5mm_NumberLabels, B.Cu at (112.0, 114.9)
- added JP38: SolderJumper_3_Open_line, Jumper:SolderJumper-3_P2.0mm_Open_TrianglePad1.0x1.5mm_NumberLabels, B.Cu at (112.0, 112.3)
- added JP39: SolderJumper_3_Open_line, Jumper:SolderJumper-3_P2.0mm_Open_TrianglePad1.0x1.5mm_NumberLabels, B.Cu at (112.0, 109.8)
- added JP4: SolderJumper_3_Open_line, Jumper:SolderJumper-3_P2.0mm_Open_TrianglePad1.0x1.5mm_NumberLabels, F.Cu at (108.0, 114.9)
- added JP40: SolderJumper_3_Open_line, Jumper:SolderJumper-3_P2.0mm_Open_TrianglePad1.0x1.5mm_NumberLabels, B.Cu at (112.0, 107.3)
- added JP41: SolderJumper_3_Open_line, Jumper:SolderJumper-3_P2.0mm_Open_TrianglePad1.0x1.5mm_NumberLabels, B.Cu at (76.0, 185.7)
- added JP42: SolderJumper_3_Open_line, Jumper:SolderJumper-3_P2.0mm_Open_TrianglePad1.0x1.5mm_NumberLabels, F.Cu at (76.0, 185.7)
- added JP43: SolderJumper_3_Open_line, Jumper:SolderJumper-3_P2.0mm_Open_TrianglePad1.0x1.5mm_NumberLabels, F.Cu at (111.6, 201.5)
- added JP44: SolderJumper_3_Open_line, Jumper:SolderJumper-3_P2.0mm_Open_TrianglePad1.0x1.5mm_NumberLabels, B.Cu at (104.3, 188.8)
- added JP45: SolderJumper_3_Open_line, Jumper:SolderJumper-3_P2.0mm_Open_TrianglePad1.0x1.5mm_NumberLabels, B.Cu at (81.2, 183.0)
- added JP46: SolderJumper_3_Open_line, Jumper:SolderJumper-3_P2.0mm_Open_TrianglePad1.0x1.5mm_NumberLabels, F.Cu at (81.2, 183.0)
- added JP47: SolderJumper_3_Open_line, Jumper:SolderJumper-3_P2.0mm_Open_TrianglePad1.0x1.5mm_NumberLabels, B.Cu at (116.1, 96.4)
- added JP48: SolderJumper_3_Open_line, Jumper:SolderJumper-3_P2.0mm_Open_TrianglePad1.0x1.5mm_NumberLabels, B.Cu at (116.1, 101.2)
- added JP49: SolderJumper_3_Open_line, Jumper:SolderJumper-3_P2.0mm_Open_TrianglePad1.0x1.5mm_NumberLabels, F.Cu at (116.1, 96.4)
- added JP5: SolderJumper_3_Open_line, Jumper:SolderJumper-3_P2.0mm_Open_TrianglePad1.0x1.5mm_NumberLabels, F.Cu at (108.0, 117.4)
- added JP50: SolderJumper_3_Open_line, Jumper:SolderJumper-3_P2.0mm_Open_TrianglePad1.0x1.5mm_NumberLabels, F.Cu at (116.1, 101.2)
- added JP6: SolderJumper_3_Open_line, Jumper:SolderJumper-3_P2.0mm_Open_TrianglePad1.0x1.5mm_NumberLabels, F.Cu at (108.0, 120.0)
- added JP7: SolderJumper_3_Open_line, Jumper:SolderJumper-3_P2.0mm_Open_TrianglePad1.0x1.5mm_NumberLabels, F.Cu at (108.0, 122.5)
- added JP8: SolderJumper_3_Open_line, Jumper:SolderJumper-3_P2.0mm_Open_TrianglePad1.0x1.5mm_NumberLabels, F.Cu at (108.0, 125.0)
- added JP9: SolderJumper_3_Open_line, Jumper:SolderJumper-3_P2.0mm_Open_TrianglePad1.0x1.5mm_NumberLabels, F.Cu at (108.0, 127.6)
- added Q2: BSS138, Package_TO_SOT_SMD:SOT-23-3, B.Cu at (122.0, 130.1)
- added Q3: BSS138, Package_TO_SOT_SMD:SOT-23-3, F.Cu at (122.0, 130.1)
- added R1: 4k7, Resistor_SMD:R_0603_1608Metric_Pad0.98x0.95mm_HandSolder, F.Cu at (121.7, 127.4)
- added R10: 22R, Resistor_SMD:R_0603_1608Metric_Pad0.98x0.95mm_HandSolder, B.Cu at (122.0, 152.7)
- added R11: 22R, Resistor_SMD:R_0603_1608Metric_Pad0.98x0.95mm_HandSolder, F.Cu at (122.0, 152.7)
- added R12: 22R, Resistor_SMD:R_0603_1608Metric_Pad0.98x0.95mm_HandSolder, F.Cu at (218.8, 186.3)
- added R13: 22R, Resistor_SMD:R_0603_1608Metric_Pad0.98x0.95mm_HandSolder, F.Cu at (122.6, 136.5)
- added R14: 10k, Resistor_SMD:R_0603_1608Metric_Pad0.98x0.95mm_HandSolder, B.Cu at (85.7, 178.8)
- added R15: 22R, Resistor_SMD:R_0603_1608Metric_Pad0.98x0.95mm_HandSolder, B.Cu at (122.6, 123.3)
- added R16: 10k, Resistor_SMD:R_0603_1608Metric_Pad0.98x0.95mm_HandSolder, B.Cu at (84.1, 179.7)
- added R17: 22R, Resistor_SMD:R_0603_1608Metric_Pad0.98x0.95mm_HandSolder, F.Cu at (122.6, 123.3)
- added R18: 10k, Resistor_SMD:R_0603_1608Metric_Pad0.98x0.95mm_HandSolder, B.Cu at (115.5, 171.6)
- added R19: 22R, Resistor_SMD:R_0603_1608Metric_Pad0.98x0.95mm_HandSolder, F.Cu at (121.4, 156.5)
- added R2: 22R, Resistor_SMD:R_0603_1608Metric_Pad0.98x0.95mm_HandSolder, B.Cu at (122.6, 121.6)
- added R20: 4k7, Resistor_SMD:R_0603_1608Metric_Pad0.98x0.95mm_HandSolder, B.Cu at (121.7, 127.4)
- added R21: 22R, Resistor_SMD:R_0603_1608Metric_Pad0.98x0.95mm_HandSolder, B.Cu at (121.4, 156.5)
- added R22: 10k, Resistor_SMD:R_0603_1608Metric_Pad0.98x0.95mm_HandSolder, B.Cu at (122.6, 132.9)
- added R23: 22R, Resistor_SMD:R_0603_1608Metric_Pad0.98x0.95mm_HandSolder, F.Cu at (122.6, 119.8)
- added R24: 10k, Resistor_SMD:R_0603_1608Metric_Pad0.98x0.95mm_HandSolder, F.Cu at (98.4, 180.4)
- added R25: 22R, Resistor_SMD:R_0603_1608Metric_Pad0.98x0.95mm_HandSolder, B.Cu at (122.6, 119.8)
- added R26: 10k, Resistor_SMD:R_0603_1608Metric_Pad0.98x0.95mm_HandSolder, F.Cu at (93.2, 178.8)
- added R27: 22R, Resistor_SMD:R_0603_1608Metric_Pad0.98x0.95mm_HandSolder, B.Cu at (122.6, 118.1)
- added R28: 22R, Resistor_SMD:R_0603_1608Metric_Pad0.98x0.95mm_HandSolder, B.Cu at (125.1, 128.3)
- added R29: 22R, Resistor_SMD:R_0603_1608Metric_Pad0.98x0.95mm_HandSolder, F.Cu at (122.6, 118.1)
- added R3: 10k, Resistor_SMD:R_0603_1608Metric_Pad0.98x0.95mm_HandSolder, F.Cu at (122.6, 132.9)
- added R30: 22R, Resistor_SMD:R_0603_1608Metric_Pad0.98x0.95mm_HandSolder, B.Cu at (122.6, 134.6)
- added R31: 22R, Resistor_SMD:R_0603_1608Metric_Pad0.98x0.95mm_HandSolder, B.Cu at (122.6, 116.3)
- added R32: 22R, Resistor_SMD:R_0603_1608Metric_Pad0.98x0.95mm_HandSolder, F.Cu at (122.6, 116.3)
- added R33: 22R, Resistor_SMD:R_0603_1608Metric_Pad0.98x0.95mm_HandSolder, F.Cu at (122.6, 114.6)
- added R34: 22R, Resistor_SMD:R_0603_1608Metric_Pad0.98x0.95mm_HandSolder, B.Cu at (122.6, 114.6)
- added R35: 22R, Resistor_SMD:R_0603_1608Metric_Pad0.98x0.95mm_HandSolder, F.Cu at (122.6, 112.8)
- added R36: 10k, Resistor_SMD:R_0603_1608Metric_Pad0.98x0.95mm_HandSolder, F.Cu at (85.7, 178.8)
- added R37: 10k, Resistor_SMD:R_0603_1608Metric_Pad0.98x0.95mm_HandSolder, F.Cu at (84.1, 179.7)
- added R38: 10k, Resistor_SMD:R_0603_1608Metric_Pad0.98x0.95mm_HandSolder, F.Cu at (88.4, 191.3)
- added R39: 10k, Resistor_SMD:R_0603_1608Metric_Pad0.98x0.95mm_HandSolder, B.Cu at (88.4, 191.3)
- added R4: 22R, Resistor_SMD:R_0603_1608Metric_Pad0.98x0.95mm_HandSolder, F.Cu at (122.6, 121.6)
- added R40: 10k, Resistor_SMD:R_0603_1608Metric_Pad0.98x0.95mm_HandSolder, B.Cu at (98.9, 186.2)
- added R41: 10k, Resistor_SMD:R_0603_1608Metric_Pad0.98x0.95mm_HandSolder, F.Cu at (98.9, 186.2)
- added R42: 22R, Resistor_SMD:R_0603_1608Metric_Pad0.98x0.95mm_HandSolder, F.Cu at (87.2, 178.0)
- added R43: 22R, Resistor_SMD:R_0603_1608Metric_Pad0.98x0.95mm_HandSolder, B.Cu at (122.6, 112.8)
- added R44: 22R, Resistor_SMD:R_0603_1608Metric_Pad0.98x0.95mm_HandSolder, F.Cu at (125.1, 128.3)
- added R46: 10k, Resistor_SMD:R_0603_1608Metric_Pad0.98x0.95mm_HandSolder, B.Cu at (108.2, 174.4)
- added R47: 10k, Resistor_SMD:R_0603_1608Metric_Pad0.98x0.95mm_HandSolder, B.Cu at (109.1, 169.6)
- added R48: 22R, Resistor_SMD:R_0603_1608Metric_Pad0.98x0.95mm_HandSolder, F.Cu at (122.6, 139.1)
- added R49: 22R, Resistor_SMD:R_0603_1608Metric_Pad0.98x0.95mm_HandSolder, B.Cu at (122.6, 139.1)
- added R5: 22R, Resistor_SMD:R_0603_1608Metric_Pad0.98x0.95mm_HandSolder, B.Cu at (122.6, 125.0)
- added R50: 22R, Resistor_SMD:R_0603_1608Metric_Pad0.98x0.95mm_HandSolder, F.Cu at (122.6, 141.6)
- added R51: 22R, Resistor_SMD:R_0603_1608Metric_Pad0.98x0.95mm_HandSolder, B.Cu at (122.6, 141.6)
- added R52: 22R, Resistor_SMD:R_0603_1608Metric_Pad0.98x0.95mm_HandSolder, F.Cu at (122.6, 144.1)
- added R53: 22R, Resistor_SMD:R_0603_1608Metric_Pad0.98x0.95mm_HandSolder, B.Cu at (122.6, 144.1)
- added R54: 22R, Resistor_SMD:R_0603_1608Metric_Pad0.98x0.95mm_HandSolder, F.Cu at (122.6, 146.6)
- added R55: 22R, Resistor_SMD:R_0603_1608Metric_Pad0.98x0.95mm_HandSolder, B.Cu at (122.6, 146.6)
- added R56: 22R, Resistor_SMD:R_0603_1608Metric_Pad0.98x0.95mm_HandSolder, B.Cu at (122.8, 149.2)
- added R57: 22R, Resistor_SMD:R_0603_1608Metric_Pad0.98x0.95mm_HandSolder, F.Cu at (122.8, 149.2)
- added R58: 22R, Resistor_SMD:R_0603_1608Metric_Pad0.98x0.95mm_HandSolder, B.Cu at (87.2, 178.0)
- added R59: 22R, Resistor_SMD:R_0603_1608Metric_Pad0.98x0.95mm_HandSolder, F.Cu at (82.6, 180.6)
- added R6: 22R, Resistor_SMD:R_0603_1608Metric_Pad0.98x0.95mm_HandSolder, F.Cu at (122.6, 134.6)
- added R60: 22R, Resistor_SMD:R_0603_1608Metric_Pad0.98x0.95mm_HandSolder, B.Cu at (82.6, 180.6)
- added R61: 22R, Resistor_SMD:R_0603_1608Metric_Pad0.98x0.95mm_HandSolder, B.Cu at (100.3, 160.3)
- added R62: 22R, Resistor_SMD:R_0603_1608Metric_Pad0.98x0.95mm_HandSolder, F.Cu at (100.3, 160.3)
- added R63: 22R, Resistor_SMD:R_0603_1608Metric_Pad0.98x0.95mm_HandSolder, B.Cu at (102.0, 160.3)
- added R64: 22R, Resistor_SMD:R_0603_1608Metric_Pad0.98x0.95mm_HandSolder, F.Cu at (102.0, 160.3)
- added R65: 10k, Resistor_SMD:R_0603_1608Metric_Pad0.98x0.95mm_HandSolder, F.Cu at (93.2, 184.3)
- added R7: 22R, Resistor_SMD:R_0603_1608Metric_Pad0.98x0.95mm_HandSolder, F.Cu at (122.6, 125.0)
- added R8: 22R, Resistor_SMD:R_0603_1608Metric_Pad0.98x0.95mm_HandSolder, B.Cu at (218.8, 186.3)
- added R9: 22R, Resistor_SMD:R_0603_1608Metric_Pad0.98x0.95mm_HandSolder, B.Cu at (122.6, 136.5)
- added RSW1: RotaryEncoder_Switch, Rotary_Encoder:RotaryEncoder_Alps_EC12E-Switch_Vertical_H20mm_CircularMountingHoles, F.Cu at (99.2, 200.1)
- added SW1: Cherry, Button_Switch_Keyboard:Kailh_socket_MX_LED, F.Cu at (138.3, 107.3)
- added SW10: Cherry, Button_Switch_Keyboard:Kailh_socket_MX_LED, B.Cu at (214.5, 107.3)
- added SW11: Cherry, Button_Switch_Keyboard:Kailh_socket_MX_LED, F.Cu at (138.3, 126.4)
- added SW12: Cherry, Button_Switch_Keyboard:Kailh_socket_MX_LED, B.Cu at (138.3, 126.4)
- added SW13: Cherry, Button_Switch_Keyboard:Kailh_socket_MX_LED, F.Cu at (157.4, 126.4)
- added SW14: Cherry, Button_Switch_Keyboard:Kailh_socket_MX_LED, B.Cu at (157.4, 126.4)
- added SW15: Cherry, Button_Switch_Keyboard:Kailh_socket_MX_LED, F.Cu at (176.4, 126.4)
- added SW16: Cherry, Button_Switch_Keyboard:Kailh_socket_MX_LED, B.Cu at (176.4, 126.4)
- added SW17: Cherry, Button_Switch_Keyboard:Kailh_socket_MX_LED, F.Cu at (195.5, 126.4)
- added SW18: Cherry, Button_Switch_Keyboard:Kailh_socket_MX_LED, B.Cu at (195.5, 126.4)
- added SW19: Cherry, Button_Switch_Keyboard:Kailh_socket_MX_LED, F.Cu at (214.5, 126.4)
- added SW2: Cherry, Button_Switch_Keyboard:Kailh_socket_MX_LED, B.Cu at (138.3, 107.3)
- added SW20: Cherry, Button_Switch_Keyboard:Kailh_socket_MX_LED, B.Cu at (214.5, 126.4)
- added SW21: Cherry, Button_Switch_Keyboard:Kailh_socket_MX_LED, F.Cu at (138.3, 145.4)
- added SW22: Cherry, Button_Switch_Keyboard:Kailh_socket_MX_LED, B.Cu at (138.3, 145.4)
- added SW23: Cherry, Button_Switch_Keyboard:Kailh_socket_MX_LED, F.Cu at (157.4, 145.4)
- added SW24: Cherry, Button_Switch_Keyboard:Kailh_socket_MX_LED, B.Cu at (157.4, 145.4)
- added SW25: Cherry, Button_Switch_Keyboard:Kailh_socket_MX_LED, F.Cu at (176.4, 145.4)
- added SW26: Cherry, Button_Switch_Keyboard:Kailh_socket_MX_LED, B.Cu at (176.4, 145.4)
- added SW27: Cherry, Button_Switch_Keyboard:Kailh_socket_MX_LED, F.Cu at (195.5, 145.4)
- added SW28: Cherry, Button_Switch_Keyboard:Kailh_socket_MX_LED, B.Cu at (195.5, 145.4)
- added SW29: Cherry, Button_Switch_Keyboard:Kailh_socket_MX_LED, F.Cu at (214.5, 145.4)
- added SW3: Cherry, Button_Switch_Keyboard:Kailh_socket_MX_LED, F.Cu at (157.4, 107.3)
- added SW30: Cherry, Button_Switch_Keyboard:Kailh_socket_MX_LED, B.Cu at (214.5, 145.4)
- added SW31: Cherry, Button_Switch_Keyboard:Kailh_socket_MX_LED, F.Cu at (138.3, 164.5)
- added SW32: Cherry, Button_Switch_Keyboard:Kailh_socket_MX_LED, B.Cu at (138.3, 164.5)
- added SW33: Cherry, Button_Switch_Keyboard:Kailh_socket_MX_LED, F.Cu at (157.4, 164.5)
- added SW34: Cherry, Button_Switch_Keyboard:Kailh_socket_MX_LED, B.Cu at (157.4, 164.5)
- added SW35: Cherry, Button_Switch_Keyboard:Kailh_socket_MX_LED, F.Cu at (176.4, 164.5)
- added SW36: Cherry, Button_Switch_Keyboard:Kailh_socket_MX_LED, B.Cu at (176.4, 164.5)
- added SW37: Cherry, Button_Switch_Keyboard:Kailh_socket_MX_LED, F.Cu at (195.5, 164.5)
- added SW38: Cherry, Button_Switch_Keyboard:Kailh_socket_MX_LED, B.Cu at (195.5, 164.5)
- added SW39: Cherry, Button_Switch_Keyboard:Kailh_socket_MX_LED, F.Cu at (214.5, 164.5)
- added SW4: Cherry, Button_Switch_Keyboard:Kailh_socket_MX_LED, B.Cu at (157.4, 107.3)
- added SW40: Cherry, Button_Switch_Keyboard:Kailh_socket_MX_LED, B.Cu at (214.5, 164.5)
- added SW41: Cherry, Button_Switch_Keyboard:Kailh_socket_MX_LED, F.Cu at (121.2, 190.1)
- added SW42: Cherry, Button_Switch_Keyboard:Kailh_socket_MX_LED, B.Cu at (121.2, 190.1)
- added SW43: Cherry, Button_Switch_Keyboard:Kailh_socket_MX_LED, F.Cu at (147.8, 189.1)
- added SW44: Cherry, Button_Switch_Keyboard:Kailh_socket_MX_LED, B.Cu at (147.8, 189.1)
- added SW45: Cherry, Button_Switch_Keyboard:Kailh_socket_MX_LED, F.Cu at (173.5, 186.4)
- added SW46: Cherry, Button_Switch_Keyboard:Kailh_socket_MX_LED, B.Cu at (173.5, 186.4)
- added SW47: Cherry, Button_Switch_Keyboard:Kailh_socket_MX_LED, F.Cu at (197.4, 186.4)
- added SW48: Cherry, Button_Switch_Keyboard:Kailh_socket_MX_LED, B.Cu at (197.4, 186.4)
- added SW5: Cherry, Button_Switch_Keyboard:Kailh_socket_MX_LED, F.Cu at (176.4, 107.3)
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Routing:
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- added copper zone on B.Cu, net GND
- added copper zone on F.Cu, net GND
Other:
- board size 363.8 x 149.2 mm -> 158.4 x 138.3 mm
- board text added: "IsoKey v5 split"
- board text added: "Plate Left"
- board text added: "Plate Right"
- board text added: "asterix24@gmail.com"
- board text added: "󰄼"
- board text added: "󰚌"
- board text added: "󰚫"
- board text added: "󰛤"
- board text added: "󰞷"
- board text added: "󰠖"
- board text added: "󰣘"
- board text removed: "DB"
- board text removed: "Iso"
- board text removed: "Key"
- board text removed: "v.4"
